File: pcb/reverse-singlerom/reverse-singlerom.kicad_sch (KiCad schematic)
At the start: 3 parts

Commit message: reversing some pins
Connections:
- net at IC2.10 (A0): now also J1.33 (Pin_33)
- net at IC1.10 (A1): now also J1.78 (Pin_78)
- net at IC1.12 (~CE): now also J1.72 (Pin_72)
- net at IC1.15 (D0): now also J1.35 (Pin_35)
- net at IC1.16 (D8): now also J1.42 (Pin_42)
- net at IC1.17 (D1): now also J1.81 (Pin_81)
- net at IC1.19 (D2): now also J1.37 (Pin_37)
- net at IC1.2 (A18): now also J1.76 (Pin_76)
- net at IC1.20 (D10): now also J1.44 (Pin_44)
- net at IC1.21 (D3): now also J1.38 (Pin_38)
- net at IC1.8 (A3): now also J1.77 (Pin_77)
- net at IC1.9 (A2): now also J1.30 (Pin_30)
Other:
- moved on the sheet: J1
Changed lines of the file:
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@@
 (kicad_sch (version 20230121) (generator eeschema)
   (paper "A4")
+  (wire (pts (xy 156.21 96.52) (xy 144.78 96.52))
+    (stroke (width 0) (type default))
+  )
+  (wire (pts (xy 133.35 25.4) (xy 234.95 25.4))
+    (stroke (width 0) (type default))
+  )
+  (wire (pts (xy 156.21 101.6) (xy 134.62 101.6))
+    (stroke (width 0) (type default))
+  )
+  (wire (pts (xy 143.51 20.32) (xy 241.3 20.32))
+    (stroke (width 0) (type default))
+  )
+  (wire (pts (xy 139.7 93.98) (xy 139.7 143.51))
+    (stroke (width 0) (type default))
+  )
+  (wire (pts (xy 125.73 91.44) (xy 125.73 125.73))
+    (stroke (width 0) (type default))
+  )
+  (wire (pts (xy 246.38 85.09) (xy 222.25 85.09))
+    (stroke (width 0) (type default))
+  )
+  (wire (pts (xy 139.7 143.51) (xy 199.39 143.51))
+    (stroke (width 0) (type default))
+  )
+  (wire (pts (xy 125.73 125.73) (xy 199.39 125.73))
+    (stroke (width 0) (type default))
+  )
+  (wire (pts (xy 234.95 72.39) (xy 222.25 72.39))
+    (stroke (width 0) (type default))
+  )
+  (wire (pts (xy 128.27 121.92) (xy 194.31 121.92))
+    (stroke (width 0) (type default))
+  )
+  (wire (pts (xy 199.39 120.65) (xy 85.09 120.65))
+    (stroke (width 0) (type default))
+  )
+  (wire (pts (xy 144.78 133.35) (xy 199.39 133.35))
+    (stroke (width 0) (type default))
+  )
+  (wire (pts (xy 241.3 74.93) (xy 222.25 74.93))
+    (stroke (width 0) (type default))
+  )
+  (wire (pts (xy 85.09 120.65) (xy 85.09 86.36))
+    (stroke (width 0) (type default))
+  )
+  (wire (pts (xy 144.78 106.68) (xy 144.78 133.35))
+    (stroke (width 0) (type default))
+  )
+  (wire (pts (xy 194.31 113.03) (xy 199.39 113.03))
+    (stroke (width 0) (type default))
+  )
+  (wire (pts (xy 260.35 62.23) (xy 222.25 62.23))
+    (stroke (width 0) (type default))
+  )
+  (wire (pts (xy 156.21 78.74) (xy 140.97 78.74))
+    (stroke (width 0) (type default))
+  )
+  (wire (pts (xy 147.32 104.14) (xy 147.32 148.59))
+    (stroke (width 0) (type default))
+  )
+  (wire (pts (xy 143.51 58.42) (xy 143.51 20.32))
+    (stroke (width 0) (type default))
+  )
+  (wire (pts (xy 194.31 121.92) (xy 194.31 113.03))
+    (stroke (width 0) (type default))
+  )
+  (wire (pts (xy 144.78 26.67) (xy 260.35 26.67))
+    (stroke (width 0) (type default))
+  )
+  (wire (pts (xy 137.16 15.24) (xy 246.38 15.24))
+    (stroke (width 0) (type default))
+  )
+  (wire (pts (xy 133.35 73.66) (xy 133.35 25.4))
+    (stroke (width 0) (type default))
+  )
+  (wire (pts (xy 156.21 106.68) (xy 144.78 106.68))
+    (stroke (width 0) (type default))
+  )
+  (wire (pts (xy 156.21 104.14) (xy 147.32 104.14))
+    (stroke (width 0) (type default))
+  )
+  (wire (pts (xy 156.21 93.98) (xy 139.7 93.98))
+    (stroke (width 0) (type default))
+  )
+  (wire (pts (xy 156.21 73.66) (xy 133.35 73.66))
+    (stroke (width 0) (type default))
+  )
+  (wire (pts (xy 147.32 148.59) (xy 199.39 148.59))
+    (stroke (width 0) (type default))
+  )
+  (wire (pts (xy 134.62 130.81) (xy 199.39 130.81))
+    (stroke (width 0) (type default))
+  )
+  (wire (pts (xy 246.38 15.24) (xy 246.38 85.09))
+    (stroke (width 0) (type default))
+  )
+  (wire (pts (xy 156.21 91.44) (xy 125.73 91.44))
+    (stroke (width 0) (type default))
+  )
+  (wire (pts (xy 128.27 76.2) (xy 128.27 121.92))
+    (stroke (width 0) (type default))
+  )
+  (wire (pts (xy 241.3 20.32) (xy 241.3 74.93))
+    (stroke (width 0) (type default))
+  )
+  (wire (pts (xy 234.95 25.4) (xy 234.95 72.39))
+    (stroke (width 0) (type default))
+  )
+  (wire (pts (xy 140.97 78.74) (xy 140.97 17.78))
+    (stroke (width 0) (type default))
+  )
+  (wire (pts (xy 156.21 58.42) (xy 143.51 58.42))
+    (stroke (width 0) (type default))
+  )
+  (wire (pts (xy 156.21 83.82) (xy 137.16 83.82))
+    (stroke (width 0) (type default))
+  )
+  (wire (pts (xy 85.09 86.36) (xy 96.52 86.36))
+    (stroke (width 0) (type default))
+  )
+  (wire (pts (xy 134.62 101.6) (xy 134.62 130.81))
+    (stroke (width 0) (type default))
+  )
+  (wire (pts (xy 156.21 76.2) (xy 128.27 76.2))
+    (stroke (width 0) (type default))
+  )
+  (wire (pts (xy 144.78 96.52) (xy 144.78 26.67))
+    (stroke (width 0) (type default))
+  )
+  (wire (pts (xy 256.54 69.85) (xy 222.25 69.85))
+    (stroke (width 0) (type default))
+  )
+  (wire (pts (xy 137.16 83.82) (xy 137.16 15.24))
+    (stroke (width 0) (type default))
+  )
+  (wire (pts (xy 256.54 17.78) (xy 256.54 69.85))
+    (stroke (width 0) (type default))
+  )
+  (wire (pts (xy 260.35 26.67) (xy 260.35 62.23))
+    (stroke (width 0) (type default))
+  )
+  (wire (pts (xy 140.97 17.78) (xy 256.54 17.78))
+    (stroke (width 0) (type default))
+  )
   (symbol (lib_id "LOOPY_Cart:HM9264BLFP") (at 106.68 60.96 0) (unit 1)
     (in_bom yes) (on_board yes) (dnp no) (fields_autoplaced)
@@
     )
   )
-  (symbol (lib_id "LOOPY_Cart:LOOPY-Cart-Connector") (at 43.18 33.02 0) (unit 1)
+  (symbol (lib_id "LOOPY_Cart:LOOPY-Cart-Connector") (at 210.82 36.83 0) (unit 1)
     (in_bom yes) (on_board yes) (dnp no) (fields_autoplaced)
-    (property "Reference" "J1" (at 43.18 31.75 0)
-      (effects (font (size 1.27 1.27)))
-    )
-    (property "Value" "~" (at 43.18 33.02 0)
-      (effects (font (size 1.27 1.27)))
-    )
-    (property "Footprint" "LOOPY_Cart:LOOPY-Edge-Connector" (at 43.18 33.02 0)
-      (effects (font (size 1.27 1.27)) hide)
-    )
-    (property "Datasheet" "" (at 43.18 33.02 0)
-      (effects (font (size 1.27 1.27)) hide)
-    )
+    (property "Reference" "J1" (at 210.82 35.56 0)
+      (effects (font (size 1.27 1.27)))
+    )
+    (property "Value" "~" (at 210.82 36.83 0)
+      (effects (font (size 1.27 1.27)))
+    )
+    (property "Footprint" "LOOPY_Cart:LOOPY-Edge-Connector" (at 210.82 36.83 0)
+      (effects (font (size 1.27 1.27)) hide)
+    )
+    (property "Datasheet" "" (at 210.82 36.83 0)
+      (effects (font (size 1.27 1.27)) hide)
+    )

Commit message: Continue tracing
Connections:
- net at IC2.22 (~OE): now also IC1.14 (~OE), J1.56 (Pin_56)
- net at IC1.11 (A0): now also J1.32 (Pin_32)
- net at IC1.18 (D9): now also J1.88 (Pin_88)
- net at IC1.22 (D11): now also J1.90 (Pin_90)
- net at IC1.24 (D4): now also J1.40 (Pin_40)
- net at IC1.25 (D12): now also J1.82 (Pin_82)
- net at IC1.26 (D5): now also J1.85 (Pin_85)
- net at IC1.27 (D13): now also J1.83 (Pin_83)
- net at IC1.28 (D6): now also J1.41 (Pin_41)
- net at IC1.29 (D14): now also J1.39 (Pin_39)
- net at IC1.30 (D7): now also J1.86 (Pin_86)
- net at IC1.31 (D15): now also J1.84 (Pin_84)
- net at IC1.36 (A14): now also J1.27 (Pin_27)
- net at IC1.43 (A19): now also J1.28 (Pin_28)
- no-connect marks 0 -> 38
Changed lines of the file:
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@@
 (kicad_sch (version 20230121) (generator eeschema)
   (paper "A4")
+  (junction (at 133.35 88.9) (diameter 0) (color 0 0 0 0)
+  )
+  (no_connect (at 199.39 80.01))
+  (no_connect (at 199.39 74.93))
+  (no_connect (at 222.25 146.05))
+  (no_connect (at 222.25 67.31))
+  (no_connect (at 199.39 46.99))
+  (no_connect (at 199.39 44.45))
+  (no_connect (at 222.25 140.97))
+  (no_connect (at 199.39 90.17))
+  (no_connect (at 222.25 133.35))
+  (no_connect (at 199.39 54.61))
+  (no_connect (at 199.39 52.07))
+  (no_connect (at 199.39 85.09))
+  (no_connect (at 199.39 123.19))
+  (no_connect (at 199.39 87.63))
+  (no_connect (at 222.25 100.33))
+  (no_connect (at 222.25 102.87))
+  (no_connect (at 199.39 115.57))
+  (no_connect (at 222.25 107.95))
+  (no_connect (at 199.39 57.15))
+  (no_connect (at 222.25 118.11))
+  (no_connect (at 199.39 146.05))
+  (no_connect (at 222.25 128.27))
+  (no_connect (at 222.25 135.89))
+  (no_connect (at 222.25 46.99))
+  (no_connect (at 222.25 64.77))
+  (no_connect (at 222.25 120.65))
+  (no_connect (at 199.39 62.23))
+  (no_connect (at 199.39 67.31))
+  (no_connect (at 199.39 41.91))
+  (no_connect (at 222.25 138.43))
+  (no_connect (at 199.39 82.55))
+  (no_connect (at 222.25 105.41))
+  (no_connect (at 199.39 49.53))
+  (no_connect (at 290.83 38.1))
+  (no_connect (at 222.25 143.51))
+  (no_connect (at 222.25 115.57))
+  (no_connect (at 222.25 151.13))
+  (no_connect (at 222.25 110.49))
+  (wire (pts (xy 177.8 106.68) (xy 182.88 106.68))
+    (stroke (width 0) (type default))
+  )
   (wire (pts (xy 156.21 96.52) (xy 144.78 96.52))
     (stroke (width 0) (type default))
@@
     (stroke (width 0) (type default))
   )
+  (wire (pts (xy 231.14 31.75) (xy 231.14 57.15))
+    (stroke (width 0) (type default))
+  )
   (wire (pts (xy 156.21 101.6) (xy 134.62 101.6))
     (stroke (width 0) (type default))
@@
     (stroke (width 0) (type default))
   )
+  (wire (pts (xy 130.81 118.11) (xy 199.39 118.11))
+    (stroke (width 0) (type default))
+  )
   (wire (pts (xy 139.7 93.98) (xy 139.7 143.51))
     (stroke (width 0) (type default))
   )
+  (wire (pts (xy 185.42 104.14) (xy 185.42 30.48))
+    (stroke (width 0) (type default))
+  )
+  (wire (pts (xy 133.35 88.9) (xy 133.35 170.18))
+    (stroke (width 0) (type default))
+  )
+  (wire (pts (xy 116.84 78.74) (xy 124.46 78.74))
+    (stroke (width 0) (type default))
+  )
+  (wire (pts (xy 236.22 24.13) (xy 236.22 52.07))
+    (stroke (width 0) (type default))
+  )
+  (wire (pts (xy 156.21 81.28) (xy 130.81 81.28))
+    (stroke (width 0) (type default))
+  )
   (wire (pts (xy 125.73 91.44) (xy 125.73 125.73))
     (stroke (width 0) (type default))
@@
     (stroke (width 0) (type default))
   )
+  (wire (pts (xy 146.05 27.94) (xy 222.25 27.94))
+    (stroke (width 0) (type default))
+  )
   (wire (pts (xy 139.7 143.51) (xy 199.39 143.51))
     (stroke (width 0) (type default))
@@
     (stroke (width 0) (type default))
   )
+  (wire (pts (xy 237.49 49.53) (xy 237.49 22.86))
+    (stroke (width 0) (type default))
+  )
   (wire (pts (xy 234.95 72.39) (xy 222.25 72.39))
     (stroke (width 0) (type default))
   )
+  (wire (pts (xy 237.49 22.86) (xy 182.88 22.86))
+    (stroke (width 0) (type default))
+  )
   (wire (pts (xy 128.27 121.92) (xy 194.31 121.92))
     (stroke (width 0) (type default))
   )
+  (wire (pts (xy 227.33 44.45) (xy 222.25 44.45))
+    (stroke (width 0) (type default))
+  )
+  (wire (pts (xy 156.21 88.9) (xy 133.35 88.9))
+    (stroke (width 0) (type default))
+  )
+  (wire (pts (xy 181.61 140.97) (xy 181.61 96.52))
+    (stroke (width 0) (type default))
+  )
   (wire (pts (xy 199.39 120.65) (xy 85.09 120.65))
     (stroke (width 0) (type default))
   )
+  (wire (pts (xy 181.61 96.52) (xy 177.8 96.52))
+    (stroke (width 0) (type default))
+  )
   (wire (pts (xy 144.78 133.35) (xy 199.39 133.35))
     (stroke (width 0) (type default))
   )
+  (wire (pts (xy 255.27 125.73) (xy 222.25 125.73))
+    (stroke (width 0) (type default))
+  )
+  (wire (pts (xy 182.88 91.44) (xy 177.8 91.44))
+    (stroke (width 0) (type default))
+  )
+  (wire (pts (xy 138.43 99.06) (xy 138.43 29.21))
+    (stroke (width 0) (type default))
+  )
+  (wire (pts (xy 186.69 58.42) (xy 186.69 107.95))
+    (stroke (width 0) (type default))
+  )
+  (wire (pts (xy 232.41 30.48) (xy 232.41 59.69))
+    (stroke (width 0) (type default))
+  )
   (wire (pts (xy 241.3 74.93) (xy 222.25 74.93))
     (stroke (width 0) (type default))
@@
     (stroke (width 0) (type default))
   )
+  (wire (pts (xy 184.15 24.13) (xy 236.22 24.13))
+    (stroke (width 0) (type default))
+  )
   (wire (pts (xy 144.78 106.68) (xy 144.78 133.35))
     (stroke (width 0) (type default))
   )
+  (wire (pts (xy 156.21 99.06) (xy 138.43 99.06))
+    (stroke (width 0) (type default))
+  )
   (wire (pts (xy 194.31 113.03) (xy 199.39 113.03))
     (stroke (width 0) (type default))
@@
     (stroke (width 0) (type default))
   )
+  (wire (pts (xy 199.39 135.89) (xy 180.34 135.89))
+    (stroke (width 0) (type default))
+  )
+  (wire (pts (xy 146.05 109.22) (xy 146.05 27.94))
+    (stroke (width 0) (type default))
+  )
   (wire (pts (xy 156.21 78.74) (xy 140.97 78.74))
     (stroke (width 0) (type default))
   )
+  (wire (pts (xy 266.7 54.61) (xy 266.7 160.02))
+    (stroke (width 0) (type default))
+  )
+  (wire (pts (xy 130.81 81.28) (xy 130.81 118.11))
+    (stroke (width 0) (type default))
+  )
+  (wire (pts (xy 180.34 93.98) (xy 177.8 93.98))
+    (stroke (width 0) (type default))
+  )
+  (wire (pts (xy 186.69 107.95) (xy 199.39 107.95))
+    (stroke (width 0) (type default))
+  )
+  (wire (pts (xy 231.14 57.15) (xy 222.25 57.15))
+    (stroke (width 0) (type default))
+  )
   (wire (pts (xy 147.32 104.14) (xy 147.32 148.59))
     (stroke (width 0) (type default))
@@
     (stroke (width 0) (type default))
   )
+  (wire (pts (xy 180.34 135.89) (xy 180.34 93.98))
+    (stroke (width 0) (type default))
+  )
   (wire (pts (xy 137.16 15.24) (xy 246.38 15.24))
     (stroke (width 0) (type default))
   )
+  (wire (pts (xy 227.33 29.21) (xy 227.33 44.45))
+    (stroke (width 0) (type default))
+  )
+  (wire (pts (xy 182.88 138.43) (xy 199.39 138.43))
+    (stroke (width 0) (type default))
+  )
+  (wire (pts (xy 222.25 54.61) (xy 266.7 54.61))
+    (stroke (width 0) (type default))
+  )
+  (wire (pts (xy 187.96 105.41) (xy 199.39 105.41))
+    (stroke (width 0) (type default))
+  )
+  (wire (pts (xy 189.23 99.06) (xy 189.23 31.75))
+    (stroke (width 0) (type default))
+  )
+  (wire (pts (xy 232.41 59.69) (xy 222.25 59.69))
+    (stroke (width 0) (type default))
+  )
+  (wire (pts (xy 187.96 76.2) (xy 187.96 105.41))
+    (stroke (width 0) (type default))
+  )
+  (wire (pts (xy 156.21 109.22) (xy 146.05 109.22))
+    (stroke (width 0) (type default))
+  )
   (wire (pts (xy 133.35 73.66) (xy 133.35 25.4))
     (stroke (width 0) (type default))
   )
+  (wire (pts (xy 189.23 31.75) (xy 231.14 31.75))
+    (stroke (width 0) (type default))
+  )
   (wire (pts (xy 156.21 106.68) (xy 144.78 106.68))
     (stroke (width 0) (type default))
   )
+  (wire (pts (xy 138.43 29.21) (xy 227.33 29.21))
+    (stroke (width 0) (type default))
+  )
+  (wire (pts (xy 177.8 99.06) (xy 189.23 99.06))
+    (stroke (width 0) (type default))
+  )
   (wire (pts (xy 156.21 104.14) (xy 147.32 104.14))
     (stroke (width 0) (type default))
@@
     (stroke (width 0) (type default))
   )
+  (wire (pts (xy 177.8 101.6) (xy 184.15 101.6))
+    (stroke (width 0) (type default))
+  )
+  (wire (pts (xy 255.27 170.18) (xy 255.27 125.73))
+    (stroke (width 0) (type default))
+  )
+  (wire (pts (xy 182.88 22.86) (xy 182.88 91.44))
+    (stroke (width 0) (type default))
+  )
+  (wire (pts (xy 177.8 58.42) (xy 186.69 58.42))
+    (stroke (width 0) (type default))
+  )
   (wire (pts (xy 156.21 91.44) (xy 125.73 91.44))
     (stroke (width 0) (type default))
@@
     (stroke (width 0) (type default))
   )
+  (wire (pts (xy 133.35 170.18) (xy 255.27 170.18))
+    (stroke (width 0) (type default))
+  )
+  (wire (pts (xy 184.15 101.6) (xy 184.15 24.13))
+    (stroke (width 0) (type default))
+  )
+  (wire (pts (xy 179.07 88.9) (xy 177.8 88.9))
+    (stroke (width 0) (type default))
+  )
+  (wire (pts (xy 177.8 104.14) (xy 185.42 104.14))
+    (stroke (width 0) (type default))
+  )
   (wire (pts (xy 156.21 58.42) (xy 143.51 58.42))
     (stroke (width 0) (type default))
   )
+  (wire (pts (xy 236.22 52.07) (xy 222.25 52.07))
+    (stroke (width 0) (type default))
+  )
   (wire (pts (xy 156.21 83.82) (xy 137.16 83.82))
     (stroke (width 0) (type default))
@@
     (stroke (width 0) (type default))
   )
+  (wire (pts (xy 179.07 160.02) (xy 179.07 88.9))
+    (stroke (width 0) (type default))
+  )
+  (wire (pts (xy 124.46 88.9) (xy 133.35 88.9))
+    (stroke (width 0) (type default))
+  )
+  (wire (pts (xy 266.7 160.02) (xy 179.07 160.02))
+    (stroke (width 0) (type default))
+  )
+  (wire (pts (xy 177.8 76.2) (xy 187.96 76.2))
+    (stroke (width 0) (type default))
+  )
   (wire (pts (xy 134.62 101.6) (xy 134.62 130.81))
     (stroke (width 0) (type default))
   )
+  (wire (pts (xy 182.88 106.68) (xy 182.88 138.43))
+    (stroke (width 0) (type default))
+  )
+  (wire (pts (xy 124.46 78.74) (xy 124.46 88.9))
+    (stroke (width 0) (type default))
+  )
   (wire (pts (xy 156.21 76.2) (xy 128.27 76.2))
     (stroke (width 0) (type default))
@@
     (stroke (width 0) (type default))
   )
+  (wire (pts (xy 199.39 140.97) (xy 181.61 140.97))
+    (stroke (width 0) (type default))
+  )
   (wire (pts (xy 137.16 83.82) (xy 137.16 15.24))
     (stroke (width 0) (type default))
@@
     (stroke (width 0) (type default))
   )
+  (wire (pts (xy 222.25 49.53) (xy 237.49 49.53))
+    (stroke (width 0) (type default))
+  )
+  (wire (pts (xy 185.42 30.48) (xy 232.41 30.48))
+    (stroke (width 0) (type default))
+  )
+  (wire (pts (xy 222.25 27.94) (xy 222.25 39.37))
+    (stroke (width 0) (type default))
+  )

Commit message: Continue tracing
Connections:
- net at IC2.10 (A0): no longer J1.33 (Pin_33)
- net D3: now reaches IC2.15 (IO4)
- net D3: now also IC1.21 (D3), J1.38 (Pin_38)
- net D2: now reaches IC2.16 (IO5)
- net D2: now also IC1.19 (D2), J1.37 (Pin_37)
- net D1: now reaches IC2.17 (IO6)
- net D1: now also IC1.17 (D1), J1.81 (Pin_81)
- net D0: now reaches IC2.18 (IO7)
- net D0: now also IC1.15 (D0), J1.35 (Pin_35)
- net D7: now reaches IC2.19 (IO8)
- net D7: now also IC1.30 (D7), J1.86 (Pin_86)
- net at IC2.20 (~CS1): now also J1.9 (Pin_9)
- net OE: now reaches IC1.14 (~OE), IC2.22 (~OE), J1.56 (Pin_56)
- net at IC2.26 (CS2): now also J1.36 (Pin_36)
- net at IC2.27 (~WE): now also J1.11 (Pin_11)
- net A1: now reaches IC1.10 (A1), J1.78 (Pin_78)
- net A0: now reaches IC1.11 (A0), J1.32 (Pin_32)
- net at IC1.12 (~CE): now also J1.54 (Pin_54); no longer J1.72 (Pin_72)
- net GND: now reaches IC1.13 (GND)
- net GND: now also IC1.32 (GND)
- net D8: now reaches IC1.16 (D8), J1.42 (Pin_42)
- net D9: now reaches IC1.18 (D9), J1.88 (Pin_88)
- net A18: now reaches IC1.2 (A18), J1.76 (Pin_76)
- net D10: now reaches IC1.20 (D10), J1.44 (Pin_44)
- net D11: now reaches IC1.22 (D11), J1.90 (Pin_90)
- net at IC1.23 (VCC): now also IC1.33 (~BYTE)
- net D4: now reaches IC1.24 (D4), J1.40 (Pin_40)
- net D12: now reaches IC1.25 (D12), J1.82 (Pin_82)
- net D5: now reaches IC1.26 (D5), J1.85 (Pin_85)
- net D13: now reaches IC1.27 (D13), J1.83 (Pin_83)
- net D6: now reaches IC1.28 (D6), J1.41 (Pin_41)
- net D14: now reaches IC1.29 (D14), J1.39 (Pin_39)
- net A17: now reaches IC1.3 (A17)
- net A17: now also J1.74 (Pin_74)
- net D15: now reaches IC1.31 (D15), J1.84 (Pin_84)
- net A16: now reaches IC1.34 (A16)
- net A16: now also J1.72 (Pin_72)
- net A15: now reaches IC1.35 (A15)
- net A15: now also J1.73 (Pin_73)
- net A14: now reaches IC1.36 (A14), J1.27 (Pin_27)
- net A13: now reaches IC1.37 (A13)
- net A13: now also J1.71 (Pin_71)
- net A12: now reaches IC1.38 (A12)
- net A12: now also J1.26 (Pin_26)
- net A11: now reaches IC1.39 (A11)
- net A11: now also J1.22 (Pin_22)
- net A7: now reaches IC1.4 (A7)
- net A7: now also J1.24 (Pin_24)
- net A10: now reaches IC1.40 (A10)
- net A10: now also J1.67 (Pin_67)
- net A9: now reaches IC1.41 (A9)
- net A9: now also J1.23 (Pin_23)
- net A8: now reaches IC1.42 (A8)
- net A8: now also J1.68 (Pin_68)
- net A19: now reaches IC1.43 (A19), J1.28 (Pin_28)
- net A6: now reaches IC1.5 (A6)
- net A6: now also J1.69 (Pin_69)
- net A5: now reaches IC1.6 (A5)
- net A5: now also J1.25 (Pin_25)
- net A4: now reaches IC1.7 (A4)
- net A4: now also J1.70 (Pin_70)
- net A3: now reaches IC1.8 (A3), J1.77 (Pin_77)
- net A2: now reaches IC1.9 (A2), J1.30 (Pin_30)

Commit message: Traced all signal routes
Connections:
- net A0: now also IC2.9 (A1)
- net A1: now also IC2.8 (A2)
- net A10: now also IC2.4 (A6)
- net A11: now also IC2.5 (A5)
- net A2: now also IC2.7 (A3)
- net A3: now also IC2.21 (A10)
- net A4: now also IC2.6 (A4)
- net A5: now also IC2.23 (A11)
- net A6: now also IC2.24 (A9)
- net A7: now also IC2.25 (A8)
- net A8: now also IC2.2 (A12)
- net A9: now also IC2.3 (A7)
- net D4: now also IC2.13 (IO3)
- net D5: now also IC2.12 (IO2)
- net D6: now also IC2.11 (IO1)
- net GND: now also IC2.14 (GND)
- net at IC2.10 (A0): now also J1.33 (Pin_33)
