File: pcb/reverse-singlerom/reverse-singlerom.kicad_sch (KiCad schematic)
At the start: 3 parts

Commit message: Annotating power nets
Connections:
- net GND: now also J1.45 (Pin_45)
- net V1: now reaches J1.1 (Pin_1)
- net V1: now also J1.14 (Pin_14), J1.29 (Pin_29), J1.57 (Pin_57), J1.89 (Pin_89)
- net V2: now reaches J1.13 (Pin_13)
- net V2: now also J1.47 (Pin_47), J1.75 (Pin_75)
Changed lines of the file:
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@@
   (no_connect (at 222.25 151.13))
   (no_connect (at 222.25 110.49))
-  (wire (pts (xy 234.95 156.21) (xy 234.95 130.81))
+  (wire (pts (xy 194.31 151.13) (xy 199.39 151.13))
+    (stroke (width 0) (type default))
+  )
+  (wire (pts (xy 234.95 158.75) (xy 234.95 130.81))
     (stroke (width 0) (type default))
   )
@@
     (stroke (width 0) (type default))
   )
-  (wire (pts (xy 149.86 156.21) (xy 234.95 156.21))
+  (wire (pts (xy 149.86 158.75) (xy 234.95 158.75))
     (stroke (width 0) (type default))
   )
@@
     (stroke (width 0) (type default))
   )
+  (wire (pts (xy 222.25 148.59) (xy 229.87 148.59))
+    (stroke (width 0) (type default))
+  )
   (wire (pts (xy 156.21 88.9) (xy 133.35 88.9))
     (stroke (width 0) (type default))
@@
     (stroke (width 0) (type default))
   )
-  (wire (pts (xy 149.86 83.82) (xy 149.86 156.21))
+  (wire (pts (xy 199.39 39.37) (xy 191.77 39.37))
+    (stroke (width 0) (type default))
+  )
+  (wire (pts (xy 149.86 83.82) (xy 149.86 158.75))
+    (stroke (width 0) (type default))
+  )
+  (wire (pts (xy 191.77 35.56) (xy 191.77 39.37))
     (stroke (width 0) (type default))
   )
@@
     (effects (font (size 1.27 1.27)) (justify right bottom))
   )
+  (label "V1" (at 199.39 110.49 180) (fields_autoplaced)
+    (effects (font (size 1.27 1.27)) (justify right bottom))
+  )
   (label "D7" (at 222.25 49.53 0) (fields_autoplaced)
     (effects (font (size 1.27 1.27)) (justify left bottom))
   )
+  (label "V1" (at 222.25 123.19 0) (fields_autoplaced)
+    (effects (font (size 1.27 1.27)) (justify left bottom))
+  )
   (label "D0" (at 156.21 91.44 180) (fields_autoplaced)
     (effects (font (size 1.27 1.27)) (justify right bottom))
@@
     (effects (font (size 1.27 1.27)) (justify right bottom))
   )
+  (label "V1" (at 222.25 41.91 0) (fields_autoplaced)
+    (effects (font (size 1.27 1.27)) (justify left bottom))
+  )
+  (label "V2" (at 222.25 77.47 0) (fields_autoplaced)
+    (effects (font (size 1.27 1.27)) (justify left bottom))
+  )
   (label "D1" (at 222.25 62.23 0) (fields_autoplaced)
     (effects (font (size 1.27 1.27)) (justify left bottom))
@@
     (effects (font (size 1.27 1.27)) (justify left bottom))
   )
+  (label "V1" (at 199.39 39.37 180) (fields_autoplaced)
+    (effects (font (size 1.27 1.27)) (justify right bottom))
+  )
+  (label "V2" (at 199.39 69.85 180) (fields_autoplaced)
+    (effects (font (size 1.27 1.27)) (justify right bottom))
+  )
   (label "A7" (at 116.84 71.12 0) (fields_autoplaced)
     (effects (font (size 1.27 1.27)) (justify left bottom))
@@
     (effects (font (size 1.27 1.27)) (justify left bottom))
   )
+  (label "V1" (at 199.39 72.39 180) (fields_autoplaced)
+    (effects (font (size 1.27 1.27)) (justify right bottom))
+  )
   (label "A2" (at 199.39 113.03 180) (fields_autoplaced)
     (effects (font (size 1.27 1.27)) (justify right bottom))
@@
     (effects (font (size 1.27 1.27)) (justify left bottom))
   )
+  (label "GND" (at 199.39 151.13 180) (fields_autoplaced)
+    (effects (font (size 1.27 1.27)) (justify right bottom))
+  )
   (label "A15" (at 222.25 82.55 0) (fields_autoplaced)
     (effects (font (size 1.27 1.27)) (justify left bottom))
@@
     (effects (font (size 1.27 1.27)) (justify right bottom))
   )
+  (label "V2" (at 222.25 148.59 0) (fields_autoplaced)
+    (effects (font (size 1.27 1.27)) (justify left bottom))
+  )
   (label "A19" (at 177.8 58.42 0) (fields_autoplaced)
     (effects (font (size 1.27 1.27)) (justify left bottom))
@@
     (effects (font (size 1.27 1.27)) (justify right bottom))
   )
+  (symbol (lib_id "power:GND") (at 194.31 151.13 0) (unit 1)
+    (in_bom yes) (on_board yes) (dnp no) (fields_autoplaced)
+    (property "Reference" "#PWR01" (at 194.31 157.48 0)
+      (effects (font (size 1.27 1.27)) hide)
+    )
+    (property "Value" "GND" (at 194.31 156.21 0)
+      (effects (font (size 1.27 1.27)))
+    )
+    (property "Footprint" "" (at 194.31 151.13 0)
+      (effects (font (size 1.27 1.27)) hide)
+    )
+    (property "Datasheet" "" (at 194.31 151.13 0)
+      (effects (font (size 1.27 1.27)) hide)
+    )
+    (pin "1")
+    (instances
+      (project "reverse-singlerom"
+        (path "/5081f4fb-0c92-4cfc-8c52-39777c6d96ed"
+          (reference "#PWR01") (unit 1)
+        )
+      )
+    )
+  )
+  (symbol (lib_id "power:PWR_FLAG") (at 229.87 148.59 0) (unit 1)
+    (in_bom yes) (on_board yes) (dnp no) (fields_autoplaced)
+    (property "Reference" "#FLG02" (at 229.87 146.685 0)
+      (effects (font (size 1.27 1.27)) hide)
+    )
+    (property "Value" "PWR_FLAG" (at 229.87 144.78 0)
+      (effects (font (size 1.27 1.27)))
+    )
+    (property "Footprint" "" (at 229.87 148.59 0)
+      (effects (font (size 1.27 1.27)) hide)
+    )
+    (property "Datasheet" "~" (at 229.87 148.59 0)
+      (effects (font (size 1.27 1.27)) hide)
+    )
+    (pin "1")
+    (instances
+      (project "reverse-singlerom"
+        (path "/5081f4fb-0c92-4cfc-8c52-39777c6d96ed"
+          (reference "#FLG02") (unit 1)
+        )
+      )
+    )
+  )
+  (symbol (lib_id "power:PWR_FLAG") (at 191.77 35.56 0) (unit 1)
+    (in_bom yes) (on_board yes) (dnp no) (fields_autoplaced)
+    (property "Reference" "#FLG03" (at 191.77 33.655 0)
+      (effects (font (size 1.27 1.27)) hide)
+    )
+    (property "Value" "PWR_FLAG" (at 191.77 31.75 0)
+      (effects (font (size 1.27 1.27)))
+    )
+    (property "Footprint" "" (at 191.77 35.56 0)
+      (effects (font (size 1.27 1.27)) hide)
+    )
+    (property "Datasheet" "~" (at 191.77 35.56 0)
+      (effects (font (size 1.27 1.27)) hide)
+    )
+    (pin "1")
+    (instances
+      (project "reverse-singlerom"
+        (path "/5081f4fb-0c92-4cfc-8c52-39777c6d96ed"
+          (reference "#FLG03") (unit 1)
+        )
+      )
+    )
+  )
   (symbol (lib_id "LOOPY_Cart:HM9264BLFP") (at 106.68 60.96 0) (unit 1)

Commit message: Update power nets
Connections:
- net V2 is gone; now on net GND: J1.13 (Pin_13), J1.47 (Pin_47), J1.75 (Pin_75)
- net V1 renamed +1V8
Changed lines of the file:
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@@
-    (stroke (width 0) (type default))
-  )
-  (wire (pts (xy 222.25 148.59) (xy 229.87 148.59))
     (stroke (width 0) (type default))
   )
@@
     (effects (font (size 1.27 1.27)) (justify left bottom))
   )
-  (label "V2" (at 222.25 77.47 0) (fields_autoplaced)
+  (label "GND" (at 222.25 77.47 0) (fields_autoplaced)
     (effects (font (size 1.27 1.27)) (justify left bottom))
   )
@@
     (effects (font (size 1.27 1.27)) (justify right bottom))
   )
-  (label "V2" (at 199.39 69.85 180) (fields_autoplaced)
+  (label "GND" (at 199.39 69.85 180) (fields_autoplaced)
     (effects (font (size 1.27 1.27)) (justify right bottom))
   )
@@
     (effects (font (size 1.27 1.27)) (justify right bottom))
   )
-  (label "V2" (at 222.25 148.59 0) (fields_autoplaced)
+  (label "GND" (at 222.25 148.59 0) (fields_autoplaced)
     (effects (font (size 1.27 1.27)) (justify left bottom))
   )
@@
         (path "/5081f4fb-0c92-4cfc-8c52-39777c6d96ed"
           (reference "#PWR01") (unit 1)
-        )
-      )
-    )
-  )
-  (symbol (lib_id "power:PWR_FLAG") (at 229.87 148.59 0) (unit 1)
-    (in_bom yes) (on_board yes) (dnp no) (fields_autoplaced)
-    (property "Reference" "#FLG02" (at 229.87 146.685 0)
-      (effects (font (size 1.27 1.27)) hide)
-    )
-    (property "Value" "PWR_FLAG" (at 229.87 144.78 0)
-      (effects (font (size 1.27 1.27)))
-    )
-    (property "Footprint" "" (at 229.87 148.59 0)
-      (effects (font (size 1.27 1.27)) hide)
-    )
-    (property "Datasheet" "~" (at 229.87 148.59 0)
-      (effects (font (size 1.27 1.27)) hide)
-    )
-    (pin "1")
-    (instances
-      (project "reverse-singlerom"
-        (path "/5081f4fb-0c92-4cfc-8c52-39777c6d96ed"
-          (reference "#FLG02") (unit 1)
-        )
-      )
-    )
-  )
-  (symbol (lib_id "power:PWR_FLAG") (at 191.77 35.56 0) (unit 1)
-    (in_bom yes) (on_board yes) (dnp no) (fields_autoplaced)
-    (property "Reference" "#FLG03" (at 191.77 33.655 0)
-      (effects (font (size 1.27 1.27)) hide)
-    )
-    (property "Value" "PWR_FLAG" (at 191.77 31.75 0)
-      (effects (font (size 1.27 1.27)))
-    )
-    (property "Footprint" "" (at 191.77 35.56 0)
-      (effects (font (size 1.27 1.27)) hide)
-    )
-    (property "Datasheet" "~" (at 191.77 35.56 0)
-      (effects (font (size 1.27 1.27)) hide)
-    )
-    (pin "1")
-    (instances
-      (project "reverse-singlerom"
-        (path "/5081f4fb-0c92-4cfc-8c52-39777c6d96ed"
-          (reference "#FLG03") (unit 1)
         )
       )
@@
         )
       )
+    )
+  )
+  (symbol (lib_id "power:+1V8") (at 191.77 35.56 0) (unit 1)
+    (in_bom yes) (on_board yes) (dnp no) (fields_autoplaced)
+    (property "Reference" "#PWR02" (at 191.77 39.37 0)
+      (effects (font (size 1.27 1.27)) hide)
+    )
+    (property "Value" "+1V8" (at 191.77 31.75 0)
+      (effects (font (size 1.27 1.27)))
+    )
+    (property "Footprint" "" (at 191.77 35.56 0)
+      (effects (font (size 1.27 1.27)) hide)
+    )
+    (property "Datasheet" "" (at 191.77 35.56 0)
+      (effects (font (size 1.27 1.27)) hide)
+    )
+    (pin "1")
+    (instances
+      (project "reverse-singlerom"
+        (path "/5081f4fb-0c92-4cfc-8c52-39777c6d96ed"
+          (reference "#PWR02") (unit 1)
+        )
+      )

Commit message: Adds power to reverse engineered cart
Parts:
- added BT1: CR-2032_HF1N, LOOPY_Batt:BAT_CR-2032_HF1N, symbol LOOPY_Batt:CR-2032_HF1N
- added C2, C3, C4: C, Capacitor_SMD:C_0805_2012Metric_Pad1.18x1.45mm_HandSolder, symbol Device:C
- added D1: MMBZxx, Package_TO_SOT_SMD:SOT-23, symbol Diode:MMBZxx
- added R1, R2: R, Resistor_SMD:R_0805_2012Metric_Pad1.20x1.40mm_HandSolder, symbol Device:R
Connections:
- net +1V8: now also IC1.23 (VCC), IC1.33 (~BYTE), C4.1, D1.1 (K)
- net GND: now also BT1.N, C2.2, C3.2, C4.2, R1.2
- net at IC2.26 (CS2), J1.36 (Pin_36): now also R1.1
- net at IC2.28 (VCC): now also C2.1, C3.1, D1.3 (A)
- new net: BT1.P, R2.1
- new net: D1.2 (K), R2.2
Other:
- note added: "Pulldown if unconnected?"
- title: (none) -> Reverse Engineered XK-403
- moved on the sheet: IC1, IC2

Commit message: Adds feature detect pins, fixes DRC errors
Parts:
- added R3, R4, R5, R6: R, Resistor_SMD:R_0805_2012Metric_Pad1.20x1.40mm_HandSolder, symbol Device:R
Connections:
- net GND: now also R4.2, R6.2
- net F16: now reaches J1.16 (Pin_16)
- net F16: now also R5.2, R6.1
- net F61: now reaches J1.61 (Pin_61)
- net F61: now also R3.2, R4.1
- net +1V8 renamed VCC
- net VCC: now also R3.1, R5.1
Other:
- note added: "Feature detect pins?"
- note added: "Pulldown when cart not connected"
- note removed: "Pulldown if unconnected?"
