File: pcb/reverse-singlerom/reverse-singlerom.kicad_sch (KiCad schematic)
At the start: 14 parts

Commit message: Adds some comments
Parts:
- C2, C3: value C -> 100nF
- C4: value C -> 120nF
- R1: value R -> 100K
- R2: value R -> 1.2K
- R3, R4, R5, R6: value R -> 1K
Other:
- note added: "Always use WORD mode BYTE always high"
- note added: "CS1/Pin 9 could be always low since CS2 controls power state"
- note added: "Power down SRAM when CS2 low Cart connected, pin 36 always HIGH = power on Cart disconnected, pulled LOW = power off"
- note added: "Shared OE indicates maskrom is OE HIGH OE high = maskrom read OE low = SRAM read/write Or, possibly maskrom CE could be used"
- note removed: "Pulldown when cart not connected"
- moved on the sheet: C2, C3, IC2, R1
