File: pcb/reverse-singlerom/reverse-singlerom.kicad_sch (KiCad schematic)
At the start: 14 parts

Commit message: Update notes, pass ERC, pass DRC
Other:
- note added: "* Hardwired to use WORD mode"
- note added: "CS1 LOW OR CS2 HIGH powers down RAM, data bus to high-impedance Note both connected"
- note added: "Note OE, address, data bus all shared between RAM/ROM"
- note added: "Pulldown powers down SRAM when cart disconnected"
- note added: "Used for SND RESET on WanWan... others?"
- note removed: "Always use WORD mode BYTE always high"
- note removed: "CS1/Pin 9 could be always low since CS2 controls power state"
- note removed: "Power down SRAM when CS2 low Cart connected, pin 36 always HIGH = power on Cart disconnected, pulled LOW = power off"
- note removed: "Shared OE indicates maskrom is OE HIGH OE high = maskrom read OE low = SRAM read/write Or, possibly maskrom CE could be used"
- moved on the sheet: C2, C4

Commit message: Add header pin breakout for SOP44 maskrom
Other:
- added sheet Maskrom Breakout (maskrom_breakout.kicad_sch)
- note added: "Simple option to build on for real dumper"
Changed lines of the file:
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@@
+    (effects (font (size 1.27 1.27)) (justify left bottom))
+  )
+  (text "Simple option to build on for real dumper" (at 118.11 186.69 0)
     (effects (font (size 1.27 1.27)) (justify left bottom))
   )
@@
       )
     )
+  )
+  (sheet (at 116.84 180.34) (size 52.07 11.43) (fields_autoplaced)
+    (stroke (width 0.1524) (type solid))
+    (fill (color 0 0 0 0.0000))
+    (property "Sheetname" "Maskrom Breakout" (at 116.84 179.6284 0) (show_name)
+      (effects (font (size 1.27 1.27)) (justify left bottom))
+    )
+    (property "Sheetfile" "maskrom_breakout.kicad_sch" (at 116.84 192.3546 0)
+      (effects (font (size 1.27 1.27)) (justify left top))
+    )
+    (instances
+      (project "reverse-singlerom"
+        (path "/5081f4fb-0c92-4cfc-8c52-39777c6d96ed" (page "2"))
+      )
+    )

Commit message: Schematic update better matching sram mapping
Connections:
- net RAMA0: now reaches IC2.10 (A0), J1.33 (RAMA0)
Changed lines of the file:
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@@
+    (effects (font (size 1.27 1.27)) (justify right bottom))
+  )
+  (label "RAMA0" (at 97.79 92.71 180) (fields_autoplaced)
     (effects (font (size 1.27 1.27)) (justify right bottom))
   )

Commit message: Remove maskrom breakout
Other:
- removed sheet Maskrom Breakout
- note removed: "Simple option to build on for real dumper"
Changed lines of the file:
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@@
-    (effects (font (size 1.27 1.27)) (justify left bottom))
-  )
-  (text "Simple option to build on for real dumper" (at 118.11 186.69 0)
     (effects (font (size 1.27 1.27)) (justify left bottom))
   )
@@
       )
     )
-  )
-  (sheet (at 116.84 180.34) (size 52.07 11.43) (fields_autoplaced)
-    (stroke (width 0.1524) (type solid))
-    (fill (color 0 0 0 0.0000))
-    (property "Sheetname" "Maskrom Breakout" (at 116.84 179.6284 0) (show_name)
-      (effects (font (size 1.27 1.27)) (justify left bottom))
-    )
-    (property "Sheetfile" "maskrom_breakout.kicad_sch" (at 116.84 192.3546 0)
-      (effects (font (size 1.27 1.27)) (justify left top))
-    )
-    (instances
-      (project "reverse-singlerom"
-        (path "/5081f4fb-0c92-4cfc-8c52-39777c6d96ed" (page "2"))
-      )
-    )
