File: pcb/singlerom-dev/singlerom-dev.kicad_sch (KiCad schematic)
At the start: 28 parts, among them J2 Back pin breakouts, J3 Front pin breakouts, J4 PWR Breakout, U2 MX29LV320EBTI-70G

Commit message: tweaks
Parts:
- removed J2: Back pin breakouts, Connector_PinHeader_2.54mm:PinHeader_1x21_P2.54mm_Vertical, symbol Connector:Conn_01x21_Socket
- removed J3: Front pin breakouts, Connector_PinHeader_2.54mm:PinHeader_1x24_P2.54mm_Vertical, symbol Connector:Conn_01x24_Socket

Commit message: Adds Pi Pico header + IO expander for on-board programming, starting over with manual routing
Parts:
- added C3: C_Small, Capacitor_SMD:C_0805_2012Metric_Pad1.18x1.45mm_HandSolder, symbol Device:C_Small
- added U3: MCP23S17-E/SS, LOOPY_IO:DIP787W46P254L3467H508Q28, symbol LOOPY_IO:MCP23S17-E/SS
- added U4: Pi Pico, LOOPY_PI:Pi Pico, symbol LOOPY_IO:Pi_Pico
- C1, C2: footprint Capacitor_SMD:C_1206_3216Metric_Pad1.33x1.80mm_HandSolder -> Capacitor_SMD:C_0805_2012Metric_Pad1.18x1.45mm_HandSolder
Connections:
- net A0: now also U4.6 (4)
- net A1: now also U4.7 (5)
- net A10: now also U4.19 (14)
- net A11: now also U4.20 (15)
- net A12: now also U4.21 (16)
- net A13: now also U4.22 (17)
- net A14: now also U4.24 (18)
- net A15: now also U4.25 (19)
- net A16: now also U4.26 (20)
- net A17: now also U4.27 (21)
- net A18: now also U4.29 (22)
- net A19: now also U4.37 (23)
- net A2: now also U4.9 (6)
- net A20: now also U4.31 (26)
- net A3: now also U4.10 (7)
- net A4: now also U4.11 (8)
- net A5: now also U4.12 (9)
- net A6: now also U4.14 (10)
- net A7: now also U4.15 (11)
- net A8: now also U4.16 (12)
- net A9: now also U4.17 (13)
- net D0: now also U3.21 (GPA0)
- net D1: now also U3.22 (GPA1)
- net D10: now also U3.3 (GPB2)
- net D11: now also U3.4 (GPB3)
- net D12: now also U3.5 (GPB4)
- net D13: now also U3.6 (GPB5)
- net D14: now also U3.7 (GPB6)
- net D15: now also U3.8 (GPB7)
- net D2: now also U3.23 (GPA2)
- net D3: now also U3.24 (GPA3)
- net D4: now also U3.25 (GPA4)
- net D5: now also U3.26 (GPA5)
- net D6: now also U3.27 (GPA6)
- net D7: now also U3.28 (GPA7)
- net D8: now also U3.1 (GPB0)
- net D9: now also U3.2 (GPB1)
- net GND: now also C3.1, U3.9 (VDD), U4.13 (GND), U4.18 (GND), U4.23 (GND), U4.28 (GND), U4.3 (GND), U4.33 (GND), U4.38 (GND), U4.8 (GND)
- net OE: now also U4.34 (28)
- net ROMCE: now also U4.35 (29)
- net VCC: now also C3.2, U3.10 (VSS), U3.18 (~{RESET}), U4.36 (3V3); no longer JP8.1 (A)
- new net ROMWE: JP8.1 (A), U4.32 (27)
- new net SPI_CLK: U3.12 (SCK), U4.4 (2)
- new net SPI_CS: U3.11 (~{CS}), U4.2 (1)
- new net SPI_MISO: U3.14 (SO), U4.1 (0)
- new net SPI_MOSI: U3.13 (SI), U4.5 (3)
- no-connect marks 0 -> 8
Other:
- note added: "Power from USB only"
- note added: "Provide 3V power to board when plugged into USB"
- moved on the sheet: J1, J4

Commit message: WIP rerouting devcart
Connections:
- net GND: no longer U4.13 (GND), U4.18 (GND), U4.23 (GND), U4.28 (GND), U4.3 (GND), U4.33 (GND), U4.38 (GND), U4.8 (GND)
- no-connect marks 8 -> 16
Changed lines of the file:
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@@
   (junction (at 80.01 158.75) (diameter 0) (color 0 0 0 0)
-  )
-  (junction (at 236.22 59.69) (diameter 0) (color 0 0 0 0)
   )
   (junction (at 152.4 163.83) (diameter 0) (color 0 0 0 0)
@@
   (junction (at 161.29 163.83) (diameter 0) (color 0 0 0 0)
   )
-  (junction (at 236.22 46.99) (diameter 0) (color 0 0 0 0)
-  )
   (junction (at 248.92 218.44) (diameter 0) (color 0 0 0 0)
-  )
-  (junction (at 274.32 46.99) (diameter 0) (color 0 0 0 0)
-  )
-  (junction (at 274.32 72.39) (diameter 0) (color 0 0 0 0)
   )
   (junction (at 224.79 78.74) (diameter 0) (color 0 0 0 0)
   )
-  (junction (at 274.32 59.69) (diameter 0) (color 0 0 0 0)
-  )
-  (junction (at 236.22 72.39) (diameter 0) (color 0 0 0 0)
-  )
   (no_connect (at 262.89 31.75))
+  (no_connect (at 245.11 72.39))
+  (no_connect (at 245.11 59.69))
   (no_connect (at 262.89 54.61))
+  (no_connect (at 245.11 46.99))
   (no_connect (at 185.42 35.56))
+  (no_connect (at 262.89 46.99))
   (no_connect (at 185.42 30.48))
+  (no_connect (at 262.89 72.39))
   (no_connect (at 220.98 30.48))
+  (no_connect (at 262.89 34.29))
   (no_connect (at 262.89 29.21))
+  (no_connect (at 262.89 59.69))
+  (no_connect (at 245.11 34.29))
   (no_connect (at 220.98 33.02))
   (no_connect (at 185.42 33.02))
   (wire (pts (xy 214.63 220.98) (xy 219.71 220.98))
-    (stroke (width 0) (type default))
-  )
-  (wire (pts (xy 236.22 59.69) (xy 236.22 72.39))
     (stroke (width 0) (type default))
   )
@@
     (stroke (width 0) (type default))
   )
-  (wire (pts (xy 245.11 34.29) (xy 236.22 34.29))
-    (stroke (width 0) (type default))
-  )
   (wire (pts (xy 210.82 134.62) (xy 219.71 134.62))
     (stroke (width 0) (type default))
@@
     (stroke (width 0) (type default))
   )
-  (wire (pts (xy 274.32 59.69) (xy 274.32 72.39))
-    (stroke (width 0) (type default))
-  )
   (wire (pts (xy 242.57 195.58) (xy 250.19 195.58))
     (stroke (width 0) (type default))
@@
   )
   (wire (pts (xy 167.64 158.75) (xy 167.64 163.83))
-    (stroke (width 0) (type default))
-  )
-  (wire (pts (xy 236.22 34.29) (xy 236.22 46.99))
-    (stroke (width 0) (type default))
-  )
-  (wire (pts (xy 236.22 46.99) (xy 245.11 46.99))
-    (stroke (width 0) (type default))
-  )
-  (wire (pts (xy 262.89 59.69) (xy 274.32 59.69))
     (stroke (width 0) (type default))
   )
@@
     (stroke (width 0) (type default))
   )
-  (wire (pts (xy 274.32 34.29) (xy 274.32 46.99))
-    (stroke (width 0) (type default))
-  )
-  (wire (pts (xy 245.11 59.69) (xy 236.22 59.69))
-    (stroke (width 0) (type default))
-  )
-  (wire (pts (xy 262.89 34.29) (xy 274.32 34.29))
-    (stroke (width 0) (type default))
-  )
   (wire (pts (xy 242.57 111.76) (xy 247.65 111.76))
-    (stroke (width 0) (type default))
-  )
-  (wire (pts (xy 236.22 46.99) (xy 236.22 59.69))
-    (stroke (width 0) (type default))
-  )
-  (wire (pts (xy 262.89 72.39) (xy 274.32 72.39))
     (stroke (width 0) (type default))
   )
@@
     (stroke (width 0) (type default))
   )
-  (wire (pts (xy 262.89 46.99) (xy 274.32 46.99))
-    (stroke (width 0) (type default))
-  )
   (wire (pts (xy 161.29 163.83) (xy 167.64 163.83))
-    (stroke (width 0) (type default))
-  )
-  (wire (pts (xy 236.22 72.39) (xy 245.11 72.39))
-    (stroke (width 0) (type default))
-  )
-  (wire (pts (xy 274.32 72.39) (xy 274.32 86.36))
     (stroke (width 0) (type default))
   )
@@
     (stroke (width 0) (type default))
   )
-  (wire (pts (xy 236.22 72.39) (xy 236.22 86.36))
+  (wire (pts (xy 236.22 34.29) (xy 236.22 86.36))
     (stroke (width 0) (type default))
   )
@@
     (stroke (width 0) (type default))
   )
-  (wire (pts (xy 274.32 46.99) (xy 274.32 59.69))
+  (wire (pts (xy 274.32 34.29) (xy 274.32 86.36))
     (stroke (width 0) (type default))
   )

Commit message: Correcting wrong flash IC, footprint, symbol. Still needs rerouting but removed incorrect one.
Parts:
- removed U2: MX29LV320EBTI-70G, LOOPY_Flash_Macronix:MX29LV320EBTI-70G, symbol LOOPY_Flash_Macronix:MX29LV320EBTI-70G
- added U2: MX29LV160DBTI-70G, LOOPY_Flash:SOP50P2000X120-48N, symbol LOOPY_Flash:MX29LV160DBTI-70G
Other:
- note added: "TODO FIX"
Changed lines of the file:
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@@
   (junction (at 80.01 158.75) (diameter 0) (color 0 0 0 0)
-  )
-  (junction (at 152.4 163.83) (diameter 0) (color 0 0 0 0)
   )
   (junction (at 137.16 54.61) (diameter 0) (color 0 0 0 0)
@@
     (stroke (width 0) (type default))
     (fill (type none))
+  )
+  (text "TODO FIX" (at 96.52 91.44 0)
+    (effects (font (size 1.27 1.27)) (justify left bottom))
   )
   (text "Power from USB only" (at 266.7 29.21 0)
@@
     )
   )
-  (symbol (lib_id "Connector:TestPoint") (at 250.19 195.58 270) (unit 1)
-    (in_bom yes) (on_board yes) (dnp no) (fields_autoplaced)
-    (property "Reference" "TP3" (at 255.27 194.945 90)
-      (effects (font (size 1.27 1.27)) (justify left) hide)
-    )
-    (property "Value" "OE" (at 255.27 197.485 90)
-      (effects (font (size 1.27 1.27)) (justify left) hide)
-    )
-    (property "Footprint" "TestPoint:TestPoint_Pad_D1.0mm" (at 250.19 200.66 0)
-      (effects (font (size 1.27 1.27)) hide)
-    )
-    (property "Datasheet" "~" (at 250.19 200.66 0)
-      (effects (font (size 1.27 1.27)) hide)
-    )
-    (property "Notes" "" (at 250.19 195.58 0)
+  (symbol (lib_id "LOOPY_Flash:MX29LV160DBTI-70G") (at 109.22 92.71 0) (unit 1)
+    (in_bom yes) (on_board yes) (dnp no) (fields_autoplaced)
+    (property "Reference" "U2" (at 127 86.36 0)
       (effects (font (size 1.27 1.27)))
     )
-    (pin "1")
-    (instances
-      (project "singlerom-dev"
-        (path "/5081f4fb-0c92-4cfc-8c52-39777c6d96ed"
-          (reference "TP3") (unit 1)
-        )
-      )
-    )
-  )
-  (symbol (lib_id "power:GND") (at 214.63 220.98 0) (unit 1)
-    (in_bom yes) (on_board yes) (dnp no) (fields_autoplaced)
-    (property "Reference" "#PWR01" (at 214.63 227.33 0)
-      (effects (font (size 1.27 1.27)) hide)
-    )
-    (property "Value" "GND" (at 214.63 226.06 0)
+    (property "Value" "MX29LV160DBTI-70G" (at 127 88.9 0)
       (effects (font (size 1.27 1.27)))
     )
-    (property "Footprint" "" (at 214.63 220.98 0)
-      (effects (font (size 1.27 1.27)) hide)
-    )
-    (property "Datasheet" "" (at 214.63 220.98 0)
-      (effects (font (size 1.27 1.27)) hide)
-    )
-    (pin "1")
-    (instances
-      (project "singlerom-dev"
-        (path "/5081f4fb-0c92-4cfc-8c52-39777c6d96ed"
-          (reference "#PWR01") (unit 1)
-        )
-      )
-    )
-  )
-  (symbol (lib_id "LOOPY_Flash_Macronix:MX29LV320EBTI-70G") (at 101.6 95.25 0) (unit 1)
-    (in_bom yes) (on_board yes) (dnp no) (fields_autoplaced)
-    (property "Reference" "U2" (at 127 83.82 0)
-      (effects (font (size 1.524 1.524)))
-    )
-    (property "Value" "MX29LV320EBTI-70G" (at 127 86.36 0)
-      (effects (font (size 1.524 1.524)))
-    )
-    (property "Footprint" "LOOPY_Flash_Macronix:MX29LV320EBTI-70G" (at 127 86.614 0)
-      (effects (font (size 1.524 1.524)) hide)
-    )
-    (property "Datasheet" "https://media.digikey.com/pdf/Data%20Sheets/Macronix/MX29LV160D(T,B).pdf" (at 101.6 95.25 0)
-      (effects (font (size 1.524 1.524)) hide)
-    )
-    (property "Notes" "" (at 101.6 95.25 0)
-      (effects (font (size 1.27 1.27)))
-    )
-    (pin "1")
-    (pin "10")
+    (property "Footprint" "LOOPY_Flash:SOP50P2000X120-48N" (at 140.97 187.63 0)
+      (effects (font (size 1.27 1.27)) (justify left top) hide)
+    )
+    (property "Datasheet" "http://uk.rs-online.com/web/p/products/9142816" (at 140.97 287.63 0)
+      (effects (font (size 1.27 1.27)) (justify left top) hide)
+    )
+    (property "Height" "1.2" (at 140.97 487.63 0)
+      (effects (font (size 1.27 1.27)) (justify left top) hide)
+    )
+    (property "Manufacturer_Name" "Macronix" (at 140.97 587.63 0)
+      (effects (font (size 1.27 1.27)) (justify left top) hide)
+    )
+    (property "Manufacturer_Part_Number" "MX29LV160DBTI-70G" (at 140.97 687.63 0)
+      (effects (font (size 1.27 1.27)) (justify left top) hide)
+    )
+    (property "Mouser Part Number" "" (at 140.97 787.63 0)
+      (effects (font (size 1.27 1.27)) (justify left top) hide)
+    )
+    (property "Mouser Price/Stock" "" (at 140.97 887.63 0)
+      (effects (font (size 1.27 1.27)) (justify left top) hide)
+    )
+    (property "Arrow Part Number" "MX29LV160DBTI-70G" (at 140.97 987.63 0)
+      (effects (font (size 1.27 1.27)) (justify left top) hide)
+    )
+    (property "Arrow Price/Stock" "https://www.arrow.com/en/products/mx29lv160dbti-70g/macronix-international?region=nac" (at 140.97 1087.63 0)
+      (effects (font (size 1.27 1.27)) (justify left top) hide)
+    )
+    (pin "1")
     (pin "10")
     (pin "11")
@@
     (pin "8")
     (pin "9")
-    (pin "13")
-    (pin "27")
-    (pin "37")
-    (pin "46")
     (instances
       (project "singlerom-dev"
@@
         )
       )
+    )
+  )
+  (symbol (lib_id "Connector:TestPoint") (at 250.19 195.58 270) (unit 1)
+    (in_bom yes) (on_board yes) (dnp no) (fields_autoplaced)
+    (property "Reference" "TP3" (at 255.27 194.945 90)
+      (effects (font (size 1.27 1.27)) (justify left) hide)
+    )
+    (property "Value" "OE" (at 255.27 197.485 90)
+      (effects (font (size 1.27 1.27)) (justify left) hide)
+    )
+    (property "Footprint" "TestPoint:TestPoint_Pad_D1.0mm" (at 250.19 200.66 0)
+      (effects (font (size 1.27 1.27)) hide)
+    )
+    (property "Datasheet" "~" (at 250.19 200.66 0)
+      (effects (font (size 1.27 1.27)) hide)
+    )
+    (property "Notes" "" (at 250.19 195.58 0)
+      (effects (font (size 1.27 1.27)))
+    )
+    (pin "1")
+    (instances
+      (project "singlerom-dev"
+        (path "/5081f4fb-0c92-4cfc-8c52-39777c6d96ed"
+          (reference "TP3") (unit 1)
+        )
+      )
+    )
+  )
+  (symbol (lib_id "power:GND") (at 214.63 220.98 0) (unit 1)
+    (in_bom yes) (on_board yes) (dnp no) (fields_autoplaced)
+    (property "Reference" "#PWR01" (at 214.63 227.33 0)
+      (effects (font (size 1.27 1.27)) hide)
+    )
+    (property "Value" "GND" (at 214.63 226.06 0)
+      (effects (font (size 1.27 1.27)))
+    )
+    (property "Footprint" "" (at 214.63 220.98 0)
+      (effects (font (size 1.27 1.27)) hide)
+    )
+    (property "Datasheet" "" (at 214.63 220.98 0)
+      (effects (font (size 1.27 1.27)) hide)
+    )
+    (pin "1")
+    (instances
+      (project "singlerom-dev"
+        (path "/5081f4fb-0c92-4cfc-8c52-39777c6d96ed"
+          (reference "#PWR01") (unit 1)
+        )
+      )

Commit message: Fix schematic with 16mbit
Parts:
- removed TP2: RY, TestPoint:TestPoint_Pad_D1.0mm, symbol Connector:TestPoint
- added R1: 10K, symbol Device:R_Small
Connections:
- net A0: now also U2.25 (A0)
- net A1: now also U2.24 (A1)
- net A10: now also U2.6 (A10)
- net A11: now also U2.5 (A11)
- net A12: now also U2.4 (A12)
- net A13: now also U2.3 (A13)
- net A14: now also U2.2 (A14)
- net A15: now also U2.1 (A15)
- net A16: now also U2.48 (A16)
- net A17: now also U2.17 (A17)
- net A18: now also U2.16 (A18)
- net A19: now also U2.9 (A19)
- net A2: now also U2.23 (A2)
- net A3: now also U2.22 (A3)
- net A4: now also U2.21 (A4)
- net A5: now also U2.20 (A5)
- net A6: now also U2.19 (A6)
- net A7: now also U2.18 (A7)
- net A8: now also U2.8 (A8)
- net A9: now also U2.7 (A9)
- net D0: now also U2.29 (Q0)
- net D1: now also U2.31 (Q1)
- net D10: now also U2.34 (Q10)
- net D11: now also U2.36 (Q11)
- net D12: now also U2.39 (Q12)
- net D13: now also U2.41 (Q13)
- net D14: now also U2.43 (Q14)
- net D15: now also U2.45 (Q15/A-1)
- net D2: now also U2.33 (Q2)
- net D3: now also U2.35 (Q3)
- net D4: now also U2.38 (Q4)
- net D5: now also U2.40 (Q5)
- net D6: now also U2.42 (Q6)
- net D7: now also U2.44 (Q7)
- net D8: now also U2.30 (Q8)
- net D9: now also U2.32 (Q9)
- net GND: now also U2.27 (GND_1), U2.46 (GND_2), U2.47 (BYTE#), U4.38 (GND); no longer U3.9 (VDD)
- net VCC: now also U2.37 (VCC), R1.1
- net at JP8.2 (B): now also U2.11 (WE#)
- net PICO_GND: now reaches U4.3 (GND)
- net PICO_GND: now also U3.9 (VDD)
- net at JP5.2 (B): now also U2.26 (CE#)
- net at U2.12 (RESET#): now also JP4.2 (B)
- net at U2.14 (WP#/ACC): now also JP7.2 (B)
- net at U2.15 (RY/BY#): now also TP1.1
- net at U2.28 (OE#): now also JP6.2 (B)
- net A20: no longer names the net of U4.31 (26)
- net ROMWE renamed PICO_ROMWE
- net PICO_ROMWE: now also R1.2
- no-connect marks 16 -> 17
Other:
- note added: "Pico acts as a switch providing a path from VCC to GND So IO expand only gets power when pico inserted?"
- note removed: "TODO FIX"
- moved on the sheet: C1

Commit message: Schematic update better matching sram mapping
Connections:
- net A10: now also U1.4 (A6); no longer U1.23 (A11)
- net A11: now also U1.5 (A5); no longer U1.2 (A12)
- net A3: now also U1.21 (A10); no longer U1.6 (A4)
- net A4: now also U1.6 (A4); no longer U1.5 (A5)
- net A5: now also U1.23 (A11); no longer U1.4 (A6)
- net A6: now also U1.24 (A9); no longer U1.3 (A7)
- net A8: now also U1.2 (A12); no longer U1.24 (A9)
- net A9: now also U1.3 (A7); no longer U1.21 (A10)
- net D0: now also U1.18 (DQ6); no longer U1.11 (DQ0)
- net D1: now also U1.17 (DQ5); no longer U1.12 (DQ1)
- net D2: now also U1.16 (DQ4); no longer U1.13 (DQ2)
- net D4: now also U1.13 (DQ2); no longer U1.16 (DQ4)
- net D5: now also U1.12 (DQ1); no longer U1.17 (DQ5)
- net D6: now also U1.11 (DQ0); no longer U1.18 (DQ6)
- net RAMCS1: now also U4.31 (26)
- no-connect marks 17 -> 16
Other:
- note added: "/CE works same"
- note added: "/OE active low observed"
- note added: "Address and data pins SHOULD be able to be rearranged arbitrarily Replicated mapping from reversed cart out of paranoia"
- note added: "FRAM"
- note added: "Flash"
- note added: "MaskROM: We should behave the same as this"
- note added: "SRAM: We should behave the same as this"
- note added: "Using CS1 and not using CS2, hopefully Loopy drives both"
- note removed: "Address and data pins can be rearranged arbitrarily"
- moved on the sheet: R1

Commit message: Forget FRAM for now, redesign around pin compatible SRAM, nuke old routes
Parts:
- removed C2: C, Capacitor_SMD:C_0805_2012Metric_Pad1.18x1.45mm_HandSolder, symbol Device:C
- removed JP1: CE, Jumper:SolderJumper-2_P1.3mm_Open_RoundedPad1.0x1.5mm, symbol Jumper:Jumper_2_Bridged
- removed JP2: OE, Jumper:SolderJumper-2_P1.3mm_Open_RoundedPad1.0x1.5mm, symbol Jumper:Jumper_2_Bridged
- removed JP3: WE, Jumper:SolderJumper-2_P1.3mm_Open_RoundedPad1.0x1.5mm, symbol Jumper:Jumper_2_Bridged
- removed U1: ~, Package_SO:SOIC-28W_7.5x17.9mm_P1.27mm, symbol LOOPY_FRAM:FM16W08-SGTR
- added R6, R7: 100K, Resistor_SMD:R_0805_2012Metric_Pad1.20x1.40mm_HandSolder, symbol Device:R_Small
- added U1: AS6C6264-55SCN, LOOPY_SRAM:SOP-28_Customized, symbol LOOPY_SRAM:AS6C6264-55SCN
- R5: renamed from R1; value 10K -> 100K; footprint (none) -> Resistor_SMD:R_0805_2012Metric_Pad1.20x1.40mm_HandSolder
- renumbered C3 to C2, J4 to J2, JP8 to JP1, JP4 to JP2, JP7 to JP3, JP6 to JP4, R3 to R1, R5 to R2, R4 to R3, R6 to R4, TP8 to TP2, TP7 to TP3, TP6 to TP4, TP3 to TP6, TP4 to TP7
Connections:
- net A0: now also U1.9 (A1)
- net A1: now also U1.8 (A2)
- net A10: now also U1.4 (A6)
- net A11: now also U1.5 (A5)
- net A2: now also U1.7 (A3)
- net A3: now also U1.21 (A10)
- net A4: now also U1.6 (A4)
- net A5: now also U1.23 (A11)
- net A6: now also U1.24 (A9)
- net A7: now also U1.25 (A8)
- net A8: now also U1.2 (A12)
- net A9: now also U1.3 (A7)
- net D0: now also U1.18 (DQ6)
- net D1: now also U1.17 (DQ5)
- net D2: now also U1.16 (DQ4)
- net D3: now also U1.15 (DQ3)
- net D4: now also U1.13 (DQ2)
- net D5: now also U1.12 (DQ1)
- net D6: now also U1.11 (DQ0)
- net D7: now also U1.19 (DQ7)
- net GND: now also R6.2, U1.14 (VSS)
- net OE: now also U1.22 (*OE)
- net RAMA0: now also U1.10 (A0)
- net RAMCS1: now also U1.20 (*CE)
- net RAMCS2: now also R6.1, U1.26 (CE2)
- net RAMWE: now also U1.27 (*WE)
- net ROMCE: now also R7.2
- net VCC: now also R7.1, U1.28 (VCC)
Other:
- note added: "AS6C6264-55SIN, modern available replacement for HM9264B, should be interchangeable"
- note added: "RAMCS2 low when disconnected, standby mode"
- note added: "When ROMCE disconnected (no cart) pull CE high for standby"
- note removed: "Address and data pins SHOULD be able to be rearranged arbitrarily Replicated mapping from reversed cart out of paranoia"
- note removed: "FRAM"
- note removed: "SRAM: We should behave the same as this"
- note removed: "Using CS1 and not using CS2, hopefully Loopy drives both"
- moved on the sheet: R5

Commit message: Routing
Parts:
- removed JP5: CE, Jumper:SolderJumper-2_P1.3mm_Open_RoundedPad1.0x1.5mm, symbol Jumper:Jumper_2_Bridged
- removed R3, R4: 1K, Resistor_SMD:R_0805_2012Metric_Pad1.20x1.40mm_HandSolder, symbol Device:R
- added C1: C, Capacitor_SMD:C_0805_2012Metric_Pad1.18x1.45mm_HandSolder, symbol Device:C
- renumbered C1 to C2, C2 to C3, R5 to R3, R6 to R4, R7 to R5
Connections:
- net GND: now also C1.2
- net ROMCE: now also U2.26 (CE#)
- net VCC: now also C1.1
Other:
- moved on the sheet: R4
