File: pcb/singlerom-dev/singlerom-dev.kicad_sch (KiCad schematic)
At the start: 25 parts, among them J2 PWR Breakout, U1 AS6C6264-55SCN, U2 MX29LV160DBTI-70G, U3 MCP23S17-E/SS, U4 Pi Pico

Commit message: Replicate power path controller for SRAM from original
Parts:
- removed U3: MCP23S17-E/SS, LOOPY_IO:DIP787W46P254L3467H508Q28, symbol LOOPY_IO:MCP23S17-E/SS
- added BT1: CR2032, LOOPY_Cart:Keystone-3034TR-MFG, symbol Device:Battery_Cell
- added D1: AZ23C3V6, Package_TO_SOT_SMD:SOT-23, symbol Diode:MMBZxx
- added R6: 1.2K, Resistor_SMD:R_0805_2012Metric_Pad1.20x1.40mm_HandSolder, symbol Device:R_Small
- added U5: TCA9539PWR, Package_SO:TSSOP-24_4.4x7.8mm_P0.65mm, symbol LOOPY_IO:TCA9539PWR
- JP1: value WE -> ~{WE}
- JP3: value RST -> ~{RESET}
- JP4: value OE -> ~{OE}
- TP1: value WP -> ~{RY/BY}
Connections:
- net D0: now also U5.4 (P00)
- net D1: now also U5.5 (P01)
- net D10: now also U5.15 (P12)
- net D11: now also U5.16 (P13)
- net D12: now also U5.17 (P14)
- net D13: now also U5.18 (P15)
- net D14: now also U5.19 (P16)
- net D15: now also U5.20 (P17)
- net D2: now also U5.6 (P02)
- net D3: now also U5.7 (P03)
- net D4: now also U5.8 (P04)
- net D5: now also U5.9 (P05)
- net D6: now also U5.10 (P06)
- net D7: now also U5.11 (P07)
- net D8: now also U5.13 (P10)
- net D9: now also U5.14 (P11)
- net GND: now also C1.1, BT1.2 (-); no longer C1.2, C3.1
- net PICO_GND: now also C3.1, U5.12 (GND), U5.2 (A1), U5.21 (A0)
- net VCC: now also D1.2 (K), U5.24 (VCC); no longer C1.1, U1.28 (VCC)
- net SPI_CLK renamed I2C_RESET
- net I2C_RESET: now also U5.3 (~{RESET})
- net SPI_CS renamed I2C_SCL
- net I2C_SCL: now also U5.22 (SCL)
- net SPI_MISO renamed I2C_SDA
- net I2C_SDA: now also U5.23 (SDA)
- net SPI_MOSI: no longer names the net of U4.5 (3)
- new net: D1.1 (K), R6.2
- new net: C1.2, D1.3 (A), U1.28 (VCC)
- new net +BATT: BT1.1 (+), R6.1
- no-connect marks 16 -> 13
Other:
- note added: "CART EDGE"
- note added: "PROGRAM"
- note added: "RAM"
- note added: "ROM"
- note added: "When Pico disconnected WE pulled high to write protect"
- moved on the sheet: C1, C3, R1, R2, R4

Commit message: Nudging clearances
Parts:
- C1: value C -> 1u
- C2: value C -> 0.1u
- C3: value C_Small -> 0.1u
Connections:
- net GND: now also R4.1; no longer R4.2
- net RAMCS2: now also R4.2; no longer R4.1
Other:
- note added: "RAMCS2 low when disconnected standby mode"
- note added: "Select power source, prevent battery charging"
- note removed: "RAMCS2 low when disconnected, standby mode"
Changed lines of the file:
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@@
   (junction (at 168.91 148.59) (diameter 0) (color 0 0 0 0)
   )
+  (junction (at 135.89 48.26) (diameter 0) (color 0 0 0 0)
+  )
   (junction (at 204.47 25.4) (diameter 0) (color 0 0 0 0)
   )
@@
     (stroke (width 0) (type default))
   )
-  (wire (pts (xy 133.35 48.26) (xy 111.76 48.26))
-    (stroke (width 0) (type default))
-  )
   (wire (pts (xy 229.87 34.29) (xy 245.11 34.29))
     (stroke (width 0) (type default))
@@
     (stroke (width 0) (type default))
   )
-  (wire (pts (xy 143.51 48.26) (xy 138.43 48.26))
-    (stroke (width 0) (type default))
-  )
   (wire (pts (xy 242.57 200.66) (xy 250.19 200.66))
     (stroke (width 0) (type default))
@@
     (stroke (width 0) (type default))
   )
+  (wire (pts (xy 135.89 55.88) (xy 135.89 58.42))
+    (stroke (width 0) (type default))
+  )
   (wire (pts (xy 210.82 134.62) (xy 219.71 134.62))
     (stroke (width 0) (type default))
@@
     (stroke (width 0) (type default))
   )
+  (wire (pts (xy 135.89 48.26) (xy 143.51 48.26))
+    (stroke (width 0) (type default))
+  )
+  (wire (pts (xy 111.76 48.26) (xy 135.89 48.26))
+    (stroke (width 0) (type default))
+  )
   (wire (pts (xy 153.67 120.65) (xy 160.02 120.65))
     (stroke (width 0) (type default))
   )
+  (wire (pts (xy 135.89 48.26) (xy 135.89 50.8))
+    (stroke (width 0) (type default))
+  )
   (wire (pts (xy 105.41 128.27) (xy 109.22 128.27))
     (stroke (width 0) (type default))
@@
     )
   )
-  (text "RAMCS2 low when disconnected, standby mode" (at 125.73 58.42 0)
+  (text "RAMCS2 low when disconnected\nstandby mode" (at 140.97 58.42 0)
     (effects (font (size 1.27 1.27)) (justify left bottom))
   )
+  (text "Select power source, prevent battery charging" (at 148.59 20.32 0)
+    (effects (font (size 1.27 1.27)) (justify right bottom))
+  )
   (text "Pico acts as a switch providing a path from VCC to GND\nSo IO expand only gets power when pico inserted?"
     (at 220.98 20.32 0)
@@
     (effects (font (size 1.27 1.27)) (justify right bottom))
   )
-  (label "RAMCS2" (at 111.76 48.26 0) (fields_autoplaced)
+  (label "RAMCS2" (at 143.51 48.26 0) (fields_autoplaced)
     (effects (font (size 1.27 1.27)) (justify left bottom))
   )
@@
       (effects (font (size 1.27 1.27)) (justify left))
     )
-    (property "Value" "C" (at 157.48 126.365 0)
+    (property "Value" "0.1u" (at 157.48 126.365 0)
       (effects (font (size 1.27 1.27)) (justify left))
     )
@@
     )
   )
+  (symbol (lib_id "Device:R_Small") (at 135.89 53.34 180) (unit 1)
+    (in_bom yes) (on_board yes) (dnp no)
+    (property "Reference" "R4" (at 133.35 53.34 90)
+      (effects (font (size 1.27 1.27)))
+    )
+    (property "Value" "100K" (at 138.43 53.34 90)
+      (effects (font (size 1.27 1.27)))
+    )
+    (property "Footprint" "Resistor_SMD:R_0805_2012Metric_Pad1.20x1.40mm_HandSolder" (at 135.89 53.34 0)
+      (effects (font (size 1.27 1.27)) hide)
+    )
+    (property "Datasheet" "~" (at 135.89 53.34 0)
+      (effects (font (size 1.27 1.27)) hide)
+    )
+    (pin "1")
+    (pin "2")
+    (instances
+      (project "singlerom-dev"
+        (path "/5081f4fb-0c92-4cfc-8c52-39777c6d96ed"
+          (reference "R4") (unit 1)
+        )
+      )
+    )
+  )
   (symbol (lib_id "Device:R_Small") (at 115.57 27.94 90) (unit 1)
     (in_bom yes) (on_board yes) (dnp no) (fields_autoplaced)
@@
       (effects (font (size 1.27 1.27)))
     )
-    (property "Value" "C" (at 135.89 33.02 90)
+    (property "Value" "1u" (at 135.89 33.02 90)
       (effects (font (size 1.27 1.27)))
     )
@@
   (symbol (lib_id "Device:C_Small") (at 207.01 25.4 270) (unit 1)
     (in_bom yes) (on_board yes) (dnp no) (fields_autoplaced)
-    (property "Reference" "C3" (at 206.3686 22.86 0)
-      (effects (font (size 1.27 1.27)) (justify right))
+    (property "Reference" "C3" (at 207.0036 20.32 90)
+      (effects (font (size 1.27 1.27)))
     )
-    (property "Value" "C_Small" (at 208.9086 22.86 0)
-      (effects (font (size 1.27 1.27)) (justify right))
+    (property "Value" "0.1u" (at 207.0036 22.86 90)
+      (effects (font (size 1.27 1.27)))
     )
     (property "Footprint" "Capacitor_SMD:C_0805_2012Metric_Pad1.18x1.45mm_HandSolder" (at 207.01 25.4 0)
@@
     )
   )
-  (symbol (lib_id "Device:R_Small") (at 135.89 48.26 90) (unit 1)
-    (in_bom yes) (on_board yes) (dnp no)
-    (property "Reference" "R4" (at 135.89 45.72 90)
-      (effects (font (size 1.27 1.27)))
-    )
-    (property "Value" "100K" (at 135.89 50.8 90)
-      (effects (font (size 1.27 1.27)))
-    )
-    (property "Footprint" "Resistor_SMD:R_0805_2012Metric_Pad1.20x1.40mm_HandSolder" (at 135.89 48.26 0)
-      (effects (font (size 1.27 1.27)) hide)
-    )
-    (property "Datasheet" "~" (at 135.89 48.26 0)
-      (effects (font (size 1.27 1.27)) hide)
-    )
-    (pin "1")
-    (pin "2")
-    (instances
-      (project "singlerom-dev"
-        (path "/5081f4fb-0c92-4cfc-8c52-39777c6d96ed"
-          (reference "R4") (unit 1)
-        )
-      )
-    )
-  )
-  (symbol (lib_id "power:GND") (at 143.51 48.26 0) (unit 1)
+  (symbol (lib_id "power:GND") (at 135.89 58.42 0) (unit 1)
     (in_bom yes) (on_board yes) (dnp no) (fields_autoplaced)
-    (property "Reference" "#PWR05" (at 143.51 54.61 0)
+    (property "Reference" "#PWR05" (at 135.89 64.77 0)
       (effects (font (size 1.27 1.27)) hide)
     )
-    (property "Value" "GND" (at 143.51 53.34 0)
+    (property "Value" "GND" (at 135.89 63.5 0)
       (effects (font (size 1.27 1.27)))
     )
-    (property "Footprint" "" (at 143.51 48.26 0)
+    (property "Footprint" "" (at 135.89 58.42 0)
       (effects (font (size 1.27 1.27)) hide)
     )
-    (property "Datasheet" "" (at 143.51 48.26 0)
+    (property "Datasheet" "" (at 135.89 58.42 0)
       (effects (font (size 1.27 1.27)) hide)
     )

Commit message: Match pin numbers on battery so + faces up
Connections:
- net +BATT: now also BT1.2 (+); no longer BT1.1 (+)
- net GND: now also BT1.1 (-); no longer BT1.2 (-)
Other:
- moved on the sheet: BT1
Changed lines of the file:
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@@
     (stroke (width 0) (type default))
   )
+  (wire (pts (xy 46.99 49.53) (xy 40.64 49.53))
+    (stroke (width 0) (type default))
+  )
   (wire (pts (xy 229.87 34.29) (xy 245.11 34.29))
     (stroke (width 0) (type default))
@@
     (stroke (width 0) (type default))
   )
-  (wire (pts (xy 40.64 46.99) (xy 40.64 50.8))
+  (wire (pts (xy 46.99 49.53) (xy 46.99 50.8))
     (stroke (width 0) (type default))
   )
@@
     (stroke (width 0) (type default))
   )
-  (wire (pts (xy 40.64 64.77) (xy 40.64 58.42))
+  (wire (pts (xy 46.99 60.96) (xy 46.99 58.42))
     (stroke (width 0) (type default))
   )
@@
     (stroke (width 0) (type default))
   )
+  (wire (pts (xy 40.64 60.96) (xy 40.64 64.77))
+    (stroke (width 0) (type default))
+  )
   (wire (pts (xy 135.89 48.26) (xy 135.89 50.8))
     (stroke (width 0) (type default))
@@
     (stroke (width 0) (type default))
   )
+  (wire (pts (xy 40.64 49.53) (xy 40.64 46.99))
+    (stroke (width 0) (type default))
+  )
+  (wire (pts (xy 46.99 60.96) (xy 40.64 60.96))
+    (stroke (width 0) (type default))
+  )
   (wire (pts (xy 219.71 109.22) (xy 214.63 109.22))
     (stroke (width 0) (type default))
@@
     )
   )
-  (symbol (lib_id "Device:Battery_Cell") (at 40.64 55.88 0) (unit 1)
-    (in_bom yes) (on_board yes) (dnp no) (fields_autoplaced)
-    (property "Reference" "BT1" (at 44.45 53.213 0)
+  (symbol (lib_id "Device:Battery_Cell") (at 46.99 55.88 0) (unit 1)
+    (in_bom yes) (on_board yes) (dnp no)
+    (property "Reference" "BT1" (at 50.8 53.213 0)
       (effects (font (size 1.27 1.27)) (justify left))
     )
-    (property "Value" "CR2032" (at 44.45 55.753 0)
+    (property "Value" "CR2032" (at 50.8 55.753 0)
       (effects (font (size 1.27 1.27)) (justify left))
     )
-    (property "Footprint" "LOOPY_Cart:Keystone-3034TR-MFG" (at 40.64 54.356 90)
+    (property "Footprint" "LOOPY_Cart:Keystone-3034TR-MFG" (at 41.91 54.61 90)
       (effects (font (size 1.27 1.27)) hide)
     )
-    (property "Datasheet" "~" (at 40.64 54.356 90)
+    (property "Datasheet" "~" (at 46.99 54.356 90)
       (effects (font (size 1.27 1.27)) hide)
     )
-    (pin "1")
+    (property "Notes" "" (at 46.99 55.88 0)
+      (effects (font (size 1.27 1.27)))
+    )
     (pin "2")
+    (pin "1")
     (instances
       (project "singlerom-dev"

Commit message: WIP some fixes, not completed but didn't want to leave broken
Parts:
- JP1: value ~{WE} -> WE
- JP2: value BYTE -> RESET
- JP3: value ~{RESET} -> WP/ACC
- JP4: value ~{OE} -> OE
- TP1: value ~{RY/BY} -> RY/BY
Connections:
- net GND: no longer U2.47 (BYTE#)
- net VCC: now also U2.47 (BYTE#)
Changed lines of the file:
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@@
     (effects (font (size 1.27 1.27)) (justify left bottom))
   )
-  (label "GND" (at 144.78 95.25 0) (fields_autoplaced)
+  (label "VCC" (at 144.78 95.25 0) (fields_autoplaced)
     (effects (font (size 1.27 1.27)) (justify left bottom))
   )
@@
   )
   (symbol (lib_id "Jumper:Jumper_2_Bridged") (at 96.52 118.11 0) (unit 1)
-    (in_bom yes) (on_board yes) (dnp no) (fields_autoplaced)
+    (in_bom yes) (on_board yes) (dnp no)
     (property "Reference" "JP1" (at 96.52 113.03 0)
       (effects (font (size 1.27 1.27)) hide)
     )
-    (property "Value" "~{WE}" (at 96.52 115.57 0)
+    (property "Value" "WE" (at 96.52 118.11 0)
       (effects (font (size 1.27 1.27)))
     )
@@
   )
   (symbol (lib_id "Jumper:Jumper_2_Bridged") (at 156.21 143.51 0) (mirror y) (unit 1)
-    (in_bom yes) (on_board yes) (dnp no) (fields_autoplaced)
+    (in_bom yes) (on_board yes) (dnp no)
     (property "Reference" "JP4" (at 156.21 138.43 0)
       (effects (font (size 1.27 1.27)) hide)
     )
-    (property "Value" "~{OE}" (at 156.21 140.97 0)
+    (property "Value" "OE" (at 156.21 144.78 0)
       (effects (font (size 1.27 1.27)))
     )
@@
       (effects (font (size 1.27 1.27)))
     )
-    (pin "2")
-    (pin "1")
+    (pin "1")
+    (pin "2")
     (instances
       (project "singlerom-dev"
@@
   )
   (symbol (lib_id "Jumper:Jumper_2_Bridged") (at 96.52 120.65 0) (unit 1)
-    (in_bom yes) (on_board yes) (dnp no) (fields_autoplaced)
+    (in_bom yes) (on_board yes) (dnp no)
     (property "Reference" "JP2" (at 96.52 115.57 0)
       (effects (font (size 1.27 1.27)) hide)
     )
-    (property "Value" "BYTE" (at 96.52 118.11 0)
-      (effects (font (size 1.27 1.27)) hide)
+    (property "Value" "RESET" (at 96.52 121.92 0)
+      (effects (font (size 1.27 1.27)))
     )
     (property "Footprint" "Jumper:SolderJumper-2_P1.3mm_Open_RoundedPad1.0x1.5mm" (at 96.52 120.65 0)
@@
   )
   (symbol (lib_id "Jumper:Jumper_2_Bridged") (at 96.52 125.73 0) (unit 1)
-    (in_bom yes) (on_board yes) (dnp no) (fields_autoplaced)
+    (in_bom yes) (on_board yes) (dnp no)
     (property "Reference" "JP3" (at 96.52 120.65 0)
       (effects (font (size 1.27 1.27)) hide)
     )
-    (property "Value" "~{RESET}" (at 96.52 123.19 0)
+    (property "Value" "WP/ACC" (at 96.52 127 0)
       (effects (font (size 1.27 1.27)))
     )
@@
   )
   (symbol (lib_id "Connector:TestPoint") (at 105.41 128.27 90) (unit 1)
-    (in_bom yes) (on_board yes) (dnp no) (fields_autoplaced)
+    (in_bom yes) (on_board yes) (dnp no)
     (property "Reference" "TP1" (at 102.108 123.19 90)
       (effects (font (size 1.27 1.27)) hide)
     )
-    (property "Value" "~{RY/BY}" (at 100.33 128.905 90)
-      (effects (font (size 1.27 1.27)) (justify left))
-    )
+    (property "Value" "RY/BY" (at 104.14 130.81 90)
+      (effects (font (size 1.27 1.27)) (justify left))
+    )

Commit message: Update diode part
Parts:
- D1: value AZ23C3V6 -> BAV70LT1G
Changed lines of the file:
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@@
       (effects (font (size 1.27 1.27)))
     )
-    (property "Value" "AZ23C3V6" (at 123.317 25.4 90)
+    (property "Value" "BAV70LT1G" (at 123.317 25.4 90)
       (effects (font (size 1.27 1.27)))
     )
@@
       (effects (font (size 1.27 1.27)) (justify left) hide)
     )
-    (property "Datasheet" "https://www.vishay.com/docs/86340/az23_series.pdf" (at 123.19 27.94 90)
+    (property "Datasheet" "" (at 123.19 27.94 90)
       (effects (font (size 1.27 1.27)) hide)
     )

Commit message: Convert Pico to castellated footprint and reroute; add logo
Parts:
- U4: footprint LOOPY_PI:Pi Pico -> LOOPY_PI:RPi_Pico_SMD_TH
Changed lines of the file:
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@@
       (effects (font (size 1.27 1.27)))
     )
-    (property "Footprint" "LOOPY_PI:Pi Pico" (at 247.65 25.4 0)
+    (property "Footprint" "LOOPY_PI:RPi_Pico_SMD_TH" (at 247.65 25.4 0)
       (effects (font (size 1.27 1.27)) hide)
     )

Commit message: Added BAT54C to Pico 3V3 line; coin cell moved to rear; forehead removed
Parts:
- added D2: BAT54C, Package_TO_SOT_SMD:SOT-23, symbol Diode:BAT54C
Connections:
- net VCC: now also D2.3; no longer U4.36 (3V3)
- new net: D2.1, D2.2, U4.36 (3V3)
Changed lines of the file:
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@@
   (junction (at 248.92 218.44) (diameter 0) (color 0 0 0 0)
   )
+  (junction (at 278.13 39.37) (diameter 0) (color 0 0 0 0)
+  )
   (junction (at 86.36 129.54) (diameter 0) (color 0 0 0 0)
   )
@@
     (stroke (width 0) (type default))
   )
+  (wire (pts (xy 288.29 53.34) (xy 294.64 53.34))
+    (stroke (width 0) (type default))
+  )
   (wire (pts (xy 135.89 55.88) (xy 135.89 58.42))
     (stroke (width 0) (type default))
@@
     (stroke (width 0) (type default))
   )
+  (wire (pts (xy 288.29 50.8) (xy 288.29 53.34))
+    (stroke (width 0) (type default))
+  )
   (wire (pts (xy 151.13 143.51) (xy 144.78 143.51))
     (stroke (width 0) (type default))
@@
     (stroke (width 0) (type default))
   )
+  (wire (pts (xy 278.13 39.37) (xy 278.13 45.72))
+    (stroke (width 0) (type default))
+  )
   (wire (pts (xy 86.36 120.65) (xy 91.44 120.65))
     (stroke (width 0) (type default))
@@
     (stroke (width 0) (type default))
   )
+  (wire (pts (xy 262.89 39.37) (xy 278.13 39.37))
+    (stroke (width 0) (type default))
+  )
   (wire (pts (xy 82.55 118.11) (xy 82.55 121.92))
     (stroke (width 0) (type default))
@@
     (stroke (width 0) (type default))
   )
+  (wire (pts (xy 299.72 45.72) (xy 295.91 45.72))
+    (stroke (width 0) (type default))
+  )
   (wire (pts (xy 128.27 36.83) (xy 132.08 36.83))
     (stroke (width 0) (type default))
@@
     (stroke (width 0) (type default))
   )
+  (wire (pts (xy 299.72 39.37) (xy 299.72 45.72))
+    (stroke (width 0) (type default))
+  )
   (wire (pts (xy 204.47 29.21) (xy 204.47 25.4))
     (stroke (width 0) (type default))
@@
     (stroke (width 0) (type default))
   )
+  (wire (pts (xy 280.67 45.72) (xy 278.13 45.72))
+    (stroke (width 0) (type default))
+  )
   (wire (pts (xy 82.55 127) (xy 82.55 129.54))
     (stroke (width 0) (type default))
   )
+  (wire (pts (xy 278.13 39.37) (xy 299.72 39.37))
+    (stroke (width 0) (type default))
+  )
   (wire (pts (xy 82.55 129.54) (xy 86.36 129.54))
     (stroke (width 0) (type default))
@@
     (effects (font (size 1.27 1.27)) (justify right bottom))
   )
-  (text "Provide 3V power to board when plugged into USB" (at 276.86 39.37 0)
+  (text "Provide 3V power to board when plugged into USB" (at 270.51 33.02 0)
     (effects (font (size 1.27 1.27)) (justify left bottom))
   )
@@
     (effects (font (size 1.27 1.27)) (justify right bottom))
   )
-  (label "VCC" (at 262.89 39.37 0) (fields_autoplaced)
-    (effects (font (size 1.27 1.27)) (justify left bottom))
+  (label "VCC" (at 294.64 53.34 180) (fields_autoplaced)
+    (effects (font (size 1.27 1.27)) (justify right bottom))
   )
   (label "D2" (at 222.25 41.91 0) (fields_autoplaced)
@@
         )
       )
+    )
+  )
+  (symbol (lib_id "Diode:BAT54C") (at 288.29 45.72 0) (unit 1)
+    (in_bom yes) (on_board yes) (dnp no) (fields_autoplaced)
+    (property "Reference" "D2" (at 288.29 41.5671 0)
+      (effects (font (size 1.27 1.27)))
+    )
+    (property "Value" "BAT54C" (at 288.29 43.4881 0)
+      (effects (font (size 1.27 1.27)))
+    )
+    (property "Footprint" "Package_TO_SOT_SMD:SOT-23" (at 290.195 42.545 0)
+      (effects (font (size 1.27 1.27)) (justify left) hide)
+    )
+    (property "Datasheet" "http://www.diodes.com/_files/datasheets/ds11005.pdf" (at 286.258 45.72 0)
+      (effects (font (size 1.27 1.27)) hide)
+    )
+    (pin "1")
+    (pin "2")
+    (pin "3")
+    (instances
+      (project "singlerom-dev"
+        (path "/5081f4fb-0c92-4cfc-8c52-39777c6d96ed"
+          (reference "D2") (unit 1)
+        )
+      )

Commit message: Removing test jumpers and points
Parts:
- removed J2: PWR Breakout, Connector_PinHeader_2.54mm:PinHeader_1x02_P2.54mm_Vertical, symbol Connector:Conn_01x02_Socket
- removed JP1: WE, Jumper:SolderJumper-2_P1.3mm_Open_RoundedPad1.0x1.5mm, symbol Jumper:Jumper_2_Bridged
- removed JP2: RESET, Jumper:SolderJumper-2_P1.3mm_Open_RoundedPad1.0x1.5mm, symbol Jumper:Jumper_2_Bridged
- removed JP3: WP/ACC, Jumper:SolderJumper-2_P1.3mm_Open_RoundedPad1.0x1.5mm, symbol Jumper:Jumper_2_Bridged
- removed JP4: OE, Jumper:SolderJumper-2_P1.3mm_Open_RoundedPad1.0x1.5mm, symbol Jumper:Jumper_2_Bridged
- removed TP1: RY/BY, TestPoint:TestPoint_Pad_D1.0mm, symbol Connector:TestPoint
- removed TP2: RAM CS1, TestPoint:TestPoint_Pad_D1.0mm, symbol Connector:TestPoint
- removed TP3: RAM WE, TestPoint:TestPoint_Pad_D1.0mm, symbol Connector:TestPoint
- removed TP4: RAM A0, TestPoint:TestPoint_Pad_D1.0mm, symbol Connector:TestPoint
- removed TP5: RAM CS2, TestPoint:TestPoint_Pad_D1.0mm, symbol Connector:TestPoint
- removed TP6: OE, TestPoint:TestPoint_Pad_D1.0mm, symbol Connector:TestPoint
- removed TP7: ROM CE, TestPoint:TestPoint_Pad_D1.0mm, symbol Connector:TestPoint
Connections:
- net OE: now also U2.28 (OE#)
- net PICO_ROMWE: now also U2.11 (WE#)
- net VCC: now also U2.12 (RESET#), U2.14 (WP#/ACC)
