File: pcb/singlerom-dev/singlerom-dev.kicad_sch (KiCad schematic)
At the start: 17 parts, among them U1 AS6C6264-55SCN, U2 MX29LV160DBTI-70G, U4 Pi Pico, U5 TCA9539PWR

Commit message: WIP
Parts:
- removed U5: TCA9539PWR, Package_SO:TSSOP-24_4.4x7.8mm_P0.65mm, symbol LOOPY_IO:TCA9539PWR
- added IC1, IC2: MCP23S17T-E_SO, SOIC127P1030X265-28N, symbol LOOPY_IO_SPI:MCP23S17T-E_SO
Connections:
- net I2C_RESET is gone; now on net A18: U4.4 (2)
- net I2C_SCL is gone; now on net A17: U4.2 (1)
- net I2C_SDA is gone; now on net A0: U4.1 (0)
- net RAMA0 is gone; now on net A0: J1.33 (RAMA0), U1.10 (A0)
- net A0: no longer J1.32 (A0), U1.9 (A1), U2.25 (A0), U4.6 (4)
- net A1: now also J1.32 (A0), U1.9 (A1), U2.25 (A0), IC2.1 (GPB0); no longer J1.78 (A1), U1.8 (A2), U2.24 (A1), U4.7 (5)
- net A10: now also J1.23 (A9), U1.3 (A7), U2.7 (A9), IC2.22 (GPA1); no longer J1.67 (A10), U1.4 (A6), U2.6 (A10), U4.19 (14)
- net A11: now also J1.67 (A10), U1.4 (A6), U2.6 (A10), IC2.23 (GPA2); no longer J1.22 (A11), U1.5 (A5), U2.5 (A11), U4.20 (15)
- net A12: now also J1.22 (A11), U1.5 (A5), U2.5 (A11), IC2.24 (GPA3); no longer J1.26 (A12), U2.4 (A12), U4.21 (16)
- net A13: now also J1.26 (A12), U2.4 (A12), IC2.25 (GPA4); no longer J1.71 (A13), U2.3 (A13), U4.22 (17)
- net A14: now also J1.71 (A13), U2.3 (A13), IC2.26 (GPA5); no longer J1.27 (A14), U2.2 (A14), U4.24 (18)
- net A15: now also J1.27 (A14), U2.2 (A14), IC2.27 (GPA6); no longer J1.73 (A15), U2.1 (A15), U4.25 (19)
- net A16: now also J1.73 (A15), U2.1 (A15), IC2.28 (GPA7); no longer J1.72 (A16), U2.48 (A16), U4.26 (20)
- net A17: now also J1.72 (A16), U2.48 (A16); no longer J1.74 (A17), U2.17 (A17), U4.27 (21)
- net A18: now also J1.74 (A17), U2.17 (A17); no longer J1.76 (A18), U2.16 (A18), U4.29 (22)
- net A19: now also J1.76 (A18), U2.16 (A18), U4.6 (4); no longer J1.28 (A19), U2.9 (A19), U4.37 (23)
- net A2: now also J1.78 (A1), U1.8 (A2), U2.24 (A1), IC2.2 (GPB1); no longer J1.30 (A2), U1.7 (A3), U2.23 (A2), U4.9 (6)
- net A3: now also J1.30 (A2), U1.7 (A3), U2.23 (A2), IC2.3 (GPB2); no longer J1.77 (A3), U1.21 (A10), U2.22 (A3), U4.10 (7)
- net A4: now also J1.77 (A3), U1.21 (A10), U2.22 (A3), IC2.4 (GPB3); no longer J1.70 (A4), U1.6 (A4), U2.21 (A4), U4.11 (8)
- net A5: now also J1.70 (A4), U1.6 (A4), U2.21 (A4), IC2.5 (GPB4); no longer J1.25 (A5), U1.23 (A11), U2.20 (A5), U4.12 (9)
- net A6: now also J1.25 (A5), U1.23 (A11), U2.20 (A5), IC2.6 (GPB5); no longer J1.69 (A6), U1.24 (A9), U2.19 (A6), U4.14 (10)
- net A7: now also J1.69 (A6), U1.24 (A9), U2.19 (A6), IC2.7 (GPB6); no longer J1.24 (A7), U1.25 (A8), U2.18 (A7), U4.15 (11)
- net A8: now also J1.24 (A7), U1.25 (A8), U2.18 (A7), IC2.8 (GPB7); no longer J1.68 (A8), U1.2 (A12), U2.8 (A8), U4.16 (12)
- net A9: now also J1.68 (A8), U1.2 (A12), U2.8 (A8), IC2.21 (GPA0); no longer J1.23 (A9), U1.3 (A7), U2.7 (A9), U4.17 (13)
- net D0: now also IC1.21 (GPA0)
- net D1: now also IC1.22 (GPA1)
- net D10: now also IC1.3 (GPB2)
- net D11: now also IC1.4 (GPB3)
- net D12: now also IC1.5 (GPB4)
- net D13: now also IC1.6 (GPB5)
- net D14: now also IC1.7 (GPB6)
- net D15: now also IC1.8 (GPB7)
- net D2: now also IC1.23 (GPA2)
- net D3: now also IC1.24 (GPA3)
- net D4: now also IC1.25 (GPA4)
- net D5: now also IC1.26 (GPA5)
- net D6: now also IC1.27 (GPA6)
- net D7: now also IC1.28 (GPA7)
- net D8: now also IC1.1 (GPB0)
- net D9: now also IC1.2 (GPB1)
- net GND: now also IC1.15 (A0), IC1.16 (A1), IC1.17 (A2), IC2.16 (A1), IC2.17 (A2); no longer U4.38 (GND)
- net OE: now also U4.14 (10); no longer U4.34 (28)
- net PICO_GND: now also IC1.10 (VSS)
- net RAMCS1: now also U4.16 (12); no longer U4.31 (26)
- net RAMCS2: now also U4.17 (13)
- net RAMWE: now also U4.20 (15)
- net ROMCE: now also U4.15 (11); no longer U4.35 (29)
- net VCC: now also IC1.9 (VDD), IC2.15 (A0)
- net PICO_ROMWE renamed ROMWE
- net ROMWE: now also U4.19 (14); no longer U4.32 (27)
- new net A20: J1.28 (A19), U2.9 (A19), U4.7 (5)
- new net A21: U4.9 (6)
- new net SPI_CLK: IC1.12 (SCK), IC2.12 (SCK), U4.24 (18)
- new net SPI_CS: IC1.11 (~{CS}), IC2.11 (~{CS}), U4.22 (17)
- new net SPI_RX: IC1.14 (SO), IC2.14 (SO), U4.21 (16)
- new net SPI_TX: IC1.13 (SI), IC2.13 (SI), U4.25 (19)
- no-connect marks 13 -> 14

Commit message: vreg and resistor packs
Parts:
- removed C3: 0.1u, Capacitor_SMD:C_0805_2012Metric_Pad1.18x1.45mm_HandSolder, symbol Device:C_Small
- removed D2: BAT54C, Package_TO_SOT_SMD:SOT-23, symbol Diode:BAT54C
- removed U2: MX29LV160DBTI-70G, LOOPY_Flash:SOP50P2000X120-48N, symbol LOOPY_Flash:MX29LV160DBTI-70G
- removed U4: Pi Pico, LOOPY_PI:RPi_Pico_SMD_TH, symbol LOOPY_IO:Pi_Pico
- added R7, R8: R_Small, Resistor_SMD:R_0805_2012Metric_Pad1.20x1.40mm_HandSolder, symbol Device:R_Small
- added RN1, RN10, RN2, RN3, RN4, RN5, RN6, RN7, RN8, RN9: R_Pack04, LOOPY_ResNet:C_ARRAY_EXB28V_PAN, symbol Device:R_Pack04
- added U2: MIC5365-3.3YD5, Package_TO_SOT_SMD:SOT-23-5, symbol Regulator_Linear:MIC5365-3.3YD5
- added U3: Pico, LOOPY_PI:RPi_Pico_SMD_TH, symbol LOOPY_Pi:Pico
- added U4: MX29LV320EBTI-70G, LOOPY_Flash:TSOPI48L12X20NORMAL_MAC, symbol LOOPY_Flash:MX29LV320EBTI-70G
- IC1, IC2: footprint SOIC127P1030X265-28N -> LOOPY_IO_SPI:SOIC127P1030X265-28N
Connections:
- net PICO_GND is gone; now on net GND: IC1.10 (VSS)
- net A0: now also RN3.4 (R4.1), U3.1 (GPIO0); no longer J1.33 (RAMA0)
- net A1: now also RN3.3 (R3.1), U4.25 (A0); no longer J1.32 (A0)
- net A10: now also RN5.3 (R3.1), U4.7 (A9); no longer J1.23 (A9)
- net A11: now also RN10.6 (R3.2), U4.6 (A10); no longer J1.67 (A10)
- net A12: now also RN5.2 (R2.1), U4.5 (A11); no longer J1.22 (A11)
- net A13: now also RN4.2 (R2.1), U4.4 (A12); no longer J1.26 (A12)
- net A14: now also RN9.6 (R3.2), U4.3 (A13); no longer J1.71 (A13)
- net A15: now also RN4.3 (R3.1), U4.2 (A14); no longer J1.27 (A14)
- net A16: now also RN9.8 (R1.2), U4.1 (A15); no longer J1.73 (A15)
- net A17: now also RN9.7 (R2.2), U3.2 (GPIO1), U4.48 (A16); no longer J1.72 (A16)
- net A18: now also RN8.5 (R4.2), U3.4 (GPIO2), U4.17 (A17); no longer J1.74 (A17)
- net A19: now also RN8.6 (R3.2), U3.6 (GPIO4), U4.16 (A18); no longer J1.76 (A18)
- net A2: now also RN8.8 (R1.2), U4.24 (A1); no longer J1.78 (A1)
- net A20: now also RN4.4 (R4.1), U3.7 (GPIO5), U4.9 (A19); no longer J1.28 (A19)
- net A21: now also RN3.2 (R2.1), U3.9 (GPIO6), U4.10 (A20)
- net A3: now also RN3.1 (R1.1), U4.23 (A2); no longer J1.30 (A2)
- net A4: now also RN8.7 (R2.2), U4.22 (A3); no longer J1.77 (A3)
- net A5: now also RN9.5 (R4.2), U4.21 (A4); no longer J1.70 (A4)
- net A6: now also RN4.1 (R1.1), U4.20 (A5); no longer J1.25 (A5)
- net A7: now also RN10.8 (R1.2), U4.19 (A6); no longer J1.69 (A6)
- net A8: now also RN5.4 (R4.1), U4.18 (A7); no longer J1.24 (A7)
- net A9: now also RN10.7 (R2.2), U4.8 (A8); no longer J1.68 (A8)
- net D0: now also RN2.1 (R1.1), U4.29 (Q0); no longer J1.35 (D0)
- net D1: now also RN7.5 (R4.2), U4.31 (Q1); no longer J1.81 (D1)
- net D10: now also RN1.4 (R4.1), U4.34 (Q10); no longer J1.44 (D10)
- net D11: now also RN6.8 (R1.2), U4.36 (Q11); no longer J1.90 (D11)
- net D12: now also RN7.6 (R3.2), U4.39 (Q12); no longer J1.82 (D12)
- net D13: now also RN7.7 (R2.2), U4.41 (Q13); no longer J1.83 (D13)
- net D14: now also RN2.4 (R4.1), U4.43 (Q14); no longer J1.39 (D14)
- net D15: now also RN7.8 (R1.2), U4.45 (Q15/A-1); no longer J1.84 (D15)
- net D2: now also RN2.2 (R2.1), U4.33 (Q2); no longer J1.37 (D2)
- net D3: now also RN2.3 (R3.1), U4.35 (Q3); no longer J1.38 (D3)
- net D4: now also RN1.1 (R1.1), U4.38 (Q4); no longer J1.40 (D4)
- net D5: now also RN6.5 (R4.2), U4.40 (Q5); no longer J1.85 (D5)
- net D6: now also RN1.2 (R2.1), U4.42 (Q6); no longer J1.41 (D6)
- net D7: now also RN6.6 (R3.2), U4.44 (Q7); no longer J1.86 (D7)
- net D8: now also RN1.3 (R3.1), U4.30 (Q8); no longer J1.42 (D8)
- net D9: now also RN6.7 (R2.2), U4.32 (Q9); no longer J1.88 (D9)
- net GND: now also IC2.10 (VSS), U2.2 (GND), U3.13 (GND), U3.18 (GND), U3.23 (GND), U3.28 (GND), U3.3 (GND), U3.38 (GND), U3.8 (GND), U4.27 (GND), U4.46 (GND); no longer J1.13 (GND)
- net OE: now also R7.2, U3.14 (GPIO10), U4.28 (OE#); no longer J1.56 (OE)
- net RAMCS1: now also U3.16 (GPIO12)
- net RAMCS2: now also U3.17 (GPIO13)
- net RAMWE: now also U3.20 (GPIO15)
- net ROMCE: now also R8.2, U3.15 (GPIO11); no longer J1.54 (~ROMCE)
- net ROMWE: now also U3.19 (GPIO14), U4.11 (WE#)
- net SPI_CLK: now also U3.24 (GPIO18)
- net SPI_CS: now also U3.22 (GPIO17)
- net SPI_RX: now also U3.21 (GPIO16)
- net SPI_TX: now also U3.25 (GPIO19)
- net VCC: now also IC2.9 (VDD), U2.1 (VIN), U2.3 (EN), U3.36 (3V3), U4.12 (RESET#), U4.14 (WP#/ACC), U4.47 (BYTE#); no longer C2.1
- net PICO_RUN: now reaches IC1.18 (~{RESET})
- net PICO_RUN: now also IC2.18 (~{RESET}), J1.13 (GND), U3.30 (RUN)
- net at J1.31 (A21): now also RN3.7 (R2.2)
- new net: J1.78 (A2), RN8.1 (R1.1)
- new net: J1.77 (A4), RN8.2 (R2.1)
- new net: J1.76 (A19), RN8.3 (R3.1)
- new net: J1.74 (A18), RN8.4 (R4.1)
- new net: J1.28 (A20), RN4.5 (R4.2)
- new net: J1.27 (A15), RN4.6 (R3.2)
- new net: J1.26 (A13), RN4.7 (R2.2)
- new net: J1.25 (A6), RN4.8 (R1.2)
- new net: J1.73 (A16), RN9.1 (R1.1)
- new net: J1.72 (A17), RN9.2 (R2.1)
- new net: J1.71 (A14), RN9.3 (R3.1)
- new net: J1.70 (A5), RN9.4 (R4.1)
- new net: C2.1, U2.5 (VOUT), U4.37 (VCC)
- new net: J1.84 (D15), RN7.1 (R1.1)
- new net: J1.83 (D13), RN7.2 (R2.1)
- new net: J1.82 (D12), RN7.3 (R3.1)
- new net: J1.81 (D1), RN7.4 (R4.1)
- new net: J1.90 (D11), RN6.1 (R1.1)
- new net: J1.88 (D9), RN6.2 (R2.1)
- new net: J1.86 (D7), RN6.3 (R3.1)
- new net: J1.85 (D5), RN6.4 (R4.1)
- new net: J1.33 (A0), RN3.5 (R4.2)
- new net: J1.32 (A1), RN3.6 (R3.2)
- new net: J1.30 (A3), RN3.8 (R1.2)
- new net: J1.24 (A8), RN5.5 (R4.2)
- new net: J1.23 (A10), RN5.6 (R3.2)
- new net: J1.22 (A12), RN5.7 (R2.2)
- new net: J1.35 (D0), RN2.8 (R1.2)
- new net: J1.37 (D2), RN2.7 (R2.2)
- new net: J1.38 (D3), RN2.6 (R3.2)
- new net: J1.39 (D14), RN2.5 (R4.2)
- new net: J1.40 (D4), RN1.8 (R1.2)
- new net: J1.41 (D6), RN1.7 (R2.2)
- new net: J1.42 (D8), RN1.6 (R3.2)
- new net: J1.44 (D10), RN1.5 (R4.2)
- new net: J1.54 (~{CS6}), R8.1
- new net: J1.56 (~{OE}), R7.1
- new net: J1.67 (A11), RN10.3 (R3.1)
- new net: J1.68 (A9), RN10.2 (R2.1)
- new net: J1.69 (A7), RN10.1 (R1.1)
- no-connect marks 14 -> 47
Other:
- note added: "Address IO (Address 0x1)"
- note added: "Data IO (Address 0x0)"
- note added: "SPI IO Expanders, sharing a bus, giving us 32 extra inputs"
- note added: "SRAM is 5V tolerant"
- note removed: "/CE works same"
- note removed: "/OE active low observed"
- note removed: "Flash"
- note removed: "MaskROM: We should behave the same as this"
- note removed: "Pico acts as a switch providing a path from VCC to GND So IO expand only gets power when pico inserted?"
- note removed: "Power from USB only"
- moved on the sheet: C2, IC1, IC2, R1, R2, R3, R5
