File: pcb/singlerom-dev/singlerom-dev.kicad_pcb (KiCad board)
At the start: 2 copper layers, 96.3 x 48.2 mm, 28 parts, among them J4 PWR Breakout, U2 MX29LV320EBTI-70G

Commit message: tweaks
Changed lines of the file:
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@@
     )
     (fp_text value "RY" (at -2 0) (layer "F.SilkS")
-        (effects (font (size 0.5 0.5) (thickness 0.1)))
+        (effects (font (size 0.8 0.8) (thickness 0.1)))
     )
     (fp_text user "${REFERENCE}" (at 0 -1.45) (layer "F.Fab") hide
@@
     )
     (fp_text value "WP" (at -2 0) (layer "F.SilkS")
-        (effects (font (size 0.5 0.5) (thickness 0.1)))
+        (effects (font (size 0.8 0.8) (thickness 0.1)))
     )
     (fp_text user "${REFERENCE}" (at 0 -1.45) (layer "F.Fab")
@@
     (attr exclude_from_pos_files)
     (fp_text reference "TP4" (at 0 -1.448) (layer "F.SilkS")
-        (effects (font (size 0.5 0.5) (thickness 0.1)))
-    )
-    (fp_text value "ROM CE" (at 0 1.55) (layer "F.SilkS")
-        (effects (font (size 0.5 0.5) (thickness 0.1)))
+        (effects (font (size 0.8 0.8) (thickness 0.1)))
+    )
+    (fp_text value "ROM CE" (at 0 2.8) (layer "F.SilkS")
+        (effects (font (size 0.8 0.8) (thickness 0.1)))
     )
     (fp_text user "${REFERENCE}" (at 0 -1.45) (layer "F.Fab")
@@
     (attr exclude_from_pos_files)
     (fp_text reference "TP3" (at 0 -1.448) (layer "F.SilkS")
-        (effects (font (size 0.5 0.5) (thickness 0.1)))
+        (effects (font (size 0.8 0.8) (thickness 0.1)))
     )
     (fp_text value "OE" (at 0 1.55) (layer "F.SilkS")
-        (effects (font (size 0.5 0.5) (thickness 0.1)))
+        (effects (font (size 0.8 0.8) (thickness 0.1)))
     )
     (fp_text user "${REFERENCE}" (at 0 -1.45) (layer "F.Fab")
@@
     (attr exclude_from_pos_files)
     (fp_text reference "TP7" (at 0 -1.448) (layer "F.SilkS")
-        (effects (font (size 0.5 0.5) (thickness 0.1)))
-    )
-    (fp_text value "RAM WE" (at 0 1.55) (layer "F.SilkS")
-        (effects (font (size 0.5 0.5) (thickness 0.1)))
+        (effects (font (size 0.8 0.8) (thickness 0.1)))
+    )
+    (fp_text value "RAM WE" (at -0.1 2.7) (layer "F.SilkS")
+        (effects (font (size 0.8 0.8) (thickness 0.1)))
     )
     (fp_text user "${REFERENCE}" (at 0 -1.45) (layer "F.Fab")
@@
     (attr exclude_from_pos_files)
     (fp_text reference "TP5" (at 0 -1.448) (layer "F.SilkS")
-        (effects (font (size 0.5 0.5) (thickness 0.1)))
+        (effects (font (size 0.8 0.8) (thickness 0.1)))
     )
     (fp_text value "RAM CS2" (at 0 1.55) (layer "F.SilkS")
-        (effects (font (size 0.5 0.5) (thickness 0.1)))
+        (effects (font (size 0.8 0.8) (thickness 0.1)))
     )
     (fp_text user "${REFERENCE}" (at 0 -1.45) (layer "F.Fab")
@@
     (attr exclude_from_pos_files)
     (fp_text reference "TP6" (at 0 -1.448) (layer "F.SilkS")
-        (effects (font (size 0.5 0.5) (thickness 0.1)))
+        (effects (font (size 0.8 0.8) (thickness 0.1)))
     )
     (fp_text value "RAM A0" (at 0 1.55) (layer "F.SilkS")
-        (effects (font (size 0.5 0.5) (thickness 0.1)))
+        (effects (font (size 0.8 0.8) (thickness 0.1)))
     )
     (fp_text user "${REFERENCE}" (at 0 -1.45) (layer "F.Fab")
@@
     (attr exclude_from_pos_files)
     (fp_text reference "TP8" (at 0 -1.448) (layer "F.SilkS")
-        (effects (font (size 0.5 0.5) (thickness 0.1)))
+        (effects (font (size 0.8 0.8) (thickness 0.1)))
     )
     (fp_text value "RAM CS1" (at 0 1.55) (layer "F.SilkS")
-        (effects (font (size 0.5 0.5) (thickness 0.1)))
+        (effects (font (size 0.8 0.8) (thickness 0.1)))
     )
     (fp_text user "${REFERENCE}" (at 0 -1.45) (layer "F.Fab")
@@
     )
   )
+  (gr_rect (start 101.3 129.7) (end 199 135.5)
+    (stroke (width 0.15) (type solid)) (fill solid) (layer "B.Mask"))
+  (gr_rect (start 101.3 129.7) (end 199 135.5)
+    (stroke (width 0.15) (type solid)) (fill solid) (layer "F.Mask"))
   (gr_line (start 101.75 111.5) (end 101.75 119.25)
     (stroke (width 0.1) (type default)) (layer "Edge.Cuts"))

Commit message: Adds Pi Pico header + IO expander for on-board programming, starting over with manual routing
Parts:
- added C3: C_Small, Capacitor_SMD:C_0805_2012Metric_Pad1.18x1.45mm_HandSolder, F.Cu at (131.0, 81.0)
- added U3: MCP23S17-E/SS, LOOPY_IO:DIP787W46P254L3467H508Q28, F.Cu at (126.0, 73.5)
- added U4: Pi Pico, LOOPY_PI:Pi Pico, F.Cu at (172.8, 73.8)
- C1, C2: footprint Capacitor_SMD:C_1206_3216Metric_Pad1.33x1.80mm_HandSolder -> Capacitor_SMD:C_0805_2012Metric_Pad1.18x1.45mm_HandSolder
- H1, H3: value MountingHole_2mm -> MountingHole_4.5mm; footprint MountingHole:MountingHole_2mm -> MountingHole:MountingHole_4.5mm
- H2, H4: value MountingHole_2mm -> MountingHole_3.2mm_M3; footprint MountingHole:MountingHole_2mm -> MountingHole:MountingHole_3.2mm_M3
- moved C1 14.5 mm to (128.0, 93.8), turned to 90 degrees
- moved JP3 10.1 mm to (131.9, 98.8), turned to 180 degrees
- moved JP1 9.68 mm to (131.9, 107.8), turned to 180 degrees
- moved JP2 7.97 mm to (131.9, 105.3), turned to 180 degrees
- moved U1 5.77 mm to (123.1, 105.6), turned to 0 degrees
- moved R3 5.67 mm to (133.9, 127.1), turned to 0 degrees
- moved TP2 4.69 mm to (148.7, 107.5)
- moved TP1 4.43 mm to (148.7, 104.6)
- moved JP5 4.01 mm to (177.3, 108.6)
- moved R5 3.67 mm to (133.9, 124.8), turned to 0 degrees
- moved JP7 3.66 mm to (148.7, 101.0)
- moved JP8 3.66 mm to (148.7, 98.5)
- moved JP6 3.27 mm to (177.3, 105.3)
- moved C2 3.20 mm to (177.3, 97.5)
- moved U2 3.20 mm to (162.6, 102.3)
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Connections:
- JP8 pad 1: VCC -> /ROMWE
Routing:
- net VCC: track 229.3 -> 102.0 mm, vias 4 -> 6
- net /D7: track 138.9 -> 18.7 mm
- net /D6: track 126.4 -> 19.1 mm, vias 2 -> 1
- net /D4: track 118.7 -> 18.1 mm, vias 2 -> 1
- net /D3: track 114.1 -> 18.5 mm, vias 2 -> 1
- net /D1: track 95.4 -> 0.00 mm, vias 1 -> 0
- net /D5: track 110.0 -> 18.6 mm, vias 2 -> 1
- net /D2: track 100.2 -> 18.0 mm, vias 2 -> 1
- net /RAMA0: track 85.9 -> 10.6 mm, vias 2 -> 0
- net /D0: track 93.1 -> 18.7 mm
- net /OE: track 85.5 -> 12.0 mm, vias 5 -> 1
- net /ROMCE: track 76.9 -> 11.1 mm, vias 5 -> 1
- net GND: track 141.4 -> 83.7 mm, vias 36 -> 3
- net /D9: track 74.7 -> 20.2 mm
- net /A4: track 79.6 -> 25.6 mm
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- removed copper zone on B.Cu, net GND
- removed copper zone on F.Cu, net GND
Other:
- board size 96.3 x 48.2 mm -> 96.3 x 73.2 mm

Commit message: Work on rerouting devcart
Parts:
- moved JP7 5.56 mm to (152.8, 97.2)
- moved JP8 5.56 mm to (152.8, 94.7)
- moved TP1 5.56 mm to (152.8, 100.8)
- moved TP2 5.56 mm to (152.8, 103.8)
- moved C2 5.56 mm to (181.4, 93.7)
- moved JP4 5.56 mm to (181.4, 98.2)
- moved JP5 5.56 mm to (181.4, 104.8)
- moved JP6 5.56 mm to (181.4, 101.5)
- moved U2 5.56 mm to (166.7, 98.5)
- moved TP6 3.51 mm to (174.1, 123.8)
- moved C1 2.43 mm to (125.5, 94.2)
- moved U1 2.43 mm to (120.7, 106.0)
- moved JP1 2.43 mm to (129.6, 108.2)
- moved JP2 2.43 mm to (129.6, 105.7)
- moved JP3 2.43 mm to (129.6, 99.2)
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Routing:
- net /A6: track 24.9 -> 95.7 mm, vias 1 -> 4
- net /A4: track 25.6 -> 95.1 mm, vias 1 -> 4
- net /A5: track 26.4 -> 93.7 mm, vias 1 -> 3
- net /A7: track 25.3 -> 87.1 mm, vias 1 -> 4
- net /A2: track 44.4 -> 102.3 mm, vias 1 -> 3
- net /A3: track 43.5 -> 99.7 mm, vias 1 -> 4
- net /A11: track 23.7 -> 70.8 mm, vias 1 -> 2
- net /A10: track 16.4 -> 61.8 mm
- net /A0: track 42.7 -> 87.6 mm, vias 1 -> 2
- net /A1: track 59.1 -> 98.9 mm, vias 3 -> 4
- net /A8: track 24.2 -> 62.4 mm, vias 1 -> 3
- net /A9: track 24.6 -> 62.5 mm, vias 1 -> 2
- net /A13: track 26.3 -> 51.9 mm
- net /A12: track 26.2 -> 51.2 mm, vias 1 -> 0
- net /A16: track 27.0 -> 51.3 mm
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
Commit message: WIP rerouting devcart
Parts:
- moved U3 48.5 mm to (174.5, 73.5), turned to -90 degrees
- moved U4 45.8 mm to (127.0, 74.1), turned to 0 degrees
- moved C3 41.2 mm to (169.5, 66.0), turned to 180 degrees
- moved J4 6.56 mm to (190.8, 101.5), turned to -90 degrees
- moved TP2 4.64 mm to (149.7, 100.3)
- moved TP1 4.14 mm to (149.7, 98.1)
- moved TP5 2.15 mm to (174.1, 120.9)
Connections:
- U4 pad 13: GND -> unconnected-(U4-GND-Pad13)
- U4 pad 18: GND -> unconnected-(U4-GND-Pad18)
- U4 pad 23: GND -> unconnected-(U4-GND-Pad23)
- U4 pad 28: GND -> unconnected-(U4-GND-Pad28)
- U4 pad 3: GND -> unconnected-(U4-GND-Pad3)
- U4 pad 33: GND -> unconnected-(U4-GND-Pad33)
- U4 pad 38: GND -> unconnected-(U4-GND-Pad38)
- U4 pad 8: GND -> unconnected-(U4-GND-Pad8)
Routing:
- net /D1: track 0.00 -> 118.4 mm, vias 0 -> 5
- net /D2: track 18.0 -> 121.6 mm, vias 1 -> 4
- net /D0: track 18.7 -> 117.5 mm, vias 2 -> 6
- net /D4: track 18.1 -> 115.4 mm, vias 1 -> 4
- net /D3: track 18.5 -> 113.0 mm, vias 1 -> 4
- net /D6: track 19.1 -> 112.2 mm, vias 1 -> 4
- net /D5: track 18.6 -> 111.5 mm, vias 1 -> 5
- net VCC: track 102.5 -> 193.7 mm, vias 6 -> 7
- net /D7: track 18.7 -> 109.4 mm, vias 1 -> 5
- net GND: track 84.2 -> 174.4 mm, vias 3 -> 7
- net /A0: track 87.6 -> 158.4 mm, vias 2 -> 5
- net /A16: track 51.3 -> 114.4 mm, vias 1 -> 4
- net /A19: track 50.0 -> 111.8 mm, vias 0 -> 4
- net /D12: track 18.4 -> 68.0 mm, vias 1 -> 3
- net /A17: track 49.5 -> 98.9 mm, vias 1 -> 6
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
Commit message: Correcting wrong flash IC, footprint, symbol. Still needs rerouting but removed incorrect one.
Parts:
- removed U2: MX29LV320EBTI-70G, LOOPY_Flash_Macronix:MX29LV320EBTI-70G

Commit message: Forget FRAM for now, redesign around pin compatible SRAM, nuke old routes
Parts:
- removed C3: C_Small, Capacitor_SMD:C_0805_2012Metric_Pad1.18x1.45mm_HandSolder
- removed J4: PWR Breakout, Connector_PinHeader_2.54mm:PinHeader_1x02_P2.54mm_Vertical
- removed JP6: OE, Jumper:SolderJumper-2_P1.3mm_Open_RoundedPad1.0x1.5mm
- removed JP7: RST, Jumper:SolderJumper-2_P1.3mm_Open_RoundedPad1.0x1.5mm
- removed JP8: WE, Jumper:SolderJumper-2_P1.3mm_Open_RoundedPad1.0x1.5mm
- removed R3: 1K, Resistor_SMD:R_0805_2012Metric_Pad1.20x1.40mm_HandSolder
- removed TP8: RAM CS1, TestPoint:TestPoint_Pad_D1.0mm
- added J2: PWR Breakout, Connector_PinHeader_2.54mm:PinHeader_1x02_P2.54mm_Vertical, F.Cu at (190.8, 101.5)
- added R1: 1K, Resistor_SMD:R_0805_2012Metric_Pad1.20x1.40mm_HandSolder, F.Cu at (206.6, 94.3)
- added R2: 1K, Resistor_SMD:R_0805_2012Metric_Pad1.20x1.40mm_HandSolder, F.Cu at (206.6, 97.2)
- added R6: 100K, Resistor_SMD:R_0805_2012Metric_Pad1.20x1.40mm_HandSolder, F.Cu at (206.6, 103.1)
- added R7: 100K, Resistor_SMD:R_0805_2012Metric_Pad1.20x1.40mm_HandSolder, F.Cu at (206.6, 106.1)
- added U2: MX29LV160DBTI-70G, LOOPY_Flash:SOP50P2000X120-48N, F.Cu at (166.5, 92.0)
- C2: value C -> C_Small
- JP1: value CE -> WE
- JP2: value OE -> BYTE
- JP3: value WE -> RST
- JP4: value BYTE -> OE
- R5: value 1K -> 100K
- TP2: value RY -> RAM CS1
- TP3: value OE -> RAM WE
- TP4: value ROM CE -> RAM A0
- TP6: value RAM A0 -> OE
- TP7: value RAM WE -> ROM CE
- U1: value ~ -> AS6C6264-55SCN; footprint Package_SO:SOIC-28W_7.5x17.9mm_P1.27mm -> LOOPY_SRAM:SOP-28_Customized
- moved TP4 91.0 mm to (210.5, 103.5)
- moved TP3 88.4 mm to (210.5, 100.4)
- moved TP7 88.1 mm to (213.6, 100.4)
- moved R5 76.8 mm to (206.6, 100.2)
- moved JP1 73.8 mm to (202.1, 94.6), turned to 0 degrees
- moved JP2 72.9 mm to (202.1, 98.1), turned to 0 degrees
- moved JP3 72.6 mm to (202.1, 101.7), turned to 0 degrees
- moved TP1 61.0 mm to (210.5, 94.3)
- moved TP2 60.9 mm to (210.5, 97.4)
- moved TP5 47.6 mm to (213.6, 94.3)
- moved TP6 47.6 mm to (213.6, 97.4)
- moved C2 32.6 mm to (211.4, 106.5)
- moved JP4 21.8 mm to (202.1, 105.2), turned to 0 degrees
- moved JP5 21.1 mm to (202.1, 108.8), turned to 0 degrees
- moved U1 0.45 mm to (120.2, 106.0)
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Connections:
- C2 pad 1: VCC -> GND
- C2 pad 2: GND -> VCC
- JP1 pad 1: /RAMCS1 -> /PICO_ROMWE
- JP2 pad 1: /OE -> VCC
- JP3 pad 1: /RAMWE -> VCC
- JP4 pad 1: VCC -> /OE
- R5 pad 2: /F16 -> /PICO_ROMWE
- TP2 pad 1: Net-(U2A-RY/BY#) -> /RAMCS1
- TP3 pad 1: /OE -> /RAMWE
- TP4 pad 1: /ROMCE -> /RAMA0
- TP6 pad 1: /RAMA0 -> /OE
- TP7 pad 1: /RAMWE -> /ROMCE
- U1 pad 11: /D0 -> /D6
- U1 pad 12: /D1 -> /D5
- U1 pad 13: /D2 -> /D4
- U1 pad 16: /D4 -> /D2
- U1 pad 17: /D5 -> /D1
- U1 pad 18: /D6 -> /D0
- U1 pad 2: /A11 -> /A8
- U1 pad 20: Net-(JP1-B) -> /RAMCS1
- U1 pad 21: /A9 -> /A3
- U1 pad 22: Net-(JP2-B) -> /OE
- U1 pad 23: /A10 -> /A5
- U1 pad 24: /A8 -> /A6
- U1 pad 26: unconnected-(U1-NC-Pad26) -> /RAMCS2
- U1 pad 27: Net-(JP3-B) -> /RAMWE
- U1 pad 3: /A6 -> /A9
- U1 pad 4: /A5 -> /A10
- U1 pad 5: /A4 -> /A11
- U1 pad 6: /A3 -> /A4
- U3 pad 9: GND -> /PICO_GND
- U4 pad 3: unconnected-(U4-GND-Pad3) -> /PICO_GND
- U4 pad 31: /A20 -> /RAMCS1
- U4 pad 32: /ROMWE -> /PICO_ROMWE
- U4 pad 38: unconnected-(U4-GND-Pad38) -> GND
Routing:
- net /D2: track 121.6 -> 52.9 mm, vias 4 -> 0
- net /D1: track 118.4 -> 51.5 mm, vias 5 -> 1
- net /D0: track 117.5 -> 52.4 mm, vias 6 -> 2
- net /D4: track 115.4 -> 51.1 mm, vias 4 -> 0
- net /A0: track 158.4 -> 94.4 mm, vias 5 -> 2
- net /D6: track 112.2 -> 50.4 mm, vias 4 -> 0
- net /D3: track 113.0 -> 51.8 mm, vias 4 -> 0
- net /D5: track 111.5 -> 51.7 mm, vias 5 -> 1
- net /D7: track 109.4 -> 51.4 mm, vias 5 -> 1
- net /A3: track 126.6 -> 71.0 mm, vias 6 -> 1
- net /ROMWE: track 49.0 -> 0.00 mm, vias 1 -> 0
- net /A11: track 98.9 -> 50.6 mm, vias 5 -> 0
- net /A6: track 99.2 -> 56.7 mm, vias 4 -> 1
- net /A1: track 136.1 -> 93.8 mm, vias 5 -> 2
- net /A5: track 104.2 -> 62.1 mm, vias 4 -> 1
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
Commit message: Routing
Parts:
- removed JP5: CE, Jumper:SolderJumper-2_P1.3mm_Open_RoundedPad1.0x1.5mm
- removed R6, R7: 100K, Resistor_SMD:R_0805_2012Metric_Pad1.20x1.40mm_HandSolder
- added C3: C_Small, Capacitor_SMD:C_0805_2012Metric_Pad1.18x1.45mm_HandSolder, F.Cu at (167.0, 66.5)
- added R3: 100K, Resistor_SMD:R_0805_2012Metric_Pad1.20x1.40mm_HandSolder, F.Cu at (154.6, 85.7)
- added R4: 100K, Resistor_SMD:R_0805_2012Metric_Pad1.20x1.40mm_HandSolder, F.Cu at (128.6, 94.2)
- C2: value C_Small -> C
- moved TP2 95.7 mm to (118.0, 121.7)
- moved TP7 94.6 mm to (121.0, 119.6)
- moved TP6 94.2 mm to (122.6, 121.7)
- moved TP3 86.6 mm to (126.6, 121.7)
- moved R1 79.7 mm to (133.9, 126.8)
- moved R2 77.7 mm to (133.9, 124.6)
- moved TP1 57.0 mm to (153.7, 98.4)
- moved JP3 51.9 mm to (150.4, 97.4)
- moved JP2 51.9 mm to (150.4, 94.0)
- moved JP1 47.8 mm to (154.3, 93.9)
- moved TP5 45.6 mm to (174.1, 117.2)
- moved TP4 41.5 mm to (173.6, 122.3)
- moved C2 30.3 mm to (183.1, 95.7), turned to 90 degrees
- moved R5 23.3 mm to (183.9, 105.3), turned to 180 degrees
- moved JP4 19.3 mm to (183.3, 100.9), turned to 180 degrees
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Connections:
- C2 pad 1: GND -> VCC
- C2 pad 2: VCC -> GND
- R5 pad 2: /PICO_ROMWE -> /ROMCE
- U2 pad 26: Net-(JP5-B) -> /ROMCE
Routing:
- net VCC: track 171.1 -> 424.4 mm, vias 6 -> 7
- net GND: track 133.9 -> 372.6 mm, vias 4 -> 10
- net /ROMCE: track 10.5 -> 153.8 mm, vias 1 -> 4
- net /OE: track 9.96 -> 139.7 mm, vias 1 -> 6
- net /D6: track 50.4 -> 142.5 mm, vias 0 -> 4
- net /D5: track 51.7 -> 143.4 mm, vias 1 -> 5
- net /D4: track 51.1 -> 140.5 mm, vias 0 -> 4
- net /D7: track 51.4 -> 134.7 mm, vias 1 -> 5
- net /D3: track 51.8 -> 130.7 mm, vias 0 -> 4
- net /D2: track 52.9 -> 127.0 mm, vias 0 -> 4
- net /RAMCS1: track 5.72 -> 78.0 mm, vias 0 -> 2
- net /D1: track 51.5 -> 123.6 mm, vias 1 -> 5
- net /D0: track 52.4 -> 121.3 mm, vias 2 -> 6
- net /PICO_GND: track 0.00 -> 68.2 mm
- net /RAMA0: track 9.44 -> 77.2 mm, vias 0 -> 2
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Other:
- board size 96.3 x 73.2 mm -> 96.3 x 75.2 mm

Commit message: WIP
Routing:
- net /D11: track 100.1 -> 98.3 mm
- net /D10: track 96.7 -> 94.8 mm
- net /D8: track 89.7 -> 87.8 mm
- net /D9: track 93.7 -> 91.8 mm
- net /D1: track 123.6 -> 124.8 mm
- net /D12: track 87.3 -> 88.2 mm
- net /D3: track 130.7 -> 130.1 mm
- net /D4: track 140.5 -> 139.9 mm
