File: pcb/singlerom-dev/singlerom-dev.kicad_pcb (KiCad board)
At the start: 2 copper layers, 96.3 x 75.2 mm, 29 parts, among them J2 PWR Breakout, U1 AS6C6264-55SCN, U2 MX29LV160DBTI-70G, U3 MCP23S17-E/SS, U4 Pi Pico

Commit message: Replicate power path controller for SRAM from original
Parts:
- removed U3: MCP23S17-E/SS, LOOPY_IO:DIP787W46P254L3467H508Q28
- added BT1: CR2032, LOOPY_Cart:Keystone-3034TR-MFG, F.Cu at (180.5, 76.5)
- added D1: AZ23C3V6, Package_TO_SOT_SMD:SOT-23, F.Cu at (119.8, 94.3)
- added R6: 1.2K, Resistor_SMD:R_0805_2012Metric_Pad1.20x1.40mm_HandSolder, F.Cu at (115.9, 92.3)
- added U5: TCA9539PWR, Package_SO:TSSOP-24_4.4x7.8mm_P0.65mm, F.Cu at (159.0, 80.0)
- JP1: value WE -> ~{WE}
- JP3: value RST -> ~{RESET}
- JP4: value OE -> ~{OE}
- TP1: value WP -> ~{RY/BY}
- moved C3 17.6 mm to (153.8, 78.2), turned to 90 degrees
- turned C1 to -90 degrees
Connections:
- C1 pad 1: VCC -> GND
- C1 pad 2: GND -> Net-(D1-A)
- C3 pad 1: GND -> /PICO_GND
- U1 pad 28: VCC -> Net-(D1-A)
- U4 pad 1: /SPI_MISO -> /I2C_SDA
- U4 pad 2: /SPI_CS -> /I2C_SCL
- U4 pad 4: /SPI_CLK -> /I2C_RESET
- U4 pad 5: /SPI_MOSI -> unconnected-(U4-3-Pad5)
Routing:
- net +BATT: track 0.00 -> 118.5 mm, vias 0 -> 2
- net /SPI_CS: track 65.7 -> 0.00 mm
- net /I2C_SDA: track 0.00 -> 61.1 mm, vias 0 -> 2
- net /SPI_MISO: track 60.6 -> 0.00 mm
- net /SPI_CLK: track 58.6 -> 0.00 mm, vias 1 -> 0
- net /I2C_SCL: track 0.00 -> 58.0 mm
- net /I2C_RESET: track 0.00 -> 55.3 mm
- net /SPI_MOSI: track 54.1 -> 0.00 mm, vias 1 -> 0
- net GND: track 372.6 -> 405.5 mm
- net VCC: track 424.4 -> 399.5 mm, vias 7 -> 9
- net /D11: track 98.3 -> 78.2 mm
- net /D10: track 94.8 -> 76.8 mm
- net /D9: track 91.8 -> 74.9 mm
- net /D8: track 87.8 -> 72.1 mm
- net /D12: track 88.2 -> 76.3 mm, vias 3 -> 5
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
Commit message: Nudging clearances
Parts:
- C1: value C -> 1u
- C2: value C -> 0.1u
- C3: value C_Small -> 0.1u
- turned R4 to -90 degrees
Connections:
- R4 pad 1: /RAMCS2 -> GND
- R4 pad 2: GND -> /RAMCS2
Routing:
- net GND: track 405.5 -> 406.2 mm
- net +BATT: track 118.5 -> 119.3 mm

Commit message: Match pin numbers on battery so + faces up
Parts:
- H1, H3: value MountingHole_4.5mm -> MountingHole_5mm; footprint MountingHole:MountingHole_4.5mm -> MountingHole:MountingHole_5mm
Connections:
- BT1 pad 1: +BATT -> GND
- BT1 pad 2: GND -> +BATT
Routing:
- net GND: track 406.2 -> 385.7 mm
- net +BATT: track 119.3 -> 136.3 mm
Changed lines of the file:
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@@
       ))
   )
-  (footprint "MountingHole:MountingHole_4.5mm" locked (layer "F.Cu")
+  (footprint "MountingHole:MountingHole_5mm" locked (layer "F.Cu")
     (at 109 90.5)
-    (descr "Mounting Hole 4.5mm, no annular")
-    (tags "mounting hole 4.5mm no annular")
+    (descr "Mounting Hole 5mm, no annular")
+    (tags "mounting hole 5mm no annular")
     (attr board_only exclude_from_pos_files exclude_from_bom)
-    (fp_text reference "H1" (at 0 -5.5) (layer "F.Fab")
+    (fp_text reference "H1" (at 0 -6) (layer "F.SilkS") hide
         (effects (font (size 1 1) (thickness 0.15)))
     )
-    (fp_text value "MountingHole_4.5mm" (at 0 5.5) (layer "F.Fab")
+    (fp_text value "MountingHole_5mm" (at 0 6) (layer "F.Fab")
         (effects (font (size 1 1) (thickness 0.15)))
     )
@@
         (effects (font (size 1 1) (thickness 0.15)))
     )
-    (fp_circle (center 0 0) (end 4.5 0)
+    (fp_circle (center 0 0) (end 5 0)
       (stroke (width 0.15) (type solid)) (fill none) (layer "Cmts.User"))
-    (fp_circle (center 0 0) (end 4.75 0)
+    (fp_circle (center 0 0) (end 5.25 0)
       (stroke (width 0.05) (type solid)) (fill none) (layer "F.CrtYd"))
-    (pad "" np_thru_hole circle locked (at 0 0) (size 4.5 4.5) (drill 4.5) (layers "*.Cu" "*.Mask"))
+    (pad "" np_thru_hole circle locked (at 0 0) (size 5 5) (drill 5) (layers "*.Cu" "*.Mask"))
   )
   (footprint "TestPoint:TestPoint_Pad_D1.0mm" (layer "F.Cu")
@@
   (footprint "LOOPY_Cart:Keystone-3034TR-MFG" (layer "F.Cu")
     (at 180.5 76.5)
+    (property "Notes" "")
     (property "Sheetfile" "singlerom-dev.kicad_sch")
     (property "Sheetname" "")
@@
       (stroke (width 0.15) (type solid)) (layer "F.Fab"))
     (pad "1" smd rect (at 0 0.673099) (size 3.9624 3.9624) (layers "F.Cu" "F.Mask")
+      (net 18 "GND") (pinfunction "-") (pintype "passive"))
+    (pad "2" smd rect (at -10.984999 0.673099) (size 1.27 5.08) (layers "F.Cu" "F.Paste" "F.Mask")
       (net 108 "+BATT") (pinfunction "+") (pintype "passive"))
-    (pad "2" smd rect (at -10.984999 0.673099) (size 1.27 5.08) (layers "F.Cu" "F.Paste" "F.Mask")
-      (net 18 "GND") (pinfunction "-") (pintype "passive"))
     (pad "2" smd rect (at 10.984999 0.6731) (size 1.27 5.08) (layers "F.Cu" "F.Paste" "F.Mask")
-      (net 18 "GND") (pinfunction "-") (pintype "passive"))
+      (net 108 "+BATT") (pinfunction "+") (pintype "passive"))
     (model "eec.models/Keystone_-_3034TR.step"
       (offset (xyz 0 0.9042399864 0))
@@
     )
   )
-  (footprint "MountingHole:MountingHole_4.5mm" locked (layer "F.Cu")
+  (footprint "MountingHole:MountingHole_5mm" locked (layer "F.Cu")
     (at 188.25 90.5)
-    (descr "Mounting Hole 4.5mm, no annular")
-    (tags "mounting hole 4.5mm no annular")
+    (descr "Mounting Hole 5mm, no annular")
+    (tags "mounting hole 5mm no annular")
     (attr board_only exclude_from_pos_files exclude_from_bom)
-    (fp_text reference "H3" (at 0 -5.5) (layer "F.Fab")
+    (fp_text reference "H3" (at 0 -6) (layer "F.SilkS") hide
         (effects (font (size 1 1) (thickness 0.15)))
     )
-    (fp_text value "MountingHole_4.5mm" (at 0 5.5) (layer "F.Fab")
+    (fp_text value "MountingHole_5mm" (at 0 6) (layer "F.Fab")
         (effects (font (size 1 1) (thickness 0.15)))
     )
@@
         (effects (font (size 1 1) (thickness 0.15)))
     )
-    (fp_circle (center 0 0) (end 4.5 0)
+    (fp_circle (center 0 0) (end 5 0)
       (stroke (width 0.15) (type solid)) (fill none) (layer "Cmts.User"))
-    (fp_circle (center 0 0) (end 4.75 0)
+    (fp_circle (center 0 0) (end 5.25 0)
       (stroke (width 0.05) (type solid)) (fill none) (layer "F.CrtYd"))
-    (pad "" np_thru_hole circle locked (at 0 0) (size 4.5 4.5) (drill 4.5) (layers "*.Cu" "*.Mask"))
+    (pad "" np_thru_hole circle locked (at 0 0) (size 5 5) (drill 5) (layers "*.Cu" "*.Mask"))
   )
   (footprint "Resistor_SMD:R_0805_2012Metric_Pad1.20x1.40mm_HandSolder" (layer "F.Cu")
@@
   (segment (start 111.91 69.3) (end 107.95 65.34) (width 0.75) (layer "F.Cu") (net 18))
   (segment (start 114.7721 114.2) (end 114.7771 114.205) (width 0.75) (layer "F.Cu") (net 18))
-  (segment (start 169.515001 77.173099) (end 169.5 77.1881) (width 1) (layer "F.Cu") (net 18))
-  (segment (start 191.484999 77.1731) (end 191.484999 74.515001) (width 0.75) (layer "F.Cu") (net 18))
+  (segment (start 180.5 77.173099) (end 185.973099 71.7) (width 0.75) (layer "F.Cu") (net 18))
   (segment (start 129.4 132.1) (end 129.4 129.8) (width 0.75) (layer "F.Cu") (net 18))
   (segment (start 183.9125 94.6125) (end 190.8 101.5) (width 0.5) (layer "F.Cu") (net 18))
   (segment (start 179.75 101.85) (end 181.249294 101.85) (width 0.25) (layer "F.Cu") (net 18))
-  (segment (start 169.5 79.2) (end 173.8 83.5) (width 1) (layer "F.Cu") (net 18))
-  (segment (start 191.484999 74.515001) (end 197 69) (width 0.75) (layer "F.Cu") (net 18))
   (segment (start 111.91 69.31) (end 111.91 69.3) (width 0.75) (layer "F.Cu") (net 18))
-  (segment (start 187.8 83.5) (end 191.484999 79.815001) (width 1) (layer "F.Cu") (net 18))
+  (segment (start 185.973099 71.7) (end 194.3 71.7) (width 0.75) (layer "F.Cu") (net 18))
   (segment (start 197 126) (end 196.5 125.5) (width 0.75) (layer "F.Cu") (net 18))
   (segment (start 179.75 91.85) (end 179.75 92.35) (width 0.25) (layer "F.Cu") (net 18))
   (segment (start 189.8 106) (end 186.9 108.9) (width 0.75) (layer "F.Cu") (net 18))
-  (segment (start 169.5 77.1881) (end 169.5 79.2) (width 1) (layer "F.Cu") (net 18))
-  (segment (start 191.484999 79.815001) (end 191.484999 77.1731) (width 1) (layer "F.Cu") (net 18))
   (segment (start 110.7 114.4) (end 110.9 114.2) (width 0.75) (layer "F.Cu") (net 18))
   (segment (start 116.82 74.22) (end 111.91 69.31) (width 0.75) (layer "F.Cu") (net 18))
@@
   (segment (start 196.6 132.1) (end 197 131.7) (width 0.75) (layer "F.Cu") (net 18))
   (segment (start 120.4 91.4) (end 123.774289 91.4) (width 0.5) (layer "F.Cu") (net 18))
-  (segment (start 173.8 83.5) (end 187.8 83.5) (width 1) (layer "F.Cu") (net 18))
   (segment (start 182 95.75) (end 182 95.7125) (width 0.25) (layer "F.Cu") (net 18))
   (segment (start 110.9 114.2) (end 114.7721 114.2) (width 0.75) (layer "F.Cu") (net 18))
@@
   (segment (start 189.8 105.9) (end 189.8 106) (width 0.75) (layer "F.Cu") (net 18))
   (segment (start 183.1 94.6125) (end 180.8375 92.35) (width 0.25) (layer "F.Cu") (net 18))
+  (segment (start 194.3 71.7) (end 197 69) (width 0.75) (layer "F.Cu") (net 18))
   (via (at 186.9 108.9) (size 0.8) (drill 0.4) (layers "F.Cu" "B.Cu") (net 18))
   (via (at 182 95.75) (size 0.8) (drill 0.4) (layers "F.Cu" "B.Cu") (net 18))
@@
   (segment (start 155.89283 79.2375) (end 153.8 79.2375) (width 0.25) (layer "F.Cu") (net 107))
   (segment (start 104.8 85.1) (end 104.3 84.6) (width 0.75) (layer "F.Cu") (net 108))
-  (segment (start 165.826901 62.5) (end 180.5 77.173099) (width 0.75) (layer "F.Cu") (net 108))
+  (segment (start 169.515001 77.173099) (end 176.541902 84.2) (width 0.75) (layer "F.Cu") (net 108))
+  (segment (start 176.541902 84.2) (end 184.8 84.2) (width 0.75) (layer "F.Cu") (net 108))
   (segment (start 111.8 85.1) (end 104.8 85.1) (width 0.75) (layer "F.Cu") (net 108))
+  (segment (start 106.1 62.5) (end 154.841902 62.5) (width 0.75) (layer "F.Cu") (net 108))
   (segment (start 115.9 89.2) (end 111.8 85.1) (width 0.75) (layer "F.Cu") (net 108))
+  (segment (start 184.8 84.2) (end 191.484999 77.515001) (width 0.75) (layer "F.Cu") (net 108))
   (segment (start 115.9 91.3) (end 115.9 89.2) (width 0.75) (layer "F.Cu") (net 108))
-  (segment (start 106.1 62.5) (end 165.826901 62.5) (width 0.75) (layer "F.Cu") (net 108))
+  (segment (start 154.841902 62.5) (end 169.515001 77.173099) (width 0.75) (layer "F.Cu") (net 108))
+  (segment (start 191.484999 77.515001) (end 191.484999 77.1731) (width 0.75) (layer "F.Cu") (net 108))
   (via (at 104.3 84.6) (size 0.8) (drill 0.4) (layers "F.Cu" "B.Cu") (net 108))
   (via (at 106.1 62.5) (size 0.8) (drill 0.4) (layers "F.Cu" "B.Cu") (net 108))

Commit message: WIP some fixes, not completed but didn't want to leave broken
Parts:
- JP1: value ~{WE} -> WE
- JP2: value BYTE -> RESET
- JP3: value ~{RESET} -> WP/ACC
- JP4: value ~{OE} -> OE
- TP1: value ~{RY/BY} -> RY/BY
Connections:
- U2 pad 47: GND -> VCC
Routing:
- net GND: track 385.7 -> 385.2 mm
Changed lines of the file:
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@@
 (kicad_pcb (version 20221018) (generator pcbnew)
   (general
-    (thickness 1.6)
+    (thickness 1)
   )
   (paper "A4")
@@
       (layer "F.Mask" (type "Top Solder Mask") (thickness 0.01))
       (layer "F.Cu" (type "copper") (thickness 0.035))
-      (layer "dielectric 1" (type "core") (thickness 1.51) (material "FR4") (epsilon_r 4.5) (loss_tangent 0.02))
+      (layer "dielectric 1" (type "core") (thickness 0.91) (material "FR4") (epsilon_r 4.5) (loss_tangent 0.02))
       (layer "B.Cu" (type "copper") (thickness 0.035))
       (layer "B.Mask" (type "Bottom Solder Mask") (thickness 0.01))
@@
         (effects (font (size 0.8 0.8) (thickness 0.15)))
     )
-    (fp_text value "~{RESET}" (at 0 2.4) (layer "F.SilkS")
+    (fp_text value "WP/ACC" (at 0 2.4) (layer "F.SilkS")
         (effects (font (size 0.8 0.8) (thickness 0.15)))
     )
@@
         (effects (font (size 0.8 0.8) (thickness 0.15)))
     )
-    (fp_text value "~{OE}" (at -0.1 1.8) (layer "F.SilkS")
+    (fp_text value "OE" (at -0.1 1.8) (layer "F.SilkS")
         (effects (font (size 0.8 0.8) (thickness 0.15)))
     )
@@
       (net 18 "GND") (pinfunction "GND_2") (pintype "passive"))
     (pad "47" smd rect (at 9.85 -5.25 90) (size 0.3 1.3) (layers "F.Cu" "F.Paste" "F.Mask")
-      (net 18 "GND") (pinfunction "BYTE#") (pintype "passive"))
+      (net 84 "VCC") (pinfunction "BYTE#") (pintype "passive"))
     (pad "48" smd rect (at 9.85 -5.75 90) (size 0.3 1.3) (layers "F.Cu" "F.Paste" "F.Mask")
       (net 13 "/A16") (pinfunction "A16") (pintype "passive"))
@@
         (effects (font (size 0.8 0.8) (thickness 0.15)))
     )
-    (fp_text value "BYTE" (at 0 -1.7) (layer "F.SilkS")
+    (fp_text value "RESET" (at 0 -1.7) (layer "F.SilkS")
         (effects (font (size 0.8 0.8) (thickness 0.15)))
     )
@@
         (effects (font (size 0.8 0.8) (thickness 0.15)))
     )
-    (fp_text value "~{RY/BY}" (at 0.1 -1.5) (layer "F.SilkS")
+    (fp_text value "RY/BY" (at 0.1 -1.5) (layer "F.SilkS")
         (effects (font (size 0.8 0.8) (thickness 0.15)))
     )
@@
         (effects (font (size 0.8 0.8) (thickness 0.15)))
     )
-    (fp_text value "~{WE}" (at 0 -1.7) (layer "F.SilkS")
+    (fp_text value "WE" (at 0 -1.7) (layer "F.SilkS")
         (effects (font (size 0.8 0.8) (thickness 0.15)))
     )
@@
   (segment (start 185.973099 71.7) (end 194.3 71.7) (width 0.75) (layer "F.Cu") (net 18))
   (segment (start 197 126) (end 196.5 125.5) (width 0.75) (layer "F.Cu") (net 18))
-  (segment (start 179.75 91.85) (end 179.75 92.35) (width 0.25) (layer "F.Cu") (net 18))
   (segment (start 189.8 106) (end 186.9 108.9) (width 0.75) (layer "F.Cu") (net 18))
   (segment (start 110.7 114.4) (end 110.9 114.2) (width 0.75) (layer "F.Cu") (net 18))

Commit message: Quick patching BYTE issue
Routing:
- net VCC: track 399.5 -> 406.5 mm
- net GND: track 385.2 -> 385.5 mm, vias 10 -> 11
Changed lines of the file:
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@@
   (segment (start 129.4 132.1) (end 129.4 129.8) (width 0.75) (layer "F.Cu") (net 18))
   (segment (start 183.9125 94.6125) (end 190.8 101.5) (width 0.5) (layer "F.Cu") (net 18))
-  (segment (start 179.75 101.85) (end 181.249294 101.85) (width 0.25) (layer "F.Cu") (net 18))
   (segment (start 111.91 69.31) (end 111.91 69.3) (width 0.75) (layer "F.Cu") (net 18))
+  (segment (start 183.1 94.6125) (end 183.1 94.3) (width 0.25) (layer "F.Cu") (net 18))
+  (segment (start 179.75 92.35) (end 180.65 92.35) (width 0.25) (layer "F.Cu") (net 18))
   (segment (start 185.973099 71.7) (end 194.3 71.7) (width 0.75) (layer "F.Cu") (net 18))
   (segment (start 197 126) (end 196.5 125.5) (width 0.75) (layer "F.Cu") (net 18))
@@
   (segment (start 129.4 129.8) (end 128 128.4) (width 0.75) (layer "F.Cu") (net 18))
   (segment (start 196.6 132.1) (end 197 131.7) (width 0.75) (layer "F.Cu") (net 18))
+  (segment (start 183.1 94.3) (end 182.4 93.6) (width 0.25) (layer "F.Cu") (net 18))
   (segment (start 120.4 91.4) (end 123.774289 91.4) (width 0.5) (layer "F.Cu") (net 18))
-  (segment (start 182 95.75) (end 182 95.7125) (width 0.25) (layer "F.Cu") (net 18))
+  (segment (start 179.75 101.85) (end 180.95 101.85) (width 0.25) (layer "F.Cu") (net 18))
   (segment (start 110.9 114.2) (end 114.7721 114.2) (width 0.75) (layer "F.Cu") (net 18))
   (segment (start 197 131.7) (end 197 126) (width 0.75) (layer "F.Cu") (net 18))
   (segment (start 125.55 93.175711) (end 128.575711 93.175711) (width 0.5) (layer "F.Cu") (net 18))
-  (segment (start 181.249294 101.85) (end 181.35 101.85) (width 0.25) (layer "F.Cu") (net 18))
   (segment (start 123.774289 91.4) (end 125.55 93.175711) (width 0.5) (layer "F.Cu") (net 18))
   (segment (start 183.1 94.6125) (end 183.9125 94.6125) (width 0.5) (layer "F.Cu") (net 18))
-  (segment (start 180.8375 92.35) (end 179.75 92.35) (width 0.25) (layer "F.Cu") (net 18))
-  (segment (start 182 95.7125) (end 183.1 94.6125) (width 0.25) (layer "F.Cu") (net 18))
-  (segment (start 181.35 101.85) (end 181.7 102.2) (width 0.25) (layer "F.Cu") (net 18))
+  (segment (start 180.65 92.35) (end 181 92.7) (width 0.25) (layer "F.Cu") (net 18))
+  (segment (start 180.95 101.85) (end 181 101.8) (width 0.25) (layer "F.Cu") (net 18))
   (segment (start 189.8 105.9) (end 189.8 106) (width 0.75) (layer "F.Cu") (net 18))
-  (segment (start 183.1 94.6125) (end 180.8375 92.35) (width 0.25) (layer "F.Cu") (net 18))
   (segment (start 194.3 71.7) (end 197 69) (width 0.75) (layer "F.Cu") (net 18))
+  (via (at 181 101.8) (size 0.6) (drill 0.4) (layers "F.Cu" "B.Cu") (net 18))
   (via (at 186.9 108.9) (size 0.8) (drill 0.4) (layers "F.Cu" "B.Cu") (net 18))
-  (via (at 182 95.75) (size 0.8) (drill 0.4) (layers "F.Cu" "B.Cu") (net 18))
-  (via (at 181.7 102.2) (size 0.6) (drill 0.4) (layers "F.Cu" "B.Cu") (net 18))
   (via (at 116.82 74.22) (size 0.8) (drill 0.4) (layers "F.Cu" "B.Cu") (net 18))
   (via (at 116.8 87.8) (size 0.8) (drill 0.4) (layers "F.Cu" "B.Cu") (net 18))
+  (via (at 181 92.7) (size 0.6) (drill 0.4) (layers "F.Cu" "B.Cu") (net 18))
   (via (at 196.5 125.5) (size 0.8) (drill 0.4) (layers "F.Cu" "B.Cu") (net 18))
   (via (at 110.7 114.4) (size 0.6) (drill 0.4) (layers "F.Cu" "B.Cu") (net 18))
   (via (at 189.8 105.9) (size 0.8) (drill 0.4) (layers "F.Cu" "B.Cu") (net 18))
+  (via (at 182.4 93.6) (size 0.6) (drill 0.4) (layers "F.Cu" "B.Cu") (net 18))
   (via (at 128 128.4) (size 0.8) (drill 0.4) (layers "F.Cu" "B.Cu") (net 18))
   (via (at 197 69) (size 0.8) (drill 0.4) (layers "F.Cu" "B.Cu") (net 18))
@@
   (segment (start 160.9 119.9) (end 160.9 123) (width 0.75) (layer "B.Cu") (net 18))
   (segment (start 189.8 102.5) (end 190.8 101.5) (width 0.75) (layer "B.Cu") (net 18))
+  (segment (start 181 92.7) (end 181 101.8) (width 0.25) (layer "B.Cu") (net 18))
   (segment (start 109.3 115.8) (end 110.7 114.4) (width 0.75) (layer "B.Cu") (net 18))
   (segment (start 107.3 125.7) (end 106.3 124.7) (width 0.75) (layer "B.Cu") (net 18))
-  (segment (start 182 101.9) (end 181.7 102.2) (width 0.25) (layer "B.Cu") (net 18))
   (segment (start 106.3 132.1) (end 106.3 124.7) (width 0.75) (layer "B.Cu") (net 18))
   (segment (start 192.62132 101.5) (end 197 97.12132) (width 0.75) (layer "B.Cu") (net 18))
@@
   (segment (start 195.4 124.4) (end 196.5 125.5) (width 0.75) (layer "B.Cu") (net 18))
   (segment (start 116.82 91.58) (end 109.3 99.1) (width 0.75) (layer "B.Cu") (net 18))
+  (segment (start 182.4 93.6) (end 181.9 93.6) (width 0.25) (layer "B.Cu") (net 18))
   (segment (start 192.62132 61) (end 112 61) (width 0.75) (layer "B.Cu") (net 18))
   (segment (start 107.95 65.05) (end 107.95 65.34) (width 0.75) (layer "B.Cu") (net 18))
-  (segment (start 182 95.75) (end 182 101.9) (width 0.25) (layer "B.Cu") (net 18))
   (segment (start 186.9 108.9) (end 186 109.8) (width 0.75) (layer "B.Cu") (net 18))
   (segment (start 189.8 105.9) (end 189.8 111.6) (width 0.75) (layer "B.Cu") (net 18))
@@
   (segment (start 125.3 125.7) (end 107.3 125.7) (width 0.75) (layer "B.Cu") (net 18))
   (segment (start 160.9 123) (end 165.1 127.2) (width 0.75) (layer "B.Cu") (net 18))
+  (segment (start 181.9 93.6) (end 181 92.7) (width 0.25) (layer "B.Cu") (net 18))
   (segment (start 195.4 117.2) (end 195.4 124.4) (width 0.75) (layer "B.Cu") (net 18))
   (segment (start 106.3 124.7) (end 106.3 118.8) (width 0.75) (layer "B.Cu") (net 18))
@@
   (segment (start 149.7 88.8) (end 149.7 93.95) (width 0.5) (layer "F.Cu") (net 84))
   (segment (start 104.2 132.1) (end 104.2 128.4) (width 0.75) (layer "F.Cu") (net 84))
-  (segment (start 182.9375 96.85) (end 183.1 96.6875) (width 0.25) (layer "F.Cu") (net 84))
+  (segment (start 181.7 95.2875) (end 183.1 96.6875) (width 0.25) (layer "F.Cu") (net 84))
   (segment (start 108.9 127) (end 106.7 127) (width 0.75) (layer "F.Cu") (net 84))
   (segment (start 163.2 131.9) (end 163 132.1) (width 0.75) (layer "F.Cu") (net 84))
   (segment (start 128.6 127) (end 124.6 127) (width 0.75) (layer "F.Cu") (net 84))
+  (segment (start 181.05 91.85) (end 181.7 92.5) (width 0.25) (layer "F.Cu") (net 84))
   (segment (start 131.5 129.9) (end 128.6 127) (width 0.75) (layer "F.Cu") (net 84))
   (segment (start 132.3 127) (end 132.9 126.4) (width 0.75) (layer "F.Cu") (net 84))
@@
   (segment (start 163.2 127.7) (end 163.2 131.9) (width 0.75) (layer "F.Cu") (net 84))
   (segment (start 104.8 125.1) (end 104.8 124.3) (width 0.75) (layer "F.Cu") (net 84))
-  (segment (start 179.75 96.85) (end 182.9375 96.85) (width 0.25) (layer "F.Cu") (net 84))
   (segment (start 106.7 127) (end 104.8 125.1) (width 0.75) (layer "F.Cu") (net 84))
   (segment (start 188.26 101.5) (end 183.4475 96.6875) (width 0.5) (layer "F.Cu") (net 84))
   (segment (start 111.02868 95.25) (end 110.93934 95.33934) (width 0.5) (layer "F.Cu") (net 84))
+  (segment (start 179.75 96.85) (end 182.9375 96.85) (width 0.25) (layer "F.Cu") (net 84))
+  (segment (start 181.7 92.5) (end 181.7 95.2875) (width 0.25) (layer "F.Cu") (net 84))
+  (segment (start 182.9375 96.85) (end 183.1 96.6875) (width 0.25) (layer "F.Cu") (net 84))
   (segment (start 155.4 77.1625) (end 155.425 77.1375) (width 0.25) (layer "F.Cu") (net 84))
   (segment (start 153.8 77.1625) (end 155.4 77.1625) (width 0.25) (layer "F.Cu") (net 84))
   (segment (start 149.75 97.4) (end 149.75 94) (width 0.25) (layer "F.Cu") (net 84))
+  (segment (start 179.75 91.85) (end 181.05 91.85) (width 0.25) (layer "F.Cu") (net 84))
   (segment (start 132.9 126.4) (end 132.9 124.8) (width 0.75) (layer "F.Cu") (net 84))
   (segment (start 156.9 86.6) (end 156 85.7) (width 0.5) (layer "F.Cu") (net 84))
@@
   (segment (start 159.2 97.85) (end 160.05 97.85) (width 0.25) (layer "F.Cu") (net 88))
   (segment (start 151.05 97.4) (end 158.75 97.4) (width 0.25) (layer "F.Cu") (net 88))
-  (segment (start 181.245405 100.9) (end 182.65 100.9) (width 0.25) (layer "F.Cu") (net 89))
-  (segment (start 179.75 101.35) (end 180.795405 101.35) (width 0.25) (layer "F.Cu") (net 89))
-  (segment (start 180.795405 101.35) (end 181.245405 100.9) (width 0.25) (layer "F.Cu") (net 89))
+  (segment (start 179.75 101.35) (end 180.637534 101.35) (width 0.25) (layer "F.Cu") (net 89))
+  (segment (start 181.087534 100.9) (end 182.65 100.9) (width 0.25) (layer "F.Cu") (net 89))
+  (segment (start 180.637534 101.35) (end 181.087534 100.9) (width 0.25) (layer "F.Cu") (net 89))
   (segment (start 154.1 98) (end 153.7 98.4) (width 0.25) (layer "F.Cu") (net 90))
   (segment (start 159.134314 98.35) (end 158.784314 98) (width 0.25) (layer "F.Cu") (net 90))

Commit message: Convert Pico to castellated footprint and reroute; add logo
Parts:
- U4: value Pi Pico -> RPi_Pico_SMD_TH; footprint LOOPY_PI:Pi Pico -> LOOPY_PI:RPi_Pico_SMD_TH
- moved C3 2.42 mm to (155.5, 76.4)
- moved U5 2.42 mm to (160.7, 78.2)
- moved R3 0.47 mm to (155.1, 85.7)
- turned U4 to 90 degrees
Routing:
- net +BATT: track 136.3 -> 120.2 mm
- net /A14: track 96.2 -> 101.9 mm, vias 3 -> 5
- net /I2C_SDA: track 61.1 -> 63.8 mm
- net /PICO_GND: track 68.6 -> 71.1 mm
- net /A2: track 134.8 -> 132.6 mm
- net /A8: track 107.3 -> 109.2 mm, vias 6 -> 7
- net GND: track 385.5 -> 387.3 mm
- net /D12: track 76.3 -> 77.9 mm
- net /D14: track 79.8 -> 81.2 mm
- net /D15: track 81.3 -> 82.6 mm
- net /A9: track 108.4 -> 109.7 mm, vias 5 -> 6
- net /A6: track 92.0 -> 93.2 mm
- net /D10: track 76.8 -> 75.7 mm, vias 2 -> 4
- net /D11: track 78.2 -> 77.1 mm, vias 1 -> 3
- net /D0: track 115.9 -> 116.9 mm
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Other:
- board size 96.3 x 75.2 mm -> 96.3 x 94.2 mm
