File: pcb/singlerom-dev/singlerom-dev.kicad_pcb (KiCad board)
At the start: 2 copper layers, 96.3 x 94.2 mm, 32 parts, among them J2 PWR Breakout, U1 AS6C6264-55SCN, U2 MX29LV160DBTI-70G, U4 RPi_Pico_SMD_TH, U5 TCA9539PWR

Commit message: Added BAT54C to Pico 3V3 line; coin cell moved to rear; forehead removed
Parts:
- added D2: BAT54C, Package_TO_SOT_SMD:SOT-23, F.Cu at (158.4, 63.5)
- BT1: moved to B.Cu
- D1: value AZ23C3V6 -> BAV70LT1G
- U4: value RPi_Pico_SMD_TH -> Pi Pico
- turned BT1 to 180 degrees
Connections:
- U4 pad 36: VCC -> Net-(U4-3V3)
Routing:
- net VCC: track 405.5 -> 352.4 mm, vias 9 -> 11
- net Net-(U4-3V3): track 0.00 -> 49.4 mm, vias 0 -> 2
- net +BATT: vias 2 -> 3
- net GND: vias 11 -> 12
Other:
- board size 96.3 x 94.2 mm -> 96.3 x 76.2 mm

Commit message: Removing test jumpers and points
Parts:
- removed J2: PWR Breakout, Connector_PinHeader_2.54mm:PinHeader_1x02_P2.54mm_Vertical
- removed JP1: WE, Jumper:SolderJumper-2_P1.3mm_Open_RoundedPad1.0x1.5mm
- removed JP2: RESET, Jumper:SolderJumper-2_P1.3mm_Open_RoundedPad1.0x1.5mm
- removed JP3: WP/ACC, Jumper:SolderJumper-2_P1.3mm_Open_RoundedPad1.0x1.5mm
- removed JP4: OE, Jumper:SolderJumper-2_P1.3mm_Open_RoundedPad1.0x1.5mm
- removed TP1: RY/BY, TestPoint:TestPoint_Pad_D1.0mm
- removed TP2: RAM CS1, TestPoint:TestPoint_Pad_D1.0mm
- removed TP3: RAM WE, TestPoint:TestPoint_Pad_D1.0mm
- removed TP4: RAM A0, TestPoint:TestPoint_Pad_D1.0mm
- removed TP5: RAM CS2, TestPoint:TestPoint_Pad_D1.0mm
- removed TP6: OE, TestPoint:TestPoint_Pad_D1.0mm
- removed TP7: ROM CE, TestPoint:TestPoint_Pad_D1.0mm
Connections:
- U2 pad 11: Net-(JP1-B) -> /PICO_ROMWE
- U2 pad 12: Net-(JP2-B) -> VCC
- U2 pad 14: Net-(JP3-B) -> VCC
- U2 pad 15: Net-(U2-RY/BY#) -> unconnected-(U2-RY/BY#-Pad15)
- U2 pad 28: Net-(JP4-B) -> /OE
Routing:
- net VCC: track 352.4 -> 368.5 mm, vias 11 -> 12
- net Net-(JP2-B): track 10.2 -> 0.00 mm
- net Net-(JP3-B): track 9.19 -> 0.00 mm
- net /PICO_ROMWE: track 49.0 -> 56.2 mm
- net Net-(U2-RY/BY#): track 6.66 -> 0.00 mm
- net Net-(JP1-B): track 6.11 -> 0.00 mm
- net GND: track 387.3 -> 390.8 mm
- net Net-(JP4-B): track 3.09 -> 0.00 mm
- net /OE: track 139.7 -> 142.4 mm
Other:
- board text removed: "GND"
- board text removed: "VCC"

Commit message: Add hand-solder footprint for Sharp Flash
Other:
- board text added: "JLCJLCJLCJLC"
Changed lines of the file:
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@@
       (outputformat 1)
       (mirror false)
-      (drillshape 1)
+      (drillshape 0)
       (scaleselection 1)
-      (outputdirectory "")
+      (outputdirectory "gerbil")
     )
   )
@@
   (gr_rect (start 101.3 129.7) (end 199 135.5)
     (stroke (width 0.15) (type solid)) (fill solid) (layer "User.4"))
+  (gr_text "JLCJLCJLCJLC" (at 161.544 93.091) (layer "F.SilkS")
+    (effects (font (size 0.8 0.8) (thickness 0.08)) (justify left bottom))
+  )
   (segment (start 121 97.3755) (end 121 106.1) (width 0.25) (layer "F.Cu") (net 1))
   (segment (start 121 106.1) (end 122.755 107.855) (width 0.25) (layer "F.Cu") (net 1))
