File: pcb/reverse-wanwan/reverse-wanwan.kicad_sch (KiCad schematic)
At the start: 27 parts, among them IC11 BA15218F-E2, U11 OKI_M6653A, X101 4.09

Commit message: Updating more pins on wanwan
Parts:
- added IC102: 74HC273, symbol 74xx:74HC273
- added R115, R116, R117, R118, R119: R_Small, symbol Device:R_Small
- renumbered U11 to IC101, IC11 to IC106
Connections:
- net F61: no longer J1.61 (F61)
- net ATST: now reaches IC101.16 (~{TEST})
- net ATST: now also R117.2
- net ARST: now reaches IC101.17 (~{RESET})
- net ARST: now also R118.2
- net AXT: now reaches IC101.22 (XT/~{CR})
- net AXT: now also R119.1
- net AOSC: now reaches IC101.5 (OSC3)
- net AOSC: now also R115.2
- net ARND: now reaches IC101.8 (~{RND})
- net ARND: now also R116.2
- net at J1.18: now also R116.1
- net at J1.20: now also R117.1
- net at J1.62: now also R115.1
- net at J1.63: now also R119.2
- net F16: no longer names the net of J1.16 (F16)
- net F16: now also R118.1
- new net FFVCC: IC102.20 (VCC), J1.61 (F61)
Other:
- moved on the sheet: C101, C113, IC101, X101

Commit message: WIP on wanwan schematic, all cart edge pins identified
Parts:
- added IC11: TC7W139, Package_SO:SOP-8_3.76x4.96mm_P1.27mm, symbol TC7W139F:TC7W139F
- added R103: R_Small, symbol Device:R_Small
Connections:
- net GND: now also IC11.4 (GND)
- net ROMCE: no longer J1.54 (~ROMCE)
- net VCC: now also IC11.8 (VCC)
- net FFCP: now reaches IC102.11 (Cp)
- net FFCP: now also R103.2
- net AMPVEE: now reaches C109.2, C110.2, IC106.4 (VEE)
- net AMPVEE: now also J1.49
- net MUXA: now reaches J1.31
- net MUXA: now also IC11.1 (A)
- net at J1.53: now also R103.1
- new net MUXB: IC11.2 (B), J1.54 (~ROMCE)
- no-connect marks 0 -> 1
Other:
- moved on the sheet: IC102
Changed lines of the file:
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@@
   (junction (at 133.35 25.4) (diameter 0) (color 0 0 0 0)
   )
+  (no_connect (at 199.39 123.19))
   (wire (pts (xy 194.31 151.13) (xy 199.39 151.13))
     (stroke (width 0) (type default))
@@
     (stroke (width 0) (type default))
   )
+  (wire (pts (xy 177.8 22.86) (xy 189.23 22.86))
+    (stroke (width 0) (type default))
+  )
   (wire (pts (xy 171.45 101.6) (xy 171.45 107.95))
     (stroke (width 0) (type default))
@@
     (stroke (width 0) (type default))
   )
+  (wire (pts (xy 222.25 133.35) (xy 231.14 133.35))
+    (stroke (width 0) (type default))
+  )
   (wire (pts (xy 116.84 52.07) (xy 119.38 52.07))
     (stroke (width 0) (type default))
@@
     (stroke (width 0) (type default))
   )
+  (wire (pts (xy 236.22 133.35) (xy 242.57 133.35))
+    (stroke (width 0) (type default))
+  )
   (wire (pts (xy 129.54 22.86) (xy 135.89 22.86))
     (stroke (width 0) (type default))
@@
     (effects (font (size 1.27 1.27)) (justify right bottom))
   )
+  (label "FFCP" (at 123.19 154.94 180) (fields_autoplaced)
+    (effects (font (size 1.27 1.27)) (justify right bottom))
+  )
   (label "RAMWE" (at 82.55 48.26 0) (fields_autoplaced)
     (effects (font (size 1.27 1.27)) (justify left bottom))
@@
     (effects (font (size 1.27 1.27)) (justify right bottom))
   )
+  (label "MUXA" (at 199.39 115.57 180) (fields_autoplaced)
+    (effects (font (size 1.27 1.27)) (justify right bottom))
+  )
   (label "D13" (at 95.25 135.89 0) (fields_autoplaced)
     (effects (font (size 1.27 1.27)) (justify left bottom))
@@
     (effects (font (size 1.27 1.27)) (justify left bottom))
   )
+  (label "GND" (at 177.8 139.7 0) (fields_autoplaced)
+    (effects (font (size 1.27 1.27)) (justify left bottom))
+  )
   (label "AOSC" (at 166.37 102.87 0) (fields_autoplaced)
     (effects (font (size 1.27 1.27)) (justify left bottom))
@@
     (effects (font (size 1.27 1.27)) (justify right bottom))
   )
+  (label "MUXB" (at 177.8 144.78 0) (fields_autoplaced)
+    (effects (font (size 1.27 1.27)) (justify left bottom))
+  )
   (label "D10" (at 199.39 148.59 180) (fields_autoplaced)
     (effects (font (size 1.27 1.27)) (justify right bottom))
@@
     (effects (font (size 1.27 1.27)) (justify right bottom))
   )
-  (label "ROMCE" (at 222.25 130.81 0) (fields_autoplaced)
-    (effects (font (size 1.27 1.27)) (justify left bottom))
-  )
   (label "A6" (at 73.66 102.87 180) (fields_autoplaced)
     (effects (font (size 1.27 1.27)) (justify right bottom))
@@
     (effects (font (size 1.27 1.27)) (justify right bottom))
   )
+  (label "MUXB" (at 222.25 130.81 0) (fields_autoplaced)
+    (effects (font (size 1.27 1.27)) (justify left bottom))
+  )
   (label "A6" (at 82.55 55.88 0) (fields_autoplaced)
     (effects (font (size 1.27 1.27)) (justify left bottom))
@@
     (effects (font (size 1.27 1.27)) (justify left bottom))
   )
+  (label "AMPVEE" (at 222.25 143.51 0) (fields_autoplaced)
+    (effects (font (size 1.27 1.27)) (justify left bottom))
+  )
   (label "D15" (at 95.25 125.73 0) (fields_autoplaced)
     (effects (font (size 1.27 1.27)) (justify left bottom))
@@
     (effects (font (size 1.27 1.27)) (justify right bottom))
   )
+  (label "MUXA" (at 177.8 147.32 0) (fields_autoplaced)
+    (effects (font (size 1.27 1.27)) (justify left bottom))
+  )
   (label "A12" (at 95.25 107.95 0) (fields_autoplaced)
     (effects (font (size 1.27 1.27)) (justify left bottom))
@@
     (effects (font (size 1.27 1.27)) (justify left bottom))
   )
+  (label "FFCP" (at 242.57 133.35 0) (fields_autoplaced)
+    (effects (font (size 1.27 1.27)) (justify left bottom))
+  )
   (label "D14" (at 95.25 130.81 0) (fields_autoplaced)
     (effects (font (size 1.27 1.27)) (justify left bottom))
@@
     (effects (font (size 1.27 1.27)) (justify right bottom))
   )
+  (label "VCC" (at 157.48 147.32 180) (fields_autoplaced)
+    (effects (font (size 1.27 1.27)) (justify right bottom))
+  )
   (label "D2" (at 199.39 130.81 180) (fields_autoplaced)
     (effects (font (size 1.27 1.27)) (justify right bottom))
@@
     (effects (font (size 1.27 1.27)) (justify right bottom))
   )
+  (label "AMPVEE" (at 189.23 22.86 0) (fields_autoplaced)
+    (effects (font (size 1.27 1.27)) (justify left bottom))
+  )
   (label "VCC" (at 106.68 146.05 180) (fields_autoplaced)
     (effects (font (size 1.27 1.27)) (justify right bottom))
@@
     (effects (font (size 1.27 1.27)) (justify right bottom))
   )
-  (label "FFVCC" (at 153.67 129.54 0) (fields_autoplaced)
+  (label "FFVCC" (at 135.89 124.46 0) (fields_autoplaced)
     (effects (font (size 1.27 1.27)) (justify left bottom))
   )
@@
     )
   )
-  (symbol (lib_id "74xx:74HC273") (at 153.67 149.86 0) (unit 1)
-    (in_bom yes) (on_board yes) (dnp no) (fields_autoplaced)
-    (property "Reference" "IC102" (at 155.6259 130.81 0)
-      (effects (font (size 1.27 1.27)) (justify left))
-    )
-    (property "Value" "74HC273" (at 155.6259 133.35 0)
-      (effects (font (size 1.27 1.27)) (justify left))
-    )
-    (property "Footprint" "" (at 153.67 149.86 0)
-      (effects (font (size 1.27 1.27)) hide)
-    )
-    (property "Datasheet" "https://assets.nexperia.com/documents/data-sheet/74HC_HCT273.pdf" (at 153.67 149.86 0)
+  (symbol (lib_id "74xx:74HC273") (at 135.89 144.78 0) (unit 1)
+    (in_bom yes) (on_board yes) (dnp no) (fields_autoplaced)
+    (property "Reference" "IC102" (at 137.8459 125.73 0)
+      (effects (font (size 1.27 1.27)) (justify left))
+    )
+    (property "Value" "74HC273" (at 137.8459 128.27 0)
+      (effects (font (size 1.27 1.27)) (justify left))
+    )
+    (property "Footprint" "" (at 135.89 144.78 0)
+      (effects (font (size 1.27 1.27)) hide)
+    )
+    (property "Datasheet" "https://assets.nexperia.com/documents/data-sheet/74HC_HCT273.pdf" (at 135.89 144.78 0)
       (effects (font (size 1.27 1.27)) hide)
     )
@@
         (path "/5081f4fb-0c92-4cfc-8c52-39777c6d96ed"
           (reference "IC2") (unit 1)
+        )
+      )
+    )
+  )
+  (symbol (lib_id "TC7W139F:TC7W139F") (at 173.99 149.86 180) (unit 1)
+    (in_bom yes) (on_board yes) (dnp no) (fields_autoplaced)
+    (property "Reference" "IC11" (at 167.64 133.35 0)
+      (effects (font (size 1.27 1.27)))
+    )
+    (property "Value" "TC7W139" (at 167.64 135.89 0)
+      (effects (font (size 1.27 1.27)))
+    )
+    (property "Footprint" "Package_SO:SOP-8_3.76x4.96mm_P1.27mm" (at 160.02 160.02 0)
+      (effects (font (size 1.27 1.27)) hide)
+    )
+    (property "Datasheet" "https://pdf1.alldatasheet.com/datasheet-pdf/view/32066/TOSHIBA/TC7W139F.html" (at 168.91 156.21 0)
+      (effects (font (size 1.27 1.27)) hide)
+    )
+    (pin "1")
+    (pin "2")
+    (pin "3")
+    (pin "4")
+    (pin "5")
+    (pin "6")
+    (pin "7")
+    (pin "8")
+    (instances
+      (project "reverse-wanwan"
+        (path "/5081f4fb-0c92-4cfc-8c52-39777c6d96ed"
+          (reference "IC11") (unit 1)
         )
       )
@@
         )
       )
+    )
+  )
+  (symbol (lib_id "Device:R_Small") (at 233.68 133.35 90) (unit 1)
+    (in_bom yes) (on_board yes) (dnp no) (fields_autoplaced)
+    (property "Reference" "R103" (at 233.68 130.81 90)
+      (effects (font (size 1.27 1.27)))
+    )
+    (property "Value" "R_Small" (at 233.68 130.81 90)
+      (effects (font (size 1.27 1.27)) hide)
+    )
+    (property "Footprint" "" (at 233.68 133.35 0)
+      (effects (font (size 1.27 1.27)) hide)
+    )
+    (property "Datasheet" "~" (at 233.68 133.35 0)
+      (effects (font (size 1.27 1.27)) hide)
+    )
+    (pin "1")
+    (pin "2")
+    (instances
+      (project "reverse-wanwan"
+        (path "/5081f4fb-0c92-4cfc-8c52-39777c6d96ed"
+          (reference "R103") (unit 1)
+        )
+      )

Commit message: Revise pin descriptions for oki sound chip
Parts:
- IC101: symbol LOOPY_PCM:OKI_M6653A -> LOOPY_PCM:OKI_M6653A_ALT
Connections:
- net AOSC renamed ACMD
- net ARND renamed AST
- net ATST renamed ACH
- net AXT renamed ANAR
Other:
- moved on the sheet: C101, C107, C108, C109, C110, C111, C112, C113, IC101, IC102, IC106, IC11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
