File: pcb/singlerom-4Mtest-kasami/singlerom-4Mtest-kasami.kicad_pcb (KiCad board)
At the start: 2 copper layers, 96.3 x 75.2 mm, 38 parts, among them J2 PWR Breakout, SW1 SW_DIP_x04, U1 AS6C6264-55SCN, U2 MX29LV160DBTI-70G, U4 Pi Pico, U5 TCA9539PWR

Commit message: Minor fix idk
Routing:
- net VCC: track 406.0 -> 397.9 mm
Changed lines of the file:
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@@
   (segment (start 151.5 87.7) (end 150.8 87.7) (width 0.5) (layer "B.Cu") (net 84))
   (segment (start 181.840812 115.95) (end 184.65 113.140812) (width 0.75) (layer "B.Cu") (net 84))
-  (segment (start 104.8 118.17868) (end 107.68934 115.28934) (width 0.75) (layer "B.Cu") (net 84))
   (segment (start 153.8 62.5) (end 192 62.5) (width 0.75) (layer "B.Cu") (net 84))
   (segment (start 184.65 109.240812) (end 186.4 107.5) (width 0.75) (layer "B.Cu") (net 84))
@@
   (segment (start 195.5 66) (end 195.5 96.5) (width 0.75) (layer "B.Cu") (net 84))
   (segment (start 126.8 129.2) (end 126.8 132.1) (width 0.75) (layer "B.Cu") (net 84))
-  (segment (start 188.3 105.3) (end 188.3 101.365) (width 0.75) (layer "B.Cu") (net 84))
   (segment (start 162.940812 115.95) (end 181.840812 115.95) (width 0.75) (layer "B.Cu") (net 84))
   (segment (start 193.9 132) (end 194 132.1) (width 0.75) (layer "B.Cu") (net 84))
