File: pcb/flash-32mbit/flash-32mbit.kicad_pcb (KiCad board)
At the start: 2 copper layers, 96.3 x 76.2 mm, 28 parts, among them U1 IS62C256AL-45ULI, U2 SN74LVC1G04, U3 RP2040-Tiny, U4 LH28F320SKTD-L70, U5 MCP23S17-E/SO, U6 MCP23S17-E/SO, U7 MCP23S17-E/SO

Commit message: Moves components out of keepout areas, RESET no longer connected
Parts:
- D1: value BAV70LT1G -> BAT54C
- R6: value 1.2K -> 1K
- moved BT1 39.0 mm to (146.7, 77.3), turned to 180 degrees
- moved C1 5.89 mm to (118.5, 94.1)
- moved D1 5.89 mm to (119.6, 89.7)
- moved R2 4.73 mm to (138.6, 125.1), turned to 180 degrees
- moved R6 2.74 mm to (123.0, 89.6), turned to 90 degrees
- moved R1 2.00 mm to (134.0, 125.1)
Connections:
- D1 pad 1: VCC -> Net-(D1-Pad1)
- D1 pad 2: Net-(D1-A-Pad2) -> VCC
- R6 pad 1: Net-(D1-A-Pad2) -> Net-(D1-Pad1)
- U7 pad 8: /RESET -> unconnected-(U7-GPB7-Pad8)
Routing:
- net /RESET: track 99.0 -> 0.00 mm, vias 2 -> 0
- net +BATT: track 30.8 -> 21.3 mm, vias 1 -> 3
- net /~{INSERTED}: track 179.4 -> 184.6 mm, vias 9 -> 7
- net Net-(D1-A-Pad2): track 3.47 -> 0.00 mm
- net GND: track 87.4 -> 90.9 mm
- net Net-(D1-Pad1): track 0.00 -> 3.23 mm
- net /F61: track 5.91 -> 8.25 mm
- net Net-(U1-VDD): track 10.6 -> 12.8 mm
- net /F16: track 7.96 -> 9.52 mm

Commit message: Gives each expander its own CS line (help bus interference?)
Parts:
- removed C3: 0.1u, Capacitor_SMD:C_0805_2012Metric_Pad1.18x1.45mm_HandSolder
- moved C2 2.35 mm to (138.0, 121.8)
Connections:
- U3 pad 5: /SPI_CS -> /MCPD_CS
- U3 pad 6: /ROMSTS -> /MCPA0_CS
- U3 pad 7: unconnected-(U3-GP7-Pad7) -> /MCPA1_CS
- U3 pad 8: unconnected-(U3-GP8-Pad8) -> /ROMSTS
- U5 pad 11: /SPI_CS -> /MCPD_CS
- U6 pad 11: /SPI_CS -> /MCPA0_CS
- U7 pad 11: /SPI_CS -> /MCPA1_CS
Routing:
- net /SPI_CS: track 83.3 -> 0.00 mm, vias 2 -> 0
- net /MCPD_CS: track 0.00 -> 62.2 mm
- net /MCPA0_CS: track 0.00 -> 48.1 mm, vias 0 -> 1
- net /MCPA1_CS: track 0.00 -> 28.0 mm
- net VCC: track 137.5 -> 144.7 mm, vias 9 -> 10
- net /ROMSTS: track 32.0 -> 25.2 mm, vias 1 -> 0
- net GND: track 90.9 -> 84.7 mm, vias 24 -> 22

Commit message: checkpoint
Parts:
- added R10: 2K2, Resistor_SMD:R_0805_2012Metric_Pad1.20x1.40mm_HandSolder, F.Cu at (111.1, 110.7)
- added R11: 1K, Resistor_SMD:R_0805_2012Metric_Pad1.20x1.40mm_HandSolder, F.Cu at (111.1, 113.6)
- added R12: 2K2, Resistor_SMD:R_0805_2012Metric_Pad1.20x1.40mm_HandSolder, F.Cu at (111.1, 116.5)
- added R13: 0R, Resistor_SMD:R_0805_2012Metric_Pad1.20x1.40mm_HandSolder, F.Cu at (104.5, 62.4)
- added R9: 1K, Resistor_SMD:R_0805_2012Metric_Pad1.20x1.40mm_HandSolder, F.Cu at (111.7, 120.6)
Connections:
- J1 pad 1: VCC -> +5V
- J1 pad 17: unconnected-(J1-PB9-Pad17) -> /TX_D0
- J1 pad 20: unconnected-(J1-PB8-Pad20) -> /RX_D0
- R8 pad 1: /~{INSERTED} -> VCC
- R8 pad 2: VCC -> /~{INSERTED}
- U3 pad 12: unconnected-(U3-GP12-Pad12) -> Net-(U3-GP12)
- U3 pad 13: unconnected-(U3-GP13-Pad13) -> Net-(U3-GP13)
- U3 pad 14: unconnected-(U3-GP14-Pad14) -> /~{INSERTED}
- U3 pad 22: unconnected-(U3-VBUS-Pad22) -> Net-(U3-VBUS)
Routing:
- net +5V: track 0.00 -> 73.9 mm
- net /~{INSERTED}: track 184.9 -> 257.7 mm
- net VCC: track 144.7 -> 124.9 mm, vias 10 -> 8
- net Net-(U3-VBUS): track 0.00 -> 5.40 mm
- net GND: track 84.7 -> 86.0 mm

Commit message: checkpoint - routed uart0
Parts:
- moved R8 80.0 mm to (109.3, 124.8), turned to -90 degrees
- moved R9 32.5 mm to (116.1, 88.4), turned to -90 degrees
- moved R11 26.4 mm to (118.8, 88.4), turned to -90 degrees
- moved R12 25.2 mm to (118.8, 92.6), turned to -90 degrees
- moved R10 18.7 mm to (116.1, 92.6), turned to -90 degrees
- moved R2 16.9 mm to (123.0, 118.5), turned to -90 degrees
- moved R1 14.8 mm to (120.7, 118.5), turned to -90 degrees
- moved R7 8.50 mm to (111.9, 124.8)
- moved C1 7.63 mm to (125.9, 96.1)
- moved R6 4.64 mm to (126.9, 92.1)
- moved D1 4.64 mm to (123.5, 92.2)
- moved R5 1.88 mm to (125.1, 118.5), turned to -90 degrees
Connections:
- J1 pad 13: /~{INSERTED} -> GND
- J1 pad 47: GND -> /~{INSERTED}
Routing:
- net /~{INSERTED}: track 257.7 -> 58.9 mm, vias 7 -> 2
- net /RX_D0: track 0.00 -> 77.7 mm, vias 0 -> 2
- net /TX_D0: track 0.00 -> 69.6 mm, vias 0 -> 2
- net VCC: track 124.9 -> 156.1 mm, vias 8 -> 11
- net /F61: track 8.25 -> 22.2 mm, vias 1 -> 3
- net GND: track 86.0 -> 98.9 mm, vias 22 -> 25
- net /F16: track 9.52 -> 21.9 mm, vias 0 -> 2
- net Net-(U3-GP12): track 0.00 -> 8.23 mm
- net Net-(U3-GP13): track 0.00 -> 8.16 mm
- net Net-(U1-VDD): track 12.8 -> 7.28 mm
- net /ROMCE: track 92.9 -> 95.7 mm
- net +BATT: track 21.3 -> 19.8 mm
- net /3V3: track 110.3 -> 109.5 mm
- net /RAMWE: track 75.0 -> 74.4 mm

Commit message: Connects two serial ports from Loopy
Parts:
- added R14: 1K, Resistor_SMD:R_0805_2012Metric_Pad1.20x1.40mm_HandSolder, F.Cu at (121.4, 88.4)
- added R15: 2K2, Resistor_SMD:R_0805_2012Metric_Pad1.20x1.40mm_HandSolder, F.Cu at (121.4, 92.6)
- added R16: 1K, Resistor_SMD:R_0805_2012Metric_Pad1.20x1.40mm_HandSolder, F.Cu at (124.0, 88.4)
- added R17: 2K2, Resistor_SMD:R_0805_2012Metric_Pad1.20x1.40mm_HandSolder, F.Cu at (124.0, 92.6)
- moved D1 3.50 mm to (127.0, 92.2)
- moved R6 3.50 mm to (130.4, 92.2)
- moved R5 0.36 mm to (125.3, 118.8)
- moved R1 0.30 mm to (120.7, 118.8)
- moved R2 0.30 mm to (123.0, 118.8)
Connections:
- net Net-(U3-GP12) renamed /UART0_TX
- net Net-(U3-GP13) renamed /UART0_RX
- J1 pad 18: unconnected-(J1-PB10-Pad18) -> /RX_D1
- J1 pad 19: unconnected-(J1-PB11-Pad19) -> /TX_D1
- U3 pad 8: /ROMSTS -> /UART1_TX
- U3 pad 9: unconnected-(U3-GP9-Pad9) -> /UART1_RX
Routing:
- net /~{INSERTED}: track 58.9 -> 204.7 mm, vias 2 -> 5
- net /RX_D1: track 0.00 -> 78.7 mm, vias 0 -> 2
- net /TX_D1: track 0.00 -> 78.5 mm, vias 0 -> 2
- net /ROMSTS: track 25.2 -> 0.00 mm
- net /UART1_TX: track 0.00 -> 7.28 mm
- net /UART1_RX: track 0.00 -> 7.25 mm
- net GND: track 98.9 -> 94.9 mm, vias 25 -> 27
- net VCC: track 156.1 -> 152.8 mm, vias 11 -> 9
- net /MCPA0_CS: track 48.1 -> 50.7 mm
- net /RX_D0: track 77.7 -> 75.4 mm
- net Net-(U1-VDD): track 7.28 -> 5.49 mm
- net /A18: track 128.4 -> 126.7 mm
- net /F61: track 22.2 -> 23.8 mm
- net +BATT: track 19.8 -> 18.3 mm
- net /TX_D0: track 69.6 -> 68.6 mm
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
Commit message: Indicates optional dev-only components
Routing:
- net GND: track 94.9 -> 93.3 mm
Other:
- board text added: "MIDI"
- board text added: "SERIAL"
Changed lines of the file:
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@@
         (effects (font (size 1 1) (thickness 0.15)))
     )
-    (fp_text value "0R" (at 0 -1.7) (layer "F.SilkS")
+    (fp_text value "0R" (at 0.7 -2.3) (layer "F.SilkS")
         (effects (font (size 1 1) (thickness 0.15)))
     )
@@
     )
     (stroke (width 0) (type solid)) (fill solid) (layer "B.SilkS"))
+  (gr_rect (start 102.5 61.1) (end 106.5 63.6)
+    (stroke (width 0.15) (type dot)) (fill none) (layer "F.SilkS"))
+  (gr_rect (start 114.8 86.2) (end 125.2 94.7)
+    (stroke (width 0.15) (type dot)) (fill none) (layer "F.SilkS"))
   (gr_poly
     (pts
@@
     (effects (font (size 1 1) (thickness 0.15)) (justify left bottom mirror))
   )
+  (gr_text "SERIAL" (at 117.5 85.9) (layer "F.SilkS")
+    (effects (font (size 0.8 0.8) (thickness 0.15)) (justify bottom))
+  )
   (gr_text "JLCJLCJLCJLC" (at 117.7 61.3) (layer "F.SilkS")
     (effects (font (size 0.8 0.8) (thickness 0.15)) (justify bottom))
   )
+  (gr_text "MIDI" (at 122.7 85.9) (layer "F.SilkS")
+    (effects (font (size 0.8 0.8) (thickness 0.15)) (justify bottom))
+  )
   (segment (start 165.771141 113.5745) (end 165.196641 113) (width 0.25) (layer "F.Cu") (net 1))
   (segment (start 141.923653 113) (end 138.85 116.073653) (width 0.25) (layer "F.Cu") (net 1))
@@
   (segment (start 140.643767 95.443767) (end 140.35 95.737534) (width 0.25) (layer "F.Cu") (net 16))
   (segment (start 146.846575 126.5) (end 146.9 126.446575) (width 0.5) (layer "F.Cu") (net 16))
-  (segment (start 142.45 124.9375) (end 142.45 126.5) (width 0.5) (layer "F.Cu") (net 16))
   (segment (start 196.6 130.65) (end 196.6 127.2) (width 0.5) (layer "F.Cu") (net 16))
   (segment (start 193.925 76.215) (end 193.925 78.755) (width 0.5) (layer "F.Cu") (net 16))
@@
   (via (at 137.7 83.3) (size 0.8) (drill 0.4) (layers "F.Cu" "B.Cu") (free) (net 16))
   (via (at 151.86 78.399) (size 0.6) (drill 0.4) (layers "F.Cu" "B.Cu") (net 16))
-  (via (at 142.45 126.5) (size 0.8) (drill 0.4) (layers "F.Cu" "B.Cu") (net 16))
+  (via (at 142.45 124.9375) (size 0.8) (drill 0.4) (layers "F.Cu" "B.Cu") (net 16))
   (via (at 146.9 126.446575) (size 0.8) (drill 0.4) (layers "F.Cu" "B.Cu") (net 16))
   (via (at 146.35 115.6) (size 0.6) (drill 0.4) (layers "F.Cu" "B.Cu") (net 16))
@@
   (via (at 138 120.7625) (size 0.8) (drill 0.4) (layers "F.Cu" "B.Cu") (net 55))
   (via (at 127.3 128.55) (size 0.8) (drill 0.4) (layers "F.Cu" "B.Cu") (net 55))
-  (via (at 120.7 117.5) (size 0.8) (drill 0.4) (layers "F.Cu" "B.Cu") (net 55))
+  (via (at 120.7 117.8) (size 0.8) (drill 0.4) (layers "F.Cu" "B.Cu") (net 55))
   (via (at 144 119.15) (size 0.6) (drill 0.4) (layers "F.Cu" "B.Cu") (net 55))
   (via (at 170.95 77.5) (size 0.8) (drill 0.4) (layers "F.Cu" "B.Cu") (net 55))

Commit message: checkpoint
Parts:
- removed R13: 0R, Resistor_SMD:R_0805_2012Metric_Pad1.20x1.40mm_HandSolder
- turned D2 to 180 degrees
- turned R8 to 90 degrees
Connections:
- J1 pad 1: +5V -> VCC
- U3 pad 22: Net-(U3-VBUS) -> unconnected-(U3-VBUS-Pad22)
Routing:
- net +5V: track 73.9 -> 0.00 mm
- net Net-(U3-VBUS): track 5.70 -> 0.00 mm
- net VCC: track 152.8 -> 157.8 mm
- net /3V3: track 109.5 -> 106.4 mm, vias 3 -> 5
- net /~{INSERTED}: track 204.7 -> 203.7 mm, vias 5 -> 4
