File: pcb/flash-32mbit/flash-32mbit.kicad_pcb (KiCad board)
At the start: 2 copper layers, 96.3 x 76.2 mm, 35 parts, among them U1 IS62C256AL-45ULI, U2 SN74LVC1G04, U3 RP2040-Tiny, U4 LH28F320SKTD-L70, U5 MCP23S17-E/SO, U6 MCP23S17-E/SO, U7 MCP23S17-E/SO

Commit message: Reverts powering pico from loopy
Parts:
- moved R8 0.43 mm to (109.7, 124.6)
- moved R7 0.20 mm to (111.9, 124.6)
Routing:
- net VCC: track 157.8 -> 226.2 mm, vias 9 -> 7
- net GND: track 93.3 -> 111.7 mm, vias 27 -> 28
- net +BATT: track 18.3 -> 15.4 mm, vias 3 -> 1
- net /3V3: track 106.4 -> 108.0 mm

Commit message: rev6 RC
Parts:
- removed R14, R16: 1K, Resistor_SMD:R_0805_2012Metric_Pad1.20x1.40mm_HandSolder
- removed R15, R17: 2K2, Resistor_SMD:R_0805_2012Metric_Pad1.20x1.40mm_HandSolder
- moved R4 20.6 mm to (130.4, 97.1)
- moved R3 4.05 mm to (134.4, 92.2), turned to 90 degrees
Connections:
- R4 pad 2: VCC -> Net-(U1-VDD)
- U3 pad 8: /UART1_TX -> unconnected-(U3-GP8-Pad8)
- U3 pad 9: /UART1_RX -> unconnected-(U3-GP9-Pad9)
Routing:
- net /RX_D1: track 78.7 -> 0.00 mm, vias 2 -> 0
- net /TX_D1: track 78.5 -> 0.00 mm, vias 2 -> 0
- net /RAMCE: track 91.9 -> 78.5 mm, vias 3 -> 4
- net /UART1_TX: track 7.28 -> 0.00 mm
- net /UART1_RX: track 7.25 -> 0.00 mm
- net Net-(U1-VDD): track 5.49 -> 8.96 mm
- net /ROMWE: track 33.4 -> 32.5 mm, vias 2 -> 3
- net VCC: track 226.2 -> 226.8 mm
- net GND: vias 28 -> 26
Other:
- board text removed: "MIDI"
- board text removed: "SERIAL"

Commit message: Nudges to increase flood volume
Routing:
- net VCC: track 226.8 -> 204.5 mm
- net GND: track 111.7 -> 92.6 mm, vias 26 -> 27
- net /RX_D0: track 75.4 -> 76.3 mm

Commit message: Rev7 hardware changes: new SRAM part
Parts:
- removed the U1 at (121.3, 106.9)
- added R13: 100K, Resistor_SMD:R_0805_2012Metric_Pad1.20x1.40mm_HandSolder, F.Cu at (127.5, 118.8)
- added U2: AS6C1008-55SIN, LOOPY_SRAM:SOIC127P1410X300-32N, F.Cu at (120.2, 105.7)
- R6: value 1K -> 1K2
- moved R4 29.1 mm to (111.9, 119.6), turned to -90 degrees
- moved R6 2.60 mm to (130.4, 89.6)
- moved C1 2.60 mm to (125.9, 93.5)
- moved D1 2.60 mm to (127.0, 89.7)
- renumbered U4 to U1, U2 to U3, U3 to U4
Connections:
- BT1 pad 1: GND -> +BATT
- BT1 pad 2: +BATT -> GND
- C1 pad 2: Net-(U1-VDD) -> /VCC_OR_BATT
- D1 pad 3: Net-(U1-VDD) -> /VCC_OR_BATT
- J1 pad 18: /RX_D1 -> unconnected-(J1-PB10-Pad18)
- J1 pad 19: /TX_D1 -> unconnected-(J1-PB11-Pad19)
- J1 pad 60: /CLK -> unconnected-(J1-CLK-Pad60)
- R4 pad 1: /RAMCE -> GND
- R4 pad 2: Net-(U1-VDD) -> /RESET
- U1 pad 53: /ROMSTS -> unconnected-(U1-STS-Pad53)
Routing:
- net /RESET: track 0.00 -> 113.9 mm, vias 0 -> 2
- net /A16: track 119.4 -> 173.1 mm, vias 2 -> 3
- net /A15: track 95.7 -> 135.0 mm, vias 3 -> 4
- net VCC: track 204.5 -> 224.6 mm, vias 7 -> 8
- net Net-(U1-VDD): track 8.96 -> 0.00 mm
- net /VCC_OR_BATT: track 0.00 -> 5.67 mm
- net /RAMCE: track 78.5 -> 82.2 mm
- net /D0: track 168.5 -> 170.6 mm
- net /D2: track 177.2 -> 179.3 mm
- net /A7: track 144.1 -> 146.2 mm
- net /A5: track 143.1 -> 145.2 mm
- net /A0: track 137.8 -> 139.9 mm
- net /A3: track 151.4 -> 153.5 mm
- net /D1: track 172.4 -> 174.5 mm
- net /A14: track 143.2 -> 145.2 mm
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Other:
- board text added: "REV${REVISION}"

Commit message: Remove redundant pullups?
Parts:
- removed R13: 100K, Resistor_SMD:R_0805_2012Metric_Pad1.20x1.40mm_HandSolder
Connections:
- net /VCC_OR_BATT renamed /RAMVDD
- R4 pad 1: GND -> VCC
Routing:
- net /RAMCE: track 82.2 -> 76.6 mm, vias 4 -> 3
- net GND: vias 28 -> 27
Changed lines of the file:
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@@
   (net 109 "/MCPA0_CS")
   (net 110 "/MCPA1_CS")
-  (net 111 "/VCC_OR_BATT")
+  (net 111 "/RAMVDD")
   (net 112 "unconnected-(U1-A0-Pad32)")
   (net 113 "unconnected-(U1-NC-Pad30)")
@@
       (net 13 "/A15") (pinfunction "A15") (pintype "passive"))
     (pad "32" smd rect (at 6.613 -9.525 90) (size 0.7 1.924) (layers "F.Cu" "F.Paste" "F.Mask")
-      (net 111 "/VCC_OR_BATT") (pinfunction "VCC") (pintype "passive"))
+      (net 111 "/RAMVDD") (pinfunction "VCC") (pintype "passive"))
     (model "${KIPRJMOD}/Libraries/LOOPY_SRAM/AS6C1008-55SIN.stp"
       (offset (xyz 0 0 0))
@@
     (property "Sheetfile" "flash-32mbit.kicad_sch")
     (property "Sheetname" "")
-    (property "ki_description" "Unpolarized capacitor")
-    (property "ki_keywords" "cap capacitor")
+    (property "ki_description" "Unpolarized capacitor, small symbol")
+    (property "ki_keywords" "capacitor cap")
     (attr smd)
     (fp_text reference "C1" (at -3.2 0) (layer "F.SilkS") hide
@@
       (net 16 "GND") (pintype "passive"))
     (pad "2" smd roundrect (at 1.0375 0) (size 1.175 1.45) (layers "F.Cu" "F.Paste" "F.Mask") (roundrect_rratio 0.2127659574)
-      (net 111 "/VCC_OR_BATT") (pintype "passive"))
+      (net 111 "/RAMVDD") (pintype "passive"))
     (model "${KICAD6_3DMODEL_DIR}/Capacitor_SMD.3dshapes/C_0805_2012Metric.wrl"
       (offset (xyz 0 0 0))
@@
     )
   )
-  (footprint "Resistor_SMD:R_0805_2012Metric_Pad1.20x1.40mm_HandSolder" (layer "F.Cu")
-    (at 127.5 118.8 -90)
-    (descr "Resistor SMD 0805 (2012 Metric), square (rectangular) end terminal, IPC_7351 nominal with elongated pad for handsoldering. (Body size source: IPC-SM-782 page 72, https://www.pcb-3d.com/wordpress/wp-content/uploads/ipc-sm-782a_amendment_1_and_2.pdf), generated with kicad-footprint-generator")
-    (tags "resistor handsolder")
-    (property "Sheetfile" "flash-32mbit.kicad_sch")
-    (property "Sheetname" "")
-    (property "ki_description" "Resistor")
-    (property "ki_keywords" "R res resistor")
-    (attr smd)
-    (fp_text reference "R13" (at 0 -1.65 90) (layer "F.SilkS") hide
-        (effects (font (size 1 1) (thickness 0.15)))
-    )
-    (fp_text value "100K" (at 4.2 0 90) (layer "F.SilkS")
-        (effects (font (size 1 1) (thickness 0.15)))
-    )
-    (fp_text user "${REFERENCE}" (at 0 0 90) (layer "F.Fab")
-        (effects (font (size 0.5 0.5) (thickness 0.08)))
-    )
-    (fp_line (start -0.227064 -0.735) (end 0.227064 -0.735)
-      (stroke (width 0.12) (type solid)) (layer "F.SilkS"))
-    (fp_line (start -0.227064 0.735) (end 0.227064 0.735)
-      (stroke (width 0.12) (type solid)) (layer "F.SilkS"))
-    (fp_line (start -1.85 -0.95) (end 1.85 -0.95)
-      (stroke (width 0.05) (type solid)) (layer "F.CrtYd"))
-    (fp_line (start -1.85 0.95) (end -1.85 -0.95)
-      (stroke (width 0.05) (type solid)) (layer "F.CrtYd"))
-    (fp_line (start 1.85 -0.95) (end 1.85 0.95)
-      (stroke (width 0.05) (type solid)) (layer "F.CrtYd"))
-    (fp_line (start 1.85 0.95) (end -1.85 0.95)
-      (stroke (width 0.05) (type solid)) (layer "F.CrtYd"))
-    (fp_line (start -1 -0.625) (end 1 -0.625)
-      (stroke (width 0.1) (type solid)) (layer "F.Fab"))
-    (fp_line (start -1 0.625) (end -1 -0.625)
-      (stroke (width 0.1) (type solid)) (layer "F.Fab"))
-    (fp_line (start 1 -0.625) (end 1 0.625)
-      (stroke (width 0.1) (type solid)) (layer "F.Fab"))
-    (fp_line (start 1 0.625) (end -1 0.625)
-      (stroke (width 0.1) (type solid)) (layer "F.Fab"))
-    (pad "1" smd roundrect (at -1 0 270) (size 1.2 1.4) (layers "F.Cu" "F.Paste" "F.Mask") (roundrect_rratio 0.2083333333)
-      (net 55 "VCC") (pintype "passive"))
-    (pad "2" smd roundrect (at 1 0 270) (size 1.2 1.4) (layers "F.Cu" "F.Paste" "F.Mask") (roundrect_rratio 0.2083333333)
-      (net 61 "/RAMCE") (pintype "passive"))
-    (model "${KICAD6_3DMODEL_DIR}/Resistor_SMD.3dshapes/R_0805_2012Metric.wrl"
-      (offset (xyz 0 0 0))
-      (scale (xyz 1 1 1))
-      (rotate (xyz 0 0 0))
-    )
-  )
   (footprint "Capacitor_SMD:C_0805_2012Metric_Pad1.18x1.45mm_HandSolder" (layer "F.Cu")
     (at 181.1 73.65 180)
@@
       (stroke (width 0.1) (type solid)) (layer "F.Fab"))
     (pad "1" smd roundrect (at -1 0 270) (size 1.2 1.4) (layers "F.Cu" "F.Paste" "F.Mask") (roundrect_rratio 0.2083333333)
-      (net 16 "GND") (pintype "passive"))
+      (net 55 "VCC") (pintype "passive"))
     (pad "2" smd roundrect (at 1 0 270) (size 1.2 1.4) (layers "F.Cu" "F.Paste" "F.Mask") (roundrect_rratio 0.2083333333)
       (net 77 "/RESET") (pintype "passive"))
@@
       (net 55 "VCC") (pintype "passive"))
     (pad "3" smd roundrect (at 0.9375 0 270) (size 1.475 0.6) (layers "F.Cu" "F.Paste" "F.Mask") (roundrect_rratio 0.25)
-      (net 111 "/VCC_OR_BATT") (pintype "passive"))
+      (net 111 "/RAMVDD") (pintype "passive"))
     (model "${KICAD6_3DMODEL_DIR}/Package_TO_SOT_SMD.3dshapes/SOT-23.wrl"
       (offset (xyz 0 0 0))
@@
     (fp_line (start 10.7315 8.191498) (end 10.7315 -8.1915)
       (stroke (width 0.15) (type solid)) (layer "B.Fab"))
-    (pad "" smd rect (at -10.984999 -0.673099 180) (size 1.27 5.08) (layers "B.Cu" "B.Paste" "B.Mask")
-      (pinfunction "+") (pintype "passive"))
+    (pad "" smd rect (at -10.984999 -0.673099 180) (size 1.27 5.08) (layers "B.Cu" "B.Paste" "B.Mask"))
     (pad "1" smd rect (at 10.984999 -0.6731 180) (size 1.27 5.08) (layers "B.Cu" "B.Paste" "B.Mask")
       (net 56 "+BATT") (pinfunction "+") (pintype "passive"))
@@
   (segment (start 125.2 128.4) (end 125.2 128.260049) (width 0.25) (layer "B.Cu") (net 14))
   (segment (start 133 120.46005) (end 133 74.3) (width 0.25) (layer "B.Cu") (net 14))
-  (segment (start 131.6 117.55) (end 129.75 117.55) (width 0.25) (layer "F.Cu") (net 15))
-  (segment (start 126.3 118.8) (end 125.3 119.8) (width 0.25) (layer "F.Cu") (net 15))
-  (segment (start 134.0245 115.1755) (end 131.65 117.55) (width 0.25) (layer "F.Cu") (net 15))
-  (segment (start 135.35 115.1755) (end 134.0245 115.1755) (width 0.25) (layer "F.Cu") (net 15))
-  (segment (start 128.5 118.8) (end 126.3 118.8) (width 0.25) (layer "F.Cu") (net 15))
+  (segment (start 134.558814 115.1755) (end 135.35 115.1755) (width 0.25) (layer "F.Cu") (net 15))
+  (segment (start 133.55 116.2) (end 133.55 116.184314) (width 0.25) (layer "F.Cu") (net 15))
+  (segment (start 131.6 118.25) (end 130 118.25) (width 0.25) (layer "F.Cu") (net 15))
+  (segment (start 131.6 118.25) (end 131.6 118.15) (width 0.25) (layer "F.Cu") (net 15))
+  (segment (start 125.35 119.75) (end 125.3 119.8) (width 0.25) (layer "F.Cu") (net 15))
   (segment (start 142.85 115.6) (end 142.85 117.084) (width 0.25) (layer "F.Cu") (net 15))
   (segment (start 142.9 115.55) (end 142.85 115.6) (width 0.25) (layer "F.Cu") (net 15))
-  (segment (start 131.65 117.55) (end 131.6 117.55) (width 0.25) (layer "F.Cu") (net 15))
-  (segment (start 129.75 117.55) (end 128.5 118.8) (width 0.25) (layer "F.Cu") (net 15))
+  (segment (start 131.6 118.15) (end 133.55 116.2) (width 0.25) (layer "F.Cu") (net 15))
+  (segment (start 130 118.25) (end 128.5 119.75) (width 0.25) (layer "F.Cu") (net 15))
+  (segment (start 128.5 119.75) (end 125.35 119.75) (width 0.25) (layer "F.Cu") (net 15))
+  (segment (start 133.55 116.184314) (end 134.558814 115.1755) (width 0.25) (layer "F.Cu") (net 15))
   (via (at 140.43 72.525) (size 0.6) (drill 0.4) (layers "F.Cu" "B.Cu") (net 15))
   (via (at 135.35 115.1755) (size 0.6) (drill 0.4) (layers "F.Cu" "B.Cu") (net 15))
-  (via (at 131.6 117.55) (size 0.6) (drill 0.4) (layers "F.Cu" "B.Cu") (net 15))
+  (via (at 131.6 118.25) (size 0.6) (drill 0.4) (layers "F.Cu" "B.Cu") (net 15))
   (via (at 142.9 115.55) (size 0.6) (drill 0.4) (layers "F.Cu" "B.Cu") (net 15))
   (segment (start 139.205 71.3) (end 133.35 71.3) (width 0.25) (layer "B.Cu") (net 15))
@@
   (via (at 132.4 70.3) (size 0.8) (drill 0.4) (layers "F.Cu" "B.Cu") (net 16))
   (via (at 148.05 87.749) (size 0.6) (drill 0.4) (layers "F.Cu" "B.Cu") (net 16))
-  (via (at 111.9 118.6) (size 0.6) (drill 0.4) (layers "F.Cu" "B.Cu") (net 16))
   (via (at 113.5 116.215) (size 0.8) (drill 0.4) (layers "F.Cu" "B.Cu") (net 16))
   (via (at 140.643767 95.443767) (size 0.6) (drill 0.4) (layers "F.Cu" "B.Cu") (net 16))
@@
   (segment (start 135.715001 79.415001) (end 135.715001 77.9731) (width 0.4) (layer "B.Cu") (net 56))
   (segment (start 131.345 108.805) (end 132.3 107.85) (width 0.25) (layer "F.Cu") (net 61))
-  (segment (start 127.5 119.8) (end 128.065686 119.8) (width 0.25) (layer "F.Cu") (net 61))
-  (segment (start 129.665686 118.2) (end 131.907923 118.2) (width 0.25) (layer "F.Cu") (net 61))
-  (segment (start 128.065686 119.8) (end 129.665686 118.2) (width 0.25) (layer "F.Cu") (net 61))
   (segment (start 122.6 128.4) (end 121 130) (width 0.25) (layer "F.Cu") (net 61))
   (segment (start 121 130) (end 121 132.1) (width 0.25) (layer "F.Cu") (net 61))
-  (segment (start 131.907923 118.2) (end 132.305838 117.802085) (width 0.25) (layer "F.Cu") (net 61))
   (segment (start 126.965 108.805) (end 131.345 108.805) (width 0.25) (layer "F.Cu") (net 61))
   (via (at 122.6 128.4) (size 0.6) (drill 0.4) (layers "F.Cu" "B.Cu") (net 61))
   (via (at 137.89 72.525) (size 0.6) (drill 0.4) (layers "F.Cu" "B.Cu") (net 61))
   (via (at 132.3 107.85) (size 0.6) (drill 0.4) (layers "F.Cu" "B.Cu") (net 61))
-  (via (at 132.305838 117.802085) (size 0.6) (drill 0.4) (layers "F.Cu" "B.Cu") (net 61))
   (segment (start 132.3 73.2) (end 133.6 71.9) (width 0.25) (layer "B.Cu") (net 61))
   (segment (start 137.265 71.9) (end 137.89 72.525) (width 0.25) (layer "B.Cu") (net 61))

Commit message: Tidying, using RESET to power down flash, marking potentially redundant pullups
Parts:
- turned R1 to 90 degrees
Connections:
- R1 pad 1: VCC -> /F61
- R1 pad 2: /F61 -> VCC
- U1 pad 16: VCC -> /RESET
Routing:
- net /RESET: track 113.9 -> 124.3 mm, vias 2 -> 4
- net VCC: track 224.6 -> 221.9 mm, vias 8 -> 7

Commit message: Now that asserting RESET low keeps some things safe, let pico drive RESET high only when ready
Parts:
- removed R4: 100K, Resistor_SMD:R_0805_2012Metric_Pad1.20x1.40mm_HandSolder
- added R13: 100K, Resistor_SMD:R_0805_2012Metric_Pad1.20x1.40mm_HandSolder, F.Cu at (127.6, 118.8)
- moved C4 2.73 mm to (140.7, 121.8)
- moved U3 0.65 mm to (134.6, 120.7)
Connections:
- U7 pad 6: unconnected-(U7-GPB5-Pad6) -> /RESET
Routing:
- net /RESET: track 124.3 -> 165.3 mm, vias 4 -> 5
- net GND: track 92.6 -> 101.6 mm
- net /RAMWE: track 74.4 -> 80.5 mm, vias 3 -> 4
- net /A21: track 138.6 -> 136.1 mm
- net VCC: track 221.9 -> 223.1 mm, vias 7 -> 6
- net /3V3: track 108.3 -> 107.2 mm
