File: pcb/flash-32mbit/flash-32mbit.kicad_pcb (KiCad board)
At the start: 2 copper layers, 96.3 x 76.2 mm, 31 parts, among them U1 LH28F320SKTD-L70, U2 AS6C1008-55SIN, U3 SN74LVC1G04, U4 RP2040-Tiny, U5 MCP23S17-E/SO, U6 MCP23S17-E/SO, U7 MCP23S17-E/SO

Commit message: /RESET pulled low, power up and down conditions should be covered by this and extra control pullups should be redundant
Parts:
- added R4: 100K, Resistor_SMD:R_0805_2012Metric_Pad1.20x1.40mm_HandSolder, F.Cu at (111.9, 119.6)
Routing:
- net GND: vias 27 -> 28
Changed lines of the file:
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@@
   (title_block
     (title "Floopy Drive")
-    (date "2023-09-27")
+    (date "2023-09-28")
     (rev "7")
     (company "@partlyhuman")
@@
     (property "ki_keywords" "R resistor")
     (attr smd)
-    (fp_text reference "R13" (at 0 -1.65 90) (layer "F.SilkS")
+    (fp_text reference "R13" (at 0 -1.65 90) (layer "F.SilkS") hide
         (effects (font (size 1 1) (thickness 0.15)))
     )
-    (fp_text value "100K" (at 0 1.65 90) (layer "F.Fab")
+    (fp_text value "100K" (at 4.2 0 90) (layer "F.SilkS")
         (effects (font (size 1 1) (thickness 0.15)))
     )
@@
     (fp_line (start 1 0.625) (end -1 0.625)
       (stroke (width 0.1) (type solid)) (layer "F.Fab"))
-    (pad "1" smd roundrect (at -1 0 270) (size 1.2 1.4) (layers "F.Cu" "F.Paste" "F.Mask") (roundrect_rratio 0.208333)
+    (pad "1" smd roundrect (at -1 0 270) (size 1.2 1.4) (layers "F.Cu" "F.Paste" "F.Mask") (roundrect_rratio 0.2083333333)
       (net 55 "VCC") (pintype "passive"))
-    (pad "2" smd roundrect (at 1 0 270) (size 1.2 1.4) (layers "F.Cu" "F.Paste" "F.Mask") (roundrect_rratio 0.208333)
+    (pad "2" smd roundrect (at 1 0 270) (size 1.2 1.4) (layers "F.Cu" "F.Paste" "F.Mask") (roundrect_rratio 0.2083333333)
       (net 14 "/RAMWE") (pintype "passive"))
     (model "${KICAD6_3DMODEL_DIR}/Resistor_SMD.3dshapes/R_0805_2012Metric.wrl"
@@
   )
   (footprint "Resistor_SMD:R_0805_2012Metric_Pad1.20x1.40mm_HandSolder" (layer "F.Cu")
+    (at 111.9 119.6 90)
+    (descr "Resistor SMD 0805 (2012 Metric), square (rectangular) end terminal, IPC_7351 nominal with elongated pad for handsoldering. (Body size source: IPC-SM-782 page 72, https://www.pcb-3d.com/wordpress/wp-content/uploads/ipc-sm-782a_amendment_1_and_2.pdf), generated with kicad-footprint-generator")
+    (tags "resistor handsolder")
+    (property "Sheetfile" "flash-32mbit.kicad_sch")
+    (property "Sheetname" "")
+    (property "ki_description" "Resistor, small symbol")
+    (property "ki_keywords" "R resistor")
+    (attr smd)
+    (fp_text reference "R4" (at 0 -1.65 90) (layer "F.SilkS") hide
+        (effects (font (size 1 1) (thickness 0.15)))
+    )
+    (fp_text value "100K" (at 0 2.1 90) (layer "F.SilkS")
+        (effects (font (size 1 1) (thickness 0.15)))
+    )
+    (fp_text user "${REFERENCE}" (at 0 0 90) (layer "F.Fab")
+        (effects (font (size 0.5 0.5) (thickness 0.08)))
+    )
+    (fp_line (start -0.227064 -0.735) (end 0.227064 -0.735)
+      (stroke (width 0.12) (type solid)) (layer "F.SilkS"))
+    (fp_line (start -0.227064 0.735) (end 0.227064 0.735)
+      (stroke (width 0.12) (type solid)) (layer "F.SilkS"))
+    (fp_line (start -1.85 -0.95) (end 1.85 -0.95)
+      (stroke (width 0.05) (type solid)) (layer "F.CrtYd"))
+    (fp_line (start -1.85 0.95) (end -1.85 -0.95)
+      (stroke (width 0.05) (type solid)) (layer "F.CrtYd"))
+    (fp_line (start 1.85 -0.95) (end 1.85 0.95)
+      (stroke (width 0.05) (type solid)) (layer "F.CrtYd"))
+    (fp_line (start 1.85 0.95) (end -1.85 0.95)
+      (stroke (width 0.05) (type solid)) (layer "F.CrtYd"))
+    (fp_line (start -1 -0.625) (end 1 -0.625)
+      (stroke (width 0.1) (type solid)) (layer "F.Fab"))
+    (fp_line (start -1 0.625) (end -1 -0.625)
+      (stroke (width 0.1) (type solid)) (layer "F.Fab"))
+    (fp_line (start 1 -0.625) (end 1 0.625)
+      (stroke (width 0.1) (type solid)) (layer "F.Fab"))
+    (fp_line (start 1 0.625) (end -1 0.625)
+      (stroke (width 0.1) (type solid)) (layer "F.Fab"))
+    (pad "1" smd roundrect (at -1 0 90) (size 1.2 1.4) (layers "F.Cu" "F.Paste" "F.Mask") (roundrect_rratio 0.2083333333)
+      (net 77 "/RESET") (pintype "passive"))
+    (pad "2" smd roundrect (at 1 0 90) (size 1.2 1.4) (layers "F.Cu" "F.Paste" "F.Mask") (roundrect_rratio 0.2083333333)
+      (net 16 "GND") (pintype "passive"))
+    (model "${KICAD6_3DMODEL_DIR}/Resistor_SMD.3dshapes/R_0805_2012Metric.wrl"
+      (offset (xyz 0 0 0))
+      (scale (xyz 1 1 1))
+      (rotate (xyz 0 0 0))
+    )
+  )
+  (footprint "Resistor_SMD:R_0805_2012Metric_Pad1.20x1.40mm_HandSolder" (layer "F.Cu")
     (at 125.3 118.8 -90)
     (descr "Resistor SMD 0805 (2012 Metric), square (rectangular) end terminal, IPC_7351 nominal with elongated pad for handsoldering. (Body size source: IPC-SM-782 page 72, https://www.pcb-3d.com/wordpress/wp-content/uploads/ipc-sm-782a_amendment_1_and_2.pdf), generated with kicad-footprint-generator")
@@
   (via (at 148.1 126) (size 0.8) (drill 0.4) (layers "F.Cu" "B.Cu") (net 16))
   (via (at 120.05 64.15) (size 0.8) (drill 0.4) (layers "F.Cu" "B.Cu") (net 16))
+  (via (at 111.9 118.6) (size 0.6) (drill 0.4) (layers "F.Cu" "B.Cu") (net 16))
   (via (at 146.35 115.6) (size 0.6) (drill 0.4) (layers "F.Cu" "B.Cu") (net 16))
   (via (at 138 122.8375) (size 0.6) (drill 0.4) (layers "F.Cu" "B.Cu") (net 16))
@@
   (segment (start 149.3 67.886827) (end 153.8 72.386827) (width 0.25) (layer "B.Cu") (net 72))
   (segment (start 155 75) (end 155 77.1) (width 0.25) (layer "B.Cu") (net 72))
-  (segment (start 111.9 120.8) (end 111.9 120.6) (width 0.25) (layer "F.Cu") (net 77))
-  (segment (start 135.562744 128) (end 142.9 128) (width 0.25) (layer "F.Cu") (net 77))
   (segment (start 143.85 118.55) (end 143.85 117.084) (width 0.25) (layer "F.Cu") (net 77))
-  (segment (start 177.5 132.775) (end 177.5 127.7) (width 0.25) (layer "F.Cu") (net 77))
-  (segment (start 144.2 118.9) (end 143.85 118.55) (width 0.25) (layer "F.Cu") (net 77))
   (segment (start 111.9 120.6) (end 116.8 120.6) (width 0.25) (layer "F.Cu") (net 77))
   (segment (start 125.219045 124.2) (end 131.762744 124.2) (width 0.25) (layer "F.Cu") (net 77))
+  (segment (start 111.9 120.8) (end 111.9 120.6) (width 0.25) (layer "F.Cu") (net 77))
+  (segment (start 119.9505 123.7505) (end 124.769545 123.7505) (width 0.25) (layer "F.Cu") (net 77))
   (segment (start 131.762744 124.2) (end 135.562744 128) (width 0.25) (layer "F.Cu") (net 77))
+  (segment (start 135.562744 128) (end 142.9 128) (width 0.25) (layer "F.Cu") (net 77))
+  (segment (start 177.5 132.775) (end 177.5 127.7) (width 0.25) (layer "F.Cu") (net 77))
+  (segment (start 142.9 128) (end 145.575 125.325) (width 0.25) (layer "F.Cu") (net 77))
+  (segment (start 124.769545 123.7505) (end 125.219045 124.2) (width 0.25) (layer "F.Cu") (net 77))
+  (segment (start 144.2 118.9) (end 143.85 118.55) (width 0.25) (layer "F.Cu") (net 77))
   (segment (start 116.8 120.6) (end 119.9505 123.7505) (width 0.25) (layer "F.Cu") (net 77))
   (segment (start 148.379595 125.325) (end 145.75 125.325) (width 0.25) (layer "F.Cu") (net 77))
@@
   (segment (start 149.029595 125.975) (end 148.379595 125.325) (width 0.25) (layer "F.Cu") (net 77))
   (segment (start 175.775 125.975) (end 149.029595 125.975) (width 0.25) (layer "F.Cu") (net 77))
-  (segment (start 119.9505 123.7505) (end 124.769545 123.7505) (width 0.25) (layer "F.Cu") (net 77))
-  (segment (start 124.769545 123.7505) (end 125.219045 124.2) (width 0.25) (layer "F.Cu") (net 77))
-  (segment (start 142.9 128) (end 145.575 125.325) (width 0.25) (layer "F.Cu") (net 77))
   (segment (start 177.5 127.7) (end 175.775 125.975) (width 0.25) (layer "F.Cu") (net 77))
   (via (at 142.97 72.525) (size 0.6) (drill 0.4) (layers "F.Cu" "B.Cu") (net 77))
@@
   (via (at 144.2 118.9) (size 0.6) (drill 0.4) (layers "F.Cu" "B.Cu") (net 77))
   (via (at 126.763 98.665) (size 0.6) (drill 0.4) (layers "F.Cu" "B.Cu") (net 77))
-  (segment (start 126.728 98.7) (end 111.95 98.7) (width 0.25) (layer "B.Cu") (net 77))
+  (segment (start 111.95 98.7) (end 126.728 98.7) (width 0.25) (layer "B.Cu") (net 77))
   (segment (start 145.975 121.438173) (end 144.7 122.713173) (width 0.25) (layer "B.Cu") (net 77))
   (segment (start 144.7 122.713173) (end 144.7 124.275) (width 0.25) (layer "B.Cu") (net 77))
-  (segment (start 110.5 100.15) (end 110.5 119.2) (width 0.25) (layer "B.Cu") (net 77))
-  (segment (start 111.95 98.7) (end 110.5 100.15) (width 0.25) (layer "B.Cu") (net 77))
   (segment (start 141.545 71.1) (end 132.625305 71.1) (width 0.25) (layer "B.Cu") (net 77))
   (segment (start 142.97 72.525) (end 141.545 71.1) (width 0.25) (layer "B.Cu") (net 77))
+  (segment (start 110.5 100.15) (end 111.95 98.7) (width 0.25) (layer "B.Cu") (net 77))
   (segment (start 132.625305 71.1) (end 130.8 72.925305) (width 0.25) (layer "B.Cu") (net 77))
   (segment (start 144.7 124.275) (end 145.75 125.325) (width 0.25) (layer "B.Cu") (net 77))
-  (segment (start 126.763 98.665) (end 126.728 98.7) (width 0.25) (layer "B.Cu") (net 77))
   (segment (start 145.975 120.151167) (end 145.975 121.438173) (width 0.25) (layer "B.Cu") (net 77))
   (segment (start 130.8 94.628) (end 126.763 98.665) (width 0.25) (layer "B.Cu") (net 77))
-  (segment (start 110.5 119.2) (end 111.9 120.6) (width 0.25) (layer "B.Cu") (net 77))
+  (segment (start 126.728 98.7) (end 126.763 98.665) (width 0.25) (layer "B.Cu") (net 77))
+  (segment (start 111.9 120.6) (end 110.5 119.2) (width 0.25) (layer "B.Cu") (net 77))
   (segment (start 144.723833 118.9) (end 145.975 120.151167) (width 0.25) (layer "B.Cu") (net 77))
   (segment (start 144.2 118.9) (end 144.723833 118.9) (width 0.25) (layer "B.Cu") (net 77))
+  (segment (start 110.5 119.2) (end 110.5 100.15) (width 0.25) (layer "B.Cu") (net 77))
   (segment (start 130.8 72.925305) (end 130.8 94.628) (width 0.25) (layer "B.Cu") (net 77))
   (segment (start 124.887673 125) (end 131.43137 125) (width 0.25) (layer "F.Cu") (net 81))
