File: pcb/flash-32mbit/flash-32mbit.kicad_pcb (KiCad board)
At the start: 2 copper layers, 96.3 x 76.2 mm, 32 parts, among them U1 LH28F320SKTD-L70, U2 AS6C1008-55SIN, U3 SN74LVC1G04, U4 RP2040-Tiny, U5 MCP23S17-E/SO, U6 MCP23S17-E/SO, U7 MCP23S17-E/SO

Commit message: Rev8 changes mostly to serial
Parts:
- added D3: BSS138, Package_TO_SOT_SMD:SOT-23, F.Cu at (123.2, 87.3)
- added R14: 100K, Resistor_SMD:R_0805_2012Metric_Pad1.20x1.40mm_HandSolder, F.Cu at (127.6, 118.8)
- R11: value 1K -> 100K
- R13: value 100K -> 1K
- moved R13 27.2 mm to (122.0, 92.2)
- moved R10 5.36 mm to (115.3, 87.3), turned to 90 degrees
- moved R6 4.39 mm to (129.5, 85.3)
- moved R9 3.88 mm to (115.3, 92.2)
- moved D1 1.66 mm to (128.6, 90.1)
- moved R11 1.10 mm to (118.9, 87.3), turned to 90 degrees
- moved R12 0.41 mm to (118.9, 92.2), turned to 90 degrees
Connections:
- net /3V3 renamed +3V3
- R10 pad 1: /TX_D0 -> /UART0_RX
- R11 pad 1: /UART0_TX -> GND
- R11 pad 2: /RX_D0 -> /UART0_TX
- R12 pad 1: /RX_D0 -> VCC
- R12 pad 2: GND -> Net-(D3-D)
- R13 pad 1: VCC -> Net-(D3-D)
- R13 pad 2: /RAMWE -> /RX_D0
Routing:
- net +3V3: track 107.2 -> 128.6 mm, vias 5 -> 6
- net Net-(D3-D): track 0.00 -> 6.56 mm
- net /UART0_RX: track 8.16 -> 11.8 mm
- net /TX_D0: track 68.3 -> 64.8 mm
- net /UART0_TX: track 8.23 -> 11.2 mm
- net /~{INSERTED}: track 203.8 -> 205.0 mm
- net +BATT: track 14.4 -> 13.2 mm

Commit message: Micro minor tweaks
Parts:
- moved C1 2.10 mm to (128.0, 93.1), turned to 180 degrees
- moved R13 1.20 mm to (123.2, 92.2)
- moved D1 0.60 mm to (128.6, 89.5)
- moved R6 0.60 mm to (129.5, 84.7)
- moved R10 0.10 mm to (115.2, 87.3)
- moved R9 0.10 mm to (115.2, 92.2)
Routing:
- net /RX_D0: track 76.7 -> 77.9 mm
- net Net-(D3-D): track 6.56 -> 7.26 mm
- net Net-(D1-Pad1): track 2.81 -> 2.21 mm
- net /RAMVDD: track 5.89 -> 6.49 mm

Commit message: Firewall VCC fill from pins
Parts:
- removed R14: 100K, Resistor_SMD:R_0805_2012Metric_Pad1.20x1.40mm_HandSolder
- added D4: BAT54C, Package_TO_SOT_SMD:SOT-23, F.Cu at (193.3, 124.6)
- added D5: BAT54C, Package_TO_SOT_SMD:SOT-23, F.Cu at (106.4, 124.6)
- R1: value 1K -> 1K2
- R6: value 1K2 -> 1K
- moved R6 42.9 mm to (140.4, 126.2), turned to 0 degrees
- moved R1 35.0 mm to (129.5, 84.9)
- moved R2 13.4 mm to (134.2, 126.2), turned to 180 degrees
- moved R5 2.38 mm to (127.5, 117.9), turned to 0 degrees
- moved U3 1.00 mm to (134.5, 121.7), turned to 0 degrees
- turned R8 to -90 degrees
Connections:
- net /RAMVDD renamed VMEM
- J1 pad 1: VCC -> +5V
- J1 pad 14: VCC -> +5V
- J1 pad 29: VCC -> +5V
- J1 pad 57: VCC -> +5V
- J1 pad 89: VCC -> +5V
- R1 pad 1: /F61 -> Net-(D1-Pad1)
- R1 pad 2: VCC -> +BATT
- R2 pad 1: VCC -> /F16
- R2 pad 2: /F16 -> +5V
- R6 pad 1: Net-(D1-Pad1) -> /F61
- R6 pad 2: +BATT -> +5V
Routing:
- net +5V: track 0.00 -> 129.3 mm, vias 0 -> 5
- net VCC: track 223.1 -> 116.0 mm, vias 6 -> 2
- net /F16: track 22.7 -> 7.26 mm, vias 2 -> 0
- net /F61: track 23.9 -> 9.95 mm, vias 3 -> 1
- net /RAMWE: track 80.5 -> 74.4 mm, vias 4 -> 3
- net GND: track 101.6 -> 97.0 mm, vias 28 -> 27
- net /ROMCE: track 95.1 -> 91.1 mm
- net /A21: track 136.1 -> 139.5 mm, vias 3 -> 5
- net /RX_D0: track 77.9 -> 80.4 mm
- net /TX_D0: track 64.8 -> 66.9 mm
- net +3V3: track 128.6 -> 130.4 mm
- net /RESET: track 165.3 -> 163.6 mm, vias 5 -> 7
- net /~{INSERTED}: track 205.0 -> 203.9 mm, vias 4 -> 6
- net /~{A21}: track 6.92 -> 6.33 mm, vias 0 -> 2

Commit message: Cleaning up REV8 design
Parts:
- added R14: 100K, Resistor_SMD:R_0805_2012Metric_Pad1.20x1.40mm_HandSolder, F.Cu at (131.8, 92.2)
- moved D5 1.70 mm to (108.1, 124.6)
- moved R7 1.70 mm to (113.6, 124.6)
- moved R8 1.60 mm to (111.3, 124.6)
- moved D4 1.30 mm to (192.0, 124.6)
Routing:
- net GND: track 97.0 -> 106.2 mm
- net VMEM: track 6.49 -> 10.0 mm
- net /RAMWE: track 74.4 -> 77.0 mm, vias 3 -> 4
- net /~{INSERTED}: track 203.9 -> 206.2 mm
- net /RESET: track 163.6 -> 161.6 mm
- net /A19: track 127.1 -> 128.1 mm
- net +5V: track 129.3 -> 128.3 mm
- net /RAMCE: track 76.6 -> 77.4 mm
- net VCC: track 116.0 -> 116.5 mm

Commit message: Consolidating blocker diodes and using higher current PMEG2005CT
Parts:
- removed D4, D5: BAT54C, Package_TO_SOT_SMD:SOT-23
- removed R7: 100K, Resistor_SMD:R_0805_2012Metric_Pad1.20x1.40mm_HandSolder
- D2: value BAT54C -> PMEG2005CT_215; footprint Package_TO_SOT_SMD:SOT-23 -> Package_TO_SOT_SMD:SOT-23-3
- moved D2 58.4 mm to (112.2, 124.3), turned to 90 degrees
- moved R4 11.9 mm to (123.3, 123.1), turned to 180 degrees
- moved R8 2.72 mm to (108.6, 124.3)
Connections:
- D2 pad 1: +3V3 -> +5V
Routing:
- net VCC: track 116.5 -> 56.7 mm
- net /RESET: track 161.6 -> 137.7 mm
- net /RX_D0: track 80.4 -> 66.1 mm
- net +5V: track 128.3 -> 123.3 mm
- net /TX_D0: track 66.9 -> 68.6 mm
- net /~{INSERTED}: track 206.2 -> 204.9 mm, vias 6 -> 4
- net +3V3: track 130.6 -> 130.0 mm, vias 6 -> 5
- net GND: track 106.2 -> 105.9 mm, vias 27 -> 26

Commit message: Rev9 minor change that moves F16/F61 pullups far away from edge connector
Parts:
- R12: value 2K2 -> 10K
- moved R6 21.4 mm to (119.2, 123.4), turned to 90 degrees
- moved R2 13.3 mm to (121.2, 123.4), turned to 90 degrees
- moved R4 4.21 mm to (120.2, 120.2)
- moved D2 3.61 mm to (115.8, 124.0)
- moved C2 0.20 mm to (138.2, 121.8)
Connections:
- D2 pad 1: +5V -> +3V3
- D2 pad 2: +3V3 -> +5V
Routing:
- net /F16: track 7.26 -> 20.9 mm
- net /F61: track 9.98 -> 22.0 mm
- net /RESET: track 137.7 -> 141.7 mm
- net +5V: track 123.3 -> 125.4 mm, vias 5 -> 4
- net /RX_D0: track 66.1 -> 64.6 mm
- net +3V3: track 130.0 -> 130.2 mm, vias 5 -> 6

Commit message: Widens battery solder pads
Parts:
- moved BT1 1.10 mm to (147.6, 77.9)
Routing:
- net +BATT: track 13.0 -> 10.7 mm
- net /A7: track 146.3 -> 148.3 mm
- net GND: track 106.2 -> 104.3 mm
Changed lines of the file:
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@@
   (title_block
     (title "Floopy Drive")
-    (date "2023-12-09")
+    (date "2024-01-16")
     (rev "9")
     (company "@partlyhuman")
@@
   )
   (footprint "LOOPY_Cart:Keystone-3034TR-MFG" (layer "B.Cu")
-    (at 146.7 77.3 180)
+    (at 147.6 77.925 180)
     (property "Notes" "")
     (property "Sheetfile" "flash-32mbit.kicad_sch")
@@
         (effects (font (size 1.27 1.27) (thickness 0.15)) (justify mirror))
     )
-    (fp_line (start -13 -0.67) (end -12 -0.67)
+    (fp_line (start -12.2 3.199999) (end -11.2 3.199999)
       (stroke (width 0.15) (type solid)) (layer "B.SilkS"))
-    (fp_line (start -12.5 -0.169999) (end -12.5 -1.17)
+    (fp_line (start -11.7 3.7) (end -11.7 2.699999)
       (stroke (width 0.15) (type solid)) (layer "B.SilkS"))
     (fp_line (start -10.73 -3.6) (end -10.73 -5.185)
@@
     (fp_line (start 10.73 4.189999) (end 10.73 2.3)
       (stroke (width 0.15) (type solid)) (layer "B.SilkS"))
-    (fp_line (start -11.644999 -8.2165) (end 11.644999 -8.2165)
+    (fp_line (start -12.9 -8.232998) (end 12.7 -8.2)
       (stroke (width 0.15) (type solid)) (layer "B.CrtYd"))
-    (fp_line (start -11.644999 8.216498) (end -11.644999 -8.2165)
+    (fp_line (start -12.9 8.2) (end -12.9 -8.232998)
       (stroke (width 0.15) (type solid)) (layer "B.CrtYd"))
-    (fp_line (start 11.644999 -8.2165) (end 11.644999 8.216498)
+    (fp_line (start 12.7 -8.2) (end 12.7 8.232998)
       (stroke (width 0.15) (type solid)) (layer "B.CrtYd"))
-    (fp_line (start 11.644999 8.216498) (end -11.644999 8.216498)
-      (stroke (width 0.15) (type solid)) (layer "B.CrtYd"))
-    (fp_line (start 11.644999 8.216498) (end 11.644999 8.216498)
+    (fp_line (start 12.7 8.232998) (end -12.9 8.2)
       (stroke (width 0.15) (type solid)) (layer "B.CrtYd"))
     (fp_line (start -10.7315 -8.1915) (end -10.7315 8.191498)
@@
     (fp_line (start 10.7315 8.191498) (end 10.7315 -8.1915)
       (stroke (width 0.15) (type solid)) (layer "B.Fab"))
-    (pad "" smd rect (at -10.984999 -0.673099 180) (size 1.27 5.08) (layers "B.Cu" "B.Paste" "B.Mask"))
-    (pad "1" smd rect (at 10.984999 -0.6731 180) (size 1.27 5.08) (layers "B.Cu" "B.Paste" "B.Mask")
+    (pad "" smd rect (at -11.374999 -0.673098 180) (size 2 5.079998) (layers "B.Cu" "B.Paste" "B.Mask"))
+    (pad "1" smd rect (at 11.524999 -0.65655 180) (size 2 5.1131) (layers "B.Cu" "B.Paste" "B.Mask")
       (net 56 "+BATT") (pinfunction "+") (pintype "passive"))
     (pad "2" smd rect (at 0 -0.673099 180) (size 3.9624 3.9624) (layers "B.Cu" "B.Mask")
@@
   (segment (start 163.831233 61.968767) (end 163.85 61.987534) (width 0.25) (layer "B.Cu") (net 2))
   (segment (start 125.63 101.83) (end 125.005 101.205) (width 0.25) (layer "F.Cu") (net 3))
-  (segment (start 139.119 75.3) (end 136.62 77.799) (width 0.25) (layer "F.Cu") (net 3))
   (segment (start 146.85 117.084) (end 146.85 118.291403) (width 0.25) (layer "F.Cu") (net 3))
-  (segment (start 159.425 75.3) (end 139.119 75.3) (width 0.25) (layer "F.Cu") (net 3))
+  (segment (start 159.4505 75.2995) (end 139.823815 75.2995) (width 0.25) (layer "F.Cu") (net 3))
   (segment (start 146.85 118.291403) (end 148.808598 120.25) (width 0.25) (layer "F.Cu") (net 3))
   (segment (start 159.4245 101.65) (end 128.18 101.65) (width 0.25) (layer "F.Cu") (net 3))
-  (segment (start 159.65 75.075) (end 159.425 75.3) (width 0.25) (layer "F.Cu") (net 3))
   (segment (start 125.005 101.205) (end 113.537 101.205) (width 0.25) (layer "F.Cu") (net 3))
+  (segment (start 139.823815 75.2995) (end 139.823315 75.3) (width 0.25) (layer "F.Cu") (net 3))
   (segment (start 148.808598 120.25) (end 159.4755 120.25) (width 0.25) (layer "F.Cu") (net 3))
+  (segment (start 139.823315 75.3) (end 139.119 75.3) (width 0.25) (layer "F.Cu") (net 3))
   (segment (start 159.65 101.8755) (end 159.4245 101.65) (width 0.25) (layer "F.Cu") (net 3))
-  (segment (start 159.4755 120.25) (end 159.65 120.4245) (width 0.25) (layer "F.Cu") (net 3))
+  (segment (start 139.119 75.3) (end 136.62 77.799) (width 0.25) (layer "F.Cu") (net 3))
   (segment (start 136.62 77.799) (end 136.62 78.399) (width 0.25) (layer "F.Cu") (net 3))
+  (segment (start 159.4755 120.25) (end 159.65 120.4245) (width 0.25) (layer "F.Cu") (net 3))
+  (segment (start 160.3 74.45) (end 159.4505 75.2995) (width 0.25) (layer "F.Cu") (net 3))
   (segment (start 128 101.83) (end 125.63 101.83) (width 0.25) (layer "F.Cu") (net 3))
   (segment (start 128.18 101.65) (end 128 101.83) (width 0.25) (layer "F.Cu") (net 3))
   (via (at 159.65 101.8755) (size 0.6) (drill 0.4) (layers "F.Cu" "B.Cu") (net 3))
   (via (at 159.65 120.4245) (size 0.6) (drill 0.4) (layers "F.Cu" "B.Cu") (net 3))
-  (via (at 159.65 75.075) (size 0.6) (drill 0.4) (layers "F.Cu" "B.Cu") (net 3))
-  (segment (start 159.65 75.075) (end 159.65 120.762563) (width 0.25) (layer "B.Cu") (net 3))
+  (via (at 160.3 74.45) (size 0.6) (drill 0.4) (layers "F.Cu" "B.Cu") (net 3))
+  (segment (start 160.5 87.775) (end 159.65 88.625) (width 0.25) (layer "B.Cu") (net 3))
+  (segment (start 159.65 88.625) (end 159.65 120.762563) (width 0.25) (layer "B.Cu") (net 3))
   (segment (start 152.3 131.9) (end 152.5 132.1) (width 0.25) (layer "B.Cu") (net 3))
+  (segment (start 160.3 74.45) (end 160.5 74.65) (width 0.25) (layer "B.Cu") (net 3))
   (segment (start 152.3 128.112563) (end 152.3 131.9) (width 0.25) (layer "B.Cu") (net 3))
   (segment (start 159.65 120.762563) (end 152.3 128.112563) (width 0.25) (layer "B.Cu") (net 3))
+  (segment (start 160.5 74.65) (end 160.5 87.775) (width 0.25) (layer "B.Cu") (net 3))
   (segment (start 113.537 102.475) (end 124.875 102.475) (width 0.25) (layer "F.Cu") (net 4))
   (segment (start 154.4 129.45) (end 155.5 128.35) (width 0.25) (layer "F.Cu") (net 4))
@@
   (segment (start 164.9 131.9) (end 165.1 132.1) (width 0.5) (layer "B.Cu") (net 16))
   (segment (start 129.7 128.4) (end 129.750579 128.4) (width 0.5) (layer "B.Cu") (net 16))
-  (segment (start 148.05 76.623099) (end 146.7 77.973099) (width 0.5) (layer "B.Cu") (net 16))
   (segment (start 106.32 62.88) (end 106.3 62.9) (width 1) (layer "B.Cu") (net 16))
   (segment (start 165.5 127.2) (end 164.9 127.8) (width 0.5) (layer "B.Cu") (net 16))
@@
   (segment (start 129.6 83.8) (end 134.6 83.8) (width 0.5) (layer "F.Cu") (net 56))
   (via (at 135.7 82.7) (size 0.8) (drill 0.4) (layers "F.Cu" "B.Cu") (net 56))
-  (segment (start 135.7 82.7) (end 135.7 77.988101) (width 0.5) (layer "B.Cu") (net 56))
-  (segment (start 135.7 77.988101) (end 135.715001 77.9731) (width 0.5) (layer "B.Cu") (net 56))
-  (segment (start 135.8 79.5) (end 135.715001 79.415001) (width 0.4) (layer "B.Cu") (net 56))
-  (segment (start 135.715001 79.415001) (end 135.715001 77.9731) (width 0.4) (layer "B.Cu") (net 56))
+  (segment (start 135.7 82.7) (end 135.7 78.738101) (width 0.5) (layer "B.Cu") (net 56))
   (segment (start 120.8 129.1) (end 120.8 131.9) (width 0.25) (layer "F.Cu") (net 61))
   (segment (start 122.6 128.4) (end 121.5 128.4) (width 0.25) (layer "F.Cu") (net 61))
