File: pcb/flash-32mbit/flash-32mbit.kicad_sch (KiCad schematic)
At the start: 26 parts, among them U1 IS62C256AL-45ULI, U2 SN74LVC1G04, U3 RP2040-Tiny, U4 LH28F320SKTD-L70, U5 MCP23S17-E/SO, U6 MCP23S17-E/SO, U7 MCP23S17-E/SO

Commit message: Update to use @kasamikona's edge connector (renumbered to match)
Parts:
- J1: footprint LOOPY_Cart:LOOPY-Edge-Connector -> LOOPY_Cart:LOOPY_Cart_Edge
Changed lines of the file:
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@@
       (effects (font (size 1.27 1.27)))
     )
-    (property "Footprint" "LOOPY_Cart:LOOPY-Edge-Connector" (at 229.87 38.1 0)
+    (property "Footprint" "LOOPY_Cart:LOOPY_Cart_Edge" (at 229.87 38.1 0)
       (effects (font (size 1.27 1.27)) hide)
     )

Commit message: Moves components out of keepout areas, RESET no longer connected
Parts:
- removed D1: BAV70LT1G, Package_TO_SOT_SMD:SOT-23, symbol Diode:BAV70W
- added D1: BAT54C, Package_TO_SOT_SMD:SOT-23, symbol Diode:BAT54C
- R6: value 1.2K -> 1K
Connections:
- net RESET: no longer U7.8 (GPB7)
- net VCC: now also D1.2
- net at C1.2, U1.28 (VDD): now also D1.3
- net at R6.1: now also D1.1
- no-connect marks 46 -> 47
Changed lines of the file:
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@@
   (no_connect (at 218.44 91.44))
   (no_connect (at 241.3 106.68))
+  (no_connect (at 419.1 114.3))
   (no_connect (at 241.3 134.62))
   (no_connect (at 218.44 58.42))
@@
     (stroke (width 0) (type default))
   )
+  (wire (pts (xy 125.73 29.21) (xy 129.54 29.21))
+    (stroke (width 0) (type default))
+  )
   (wire (pts (xy 111.76 132.08) (xy 120.65 132.08))
     (stroke (width 0) (type default))
@@
   )
   (wire (pts (xy 208.28 142.24) (xy 218.44 142.24))
+    (stroke (width 0) (type default))
+  )
+  (wire (pts (xy 154.94 29.21) (xy 149.86 29.21))
     (stroke (width 0) (type default))
   )
@@
   (label "A11" (at 109.22 55.88 0) (fields_autoplaced)
     (effects (font (size 1.27 1.27)) (justify left bottom))
-  )
-  (label "RESET" (at 419.1 114.3 180) (fields_autoplaced)
-    (effects (font (size 1.27 1.27)) (justify right bottom))
   )
   (label "SPI_CLK" (at 358.14 124.46 180) (fields_autoplaced)
@@
       (effects (font (size 1.27 1.27)))
     )
-    (property "Value" "1.2K" (at 147.32 26.67 90)
+    (property "Value" "1K" (at 147.32 26.67 90)
       (effects (font (size 1.27 1.27)))
     )
@@
         (path "/5081f4fb-0c92-4cfc-8c52-39777c6d96ed"
           (reference "#PWR013") (unit 1)
-        )
-      )
-    )
-  )
-  (symbol (lib_id "Diode:BAV70W") (at 137.16 29.21 0) (unit 1)
-    (in_bom yes) (on_board yes) (dnp no)
-    (property "Reference" "D1" (at 137.16 22.86 0)
-      (effects (font (size 1.27 1.27)))
-    )
-    (property "Value" "BAV70LT1G" (at 137.16 25.4 0)
-      (effects (font (size 1.27 1.27)))
-    )
-    (property "Footprint" "Package_TO_SOT_SMD:SOT-23" (at 137.16 29.21 0)
-      (effects (font (size 1.27 1.27)) hide)
-    )
-    (property "Datasheet" "https://assets.nexperia.com/documents/data-sheet/BAV70_SER.pdf" (at 137.16 29.21 0)
-      (effects (font (size 1.27 1.27)) hide)
-    )
-    (property "Notes" "" (at 137.16 29.21 0)
-      (effects (font (size 1.27 1.27)))
-    )
-    (pin "1")
-    (pin "2")
-    (pin "3")
-    (instances
-      (project "flash-32mbit"
-        (path "/5081f4fb-0c92-4cfc-8c52-39777c6d96ed"
-          (reference "D1") (unit 1)
         )
       )
@@
     )
   )
+  (symbol (lib_id "Diode:BAT54C") (at 137.16 29.21 0) (mirror y) (unit 1)
+    (in_bom yes) (on_board yes) (dnp no) (fields_autoplaced)
+    (property "Reference" "D1" (at 137.16 22.86 0)
+      (effects (font (size 1.27 1.27)))
+    )
+    (property "Value" "BAT54C" (at 137.16 25.4 0)
+      (effects (font (size 1.27 1.27)))
+    )
+    (property "Footprint" "Package_TO_SOT_SMD:SOT-23" (at 135.255 26.035 0)
+      (effects (font (size 1.27 1.27)) (justify left) hide)
+    )
+    (property "Datasheet" "http://www.diodes.com/_files/datasheets/ds11005.pdf" (at 139.192 29.21 0)
+      (effects (font (size 1.27 1.27)) hide)
+    )
+    (pin "1")
+    (pin "2")
+    (pin "3")
+    (instances
+      (project "flash-32mbit"
+        (path "/5081f4fb-0c92-4cfc-8c52-39777c6d96ed"
+          (reference "D1") (unit 1)
+        )
+      )
+    )
+  )
   (symbol (lib_id "power:GND") (at 405.13 121.92 0) (unit 1)
     (in_bom yes) (on_board yes) (dnp no) (fields_autoplaced)
@@
     )
   )
-  (symbol (lib_id "power:VCC") (at 129.54 29.21 90) (unit 1)
-    (in_bom yes) (on_board yes) (dnp no) (fields_autoplaced)
-    (property "Reference" "#PWR04" (at 133.35 29.21 0)
-      (effects (font (size 1.27 1.27)) hide)
-    )
-    (property "Value" "VCC" (at 125.73 29.21 90)
-      (effects (font (size 1.27 1.27)) (justify left))
-    )
-    (property "Footprint" "" (at 129.54 29.21 0)
-      (effects (font (size 1.27 1.27)) hide)
-    )
-    (property "Datasheet" "" (at 129.54 29.21 0)
+  (symbol (lib_id "power:VCC") (at 125.73 29.21 0) (unit 1)
+    (in_bom yes) (on_board yes) (dnp no) (fields_autoplaced)
+    (property "Reference" "#PWR04" (at 125.73 33.02 0)
+      (effects (font (size 1.27 1.27)) hide)
+    )
+    (property "Value" "VCC" (at 125.73 24.13 0)
+      (effects (font (size 1.27 1.27)))
+    )
+    (property "Footprint" "" (at 125.73 29.21 0)
+      (effects (font (size 1.27 1.27)) hide)
+    )
+    (property "Datasheet" "" (at 125.73 29.21 0)
       (effects (font (size 1.27 1.27)) hide)
     )
@@
     )
   )
-  (symbol (lib_id "power:+BATT") (at 149.86 29.21 270) (unit 1)
-    (in_bom yes) (on_board yes) (dnp no) (fields_autoplaced)
-    (property "Reference" "#PWR011" (at 146.05 29.21 0)
-      (effects (font (size 1.27 1.27)) hide)
-    )
-    (property "Value" "+BATT" (at 153.67 29.21 90)
-      (effects (font (size 1.27 1.27)) (justify left))
-    )
-    (property "Footprint" "" (at 149.86 29.21 0)
-      (effects (font (size 1.27 1.27)) hide)
-    )
-    (property "Datasheet" "" (at 149.86 29.21 0)
-      (effects (font (size 1.27 1.27)) hide)
-    )
+  (symbol (lib_id "power:+BATT") (at 154.94 29.21 0) (unit 1)
+    (in_bom yes) (on_board yes) (dnp no) (fields_autoplaced)
+    (property "Reference" "#PWR011" (at 154.94 33.02 0)
+      (effects (font (size 1.27 1.27)) hide)
+    )
+    (property "Value" "+BATT" (at 154.94 24.13 0)
+      (effects (font (size 1.27 1.27)))
+    )
+    (property "Footprint" "" (at 154.94 29.21 0)
+      (effects (font (size 1.27 1.27)) hide)
+    )
+    (property "Datasheet" "" (at 154.94 29.21 0)
+      (effects (font (size 1.27 1.27)) hide)
+    )

Commit message: Gives each expander its own CS line (help bus interference?)
Parts:
- C3: now not fitted
Connections:
- net GND: no longer C3.2
- net ROMSTS: now also U3.8 (GP8); no longer U3.6 (GP6)
- net MCPA1_CS: now reaches U3.7 (GP7)
- net MCPA1_CS: now also U7.11 (~{CS})
- net SPI_CS renamed MCPD_CS
- net MCPD_CS: no longer U6.11 (~{CS}), U7.11 (~{CS})
- new net MCPA0_CS: U3.6 (GP6), U6.11 (~{CS})
- no-connect marks 47 -> 45
Other:
- note added: "Shares decoupling cap with neighbouring C2"
- note added: "mcpAddr0"
- note added: "mcpAddr1"
- note added: "mcpData"
- note removed: "Address1 IO (Address 0x1)"
- note removed: "Address2/Control IO (Address 0x2)"
- note removed: "Data IO (Address 0x0)"
Changed lines of the file:
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@@
   (junction (at 72.39 124.46) (diameter 0) (color 0 0 0 0)
-  )
-  (junction (at 97.79 208.28) (diameter 0) (color 0 0 0 0)
   )
   (junction (at 405.13 119.38) (diameter 0) (color 0 0 0 0)
@@
   (no_connect (at 358.14 55.88))
   (no_connect (at 218.44 83.82))
-  (no_connect (at 388.62 60.96))
   (no_connect (at 449.58 99.06))
   (no_connect (at 373.38 68.58))
@@
   (no_connect (at 241.3 134.62))
   (no_connect (at 218.44 58.42))
-  (no_connect (at 388.62 58.42))
   (no_connect (at 358.14 40.64))
   (no_connect (at 218.44 48.26))
@@
     (stroke (width 0) (type default))
   )
-  (wire (pts (xy 97.79 208.28) (xy 106.68 208.28))
-    (stroke (width 0) (type default))
-  )
   (wire (pts (xy 53.34 140.97) (xy 53.34 139.7))
     (stroke (width 0) (type default))
@@
     (stroke (width 0) (type default))
   )
-  (wire (pts (xy 97.79 208.28) (xy 97.79 204.47))
-    (stroke (width 0) (type default))
-  )
   (wire (pts (xy 129.54 124.46) (xy 129.54 125.73))
     (stroke (width 0) (type default))
@@
     (stroke (width 0) (type default))
   )
-  (wire (pts (xy 97.79 208.28) (xy 97.79 210.82))
+  (wire (pts (xy 97.79 204.47) (xy 97.79 210.82))
     (stroke (width 0) (type default))
   )
@@
     (effects (font (size 2.54 2.54)) (justify left bottom))
   )
+  (text "Shares decoupling cap with neighbouring C2" (at 106.68 213.36 0)
+    (effects (font (size 1.27 1.27)) (justify left bottom))
+  )
   (text "ROM" (at 50.8 95.25 0)
     (effects (font (size 2.54 2.54)) (justify left bottom))
@@
     (effects (font (size 2.54 2.54)) (justify left bottom))
   )
-  (text "Address1 IO\n(Address 0x1)" (at 363.22 137.16 0)
+  (text "mcpAddr0" (at 363.22 135.89 0)
     (effects (font (size 1.27 1.27)) (justify left bottom))
   )
@@
     (effects (font (size 1.27 1.27)) (justify left bottom))
   )
-  (text "Address2/Control IO\n(Address 0x2)" (at 424.18 137.16 0)
+  (text "mcpAddr1" (at 424.18 135.89 0)
     (effects (font (size 1.27 1.27)) (justify left bottom))
   )
@@
     (effects (font (size 2.54 2.54)) (justify left bottom))
   )
-  (text "Data IO\n(Address 0x0)" (at 302.26 137.16 0)
+  (text "mcpData" (at 302.26 135.89 0)
     (effects (font (size 1.27 1.27)) (justify left bottom))
   )
@@
     (effects (font (size 1.27 1.27)) (justify right bottom))
   )
-  (label "SPI_CS" (at 297.18 121.92 180) (fields_autoplaced)
+  (label "MCPD_CS" (at 297.18 121.92 180) (fields_autoplaced)
     (effects (font (size 1.27 1.27)) (justify right bottom))
   )
@@
     (effects (font (size 1.27 1.27)) (justify left bottom))
   )
+  (label "MCPA0_CS" (at 388.62 55.88 0) (fields_autoplaced)
+    (effects (font (size 1.27 1.27)) (justify left bottom))
+  )
   (label "SPI_CLK" (at 358.14 124.46 180) (fields_autoplaced)
     (effects (font (size 1.27 1.27)) (justify right bottom))
@@
     (effects (font (size 1.27 1.27)) (justify left bottom))
   )
+  (label "ROMSTS" (at 388.62 60.96 0) (fields_autoplaced)
+    (effects (font (size 1.27 1.27)) (justify left bottom))
+  )
   (label "D1" (at 251.46 63.5 180) (fields_autoplaced)
     (effects (font (size 1.27 1.27)) (justify right bottom))
@@
     (effects (font (size 1.27 1.27)) (justify left bottom))
   )
-  (label "SPI_CS" (at 419.1 121.92 180) (fields_autoplaced)
+  (label "MCPA1_CS" (at 419.1 121.92 180) (fields_autoplaced)
     (effects (font (size 1.27 1.27)) (justify right bottom))
   )
@@
     (effects (font (size 1.27 1.27)) (justify left bottom))
   )
-  (label "SPI_CS" (at 358.14 121.92 180) (fields_autoplaced)
+  (label "MCPA0_CS" (at 358.14 121.92 180) (fields_autoplaced)
     (effects (font (size 1.27 1.27)) (justify right bottom))
   )
@@
     (effects (font (size 1.27 1.27)) (justify right bottom))
   )
+  (label "MCPD_CS" (at 388.62 53.34 0) (fields_autoplaced)
+    (effects (font (size 1.27 1.27)) (justify left bottom))
+  )
   (label "A14" (at 77.47 129.54 0) (fields_autoplaced)
     (effects (font (size 1.27 1.27)) (justify left bottom))
@@
     (effects (font (size 1.27 1.27)) (justify left bottom))
   )
-  (label "SPI_CS" (at 388.62 53.34 0) (fields_autoplaced)
-    (effects (font (size 1.27 1.27)) (justify left bottom))
-  )
   (label "A11" (at 251.46 99.06 180) (fields_autoplaced)
     (effects (font (size 1.27 1.27)) (justify right bottom))
@@
     (effects (font (size 1.27 1.27)) (justify left bottom))
   )
-  (label "ROMSTS" (at 388.62 55.88 0) (fields_autoplaced)
-    (effects (font (size 1.27 1.27)) (justify left bottom))
-  )
   (label "~{INSERTED}" (at 388.62 121.92 0) (fields_autoplaced)
     (effects (font (size 1.27 1.27)) (justify left bottom))
@@
   )
   (label "A3" (at 77.47 167.64 0) (fields_autoplaced)
+    (effects (font (size 1.27 1.27)) (justify left bottom))
+  )
+  (label "MCPA1_CS" (at 388.62 58.42 0) (fields_autoplaced)
     (effects (font (size 1.27 1.27)) (justify left bottom))
   )
@@
   )
   (symbol (lib_id "Device:C_Small") (at 106.68 205.74 0) (unit 1)
-    (in_bom yes) (on_board yes) (dnp no) (fields_autoplaced)
+    (in_bom yes) (on_board no) (dnp yes) (fields_autoplaced)
     (property "Reference" "C3" (at 110.49 205.105 0)
       (effects (font (size 1.27 1.27)) (justify left))
@@
       (effects (font (size 1.27 1.27)) hide)
     )
-    (pin "1")
+    (property "Notes" "" (at 106.68 205.74 0)
+      (effects (font (size 1.27 1.27)))
+    )
+    (pin "1")

Commit message: checkpoint
Parts:
- added R10, R12: 2K2, Resistor_SMD:R_0805_2012Metric_Pad1.20x1.40mm_HandSolder, symbol Device:R
- added R11, R9: 1K, Resistor_SMD:R_0805_2012Metric_Pad1.20x1.40mm_HandSolder, symbol Device:R
- added R13: 0R, Resistor_SMD:R_0805_2012Metric_Pad1.20x1.40mm_HandSolder, symbol Device:R
Connections:
- net GND: now also R10.2, R12.2
- net VCC: now also R8.1; no longer J1.1 (+5V), R8.2
- net ~{INSERTED}: now also R8.2, U3.14 (GP14); no longer R8.1
- net TX_D0: now reaches J1.17 (PB9)
- net TX_D0: now also R10.1, R9.2
- net RX_D0: now reaches J1.20 (PB8)
- net RX_D0: now also R11.2, R12.1
- net at U3.12 (GP12): now also R11.1
- net at U3.13 (GP13): now also R9.1
- net at U3.22 (VBUS): now also R13.2
- new net +5V: J1.1 (+5V), R13.1
- no-connect marks 45 -> 39
Other:
- note added: "Inserted allows Pico to run a different program when connected to USB or Loopy for example, run a USB host and forward serial when connected to Loopy but run the flashing firmware when connected to USB"
- note added: "Power the Pico when inserted in Loopy for monitoring serial etc use the 0R as a jumper to enable this option uses one of the +5V from cart edge, not connected to VCC"
- note added: "Use one of the +5V pins, which are connected on the console side, to power Pico when inserted. When USB connected, this goes to nowhere."
- moved on the sheet: C5, C6, C7, D2, R8, U5, U6, U7

Commit message: checkpoint - routed uart0
Connections:
- net GND: now also J1.13 (GND); no longer J1.47 (GND)
- net ~{INSERTED}: now also J1.47 (GND); no longer J1.13 (GND)
Other:
- moved on the sheet: R1, R2, R8

Commit message: Connects two serial ports from Loopy
Parts:
- added R14, R16: 1K, Resistor_SMD:R_0805_2012Metric_Pad1.20x1.40mm_HandSolder, symbol Device:R
- added R15, R17: 2K2, Resistor_SMD:R_0805_2012Metric_Pad1.20x1.40mm_HandSolder, symbol Device:R
Connections:
- net GND: now also R15.2, R17.2
- net ROMSTS: no longer U3.8 (GP8)
- net UART0_TX: now reaches R11.1, U3.12 (GP12)
- net UART0_RX: now reaches R9.1, U3.13 (GP13)
- net RX_D1: now reaches J1.18 (PB10)
- net RX_D1: now also R16.2, R17.1
- net TX_D1: now reaches J1.19 (PB11)
- net TX_D1: now also R14.2, R15.1
- net UART1_RX: now reaches U3.9 (GP9)
- net UART1_RX: now also R14.1
- new net UART1_TX: R16.1, U3.8 (GP8)
- no-connect marks 39 -> 36
Other:
- note added: "Loopy UART D0 = available for brew D1 = MIDI"

Commit message: Indicates optional dev-only components
Other:
- note added: "Provide 3V power to board when plugged into USB Protect board from being powered when plugged into console or 5V entering 3.3V net when R13 populated"
- note removed: "Provide 3V power to board when plugged into USB Protect board from being powered when plugged into console"
- note removed: "TODO double check write protect behaviour"
Changed lines of the file:
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@@
     (effects (font (size 1.27 1.27)) (justify right bottom))
-  )
-  (text "TODO double check write protect behaviour" (at 146.05 96.52 0)
-    (effects (font (size 1.27 1.27)) (justify left bottom))
   )
   (text "Power the Pico when inserted in Loopy\nfor monitoring serial etc\nuse the 0R as a jumper to enable this option\nuses one of the +5V from cart edge, not connected to VCC"
@@
     (effects (font (size 1.27 1.27)) (justify left bottom))
   )
-  (text "Provide 3V power to board when plugged into USB\nProtect board from being powered when plugged into console"
+  (text "Provide 3V power to board when plugged into USB\nProtect board from being powered when plugged into console\nor 5V entering 3.3V net when R13 populated"
     (at 339.09 67.31 0)
     (effects (font (size 1.27 1.27)) (justify right bottom))

Commit message: checkpoint
Parts:
- removed R13: 0R, Resistor_SMD:R_0805_2012Metric_Pad1.20x1.40mm_HandSolder, symbol Device:R
Connections:
- net +5V is gone; now on net VCC: J1.1 (+5V)
- no-connect marks 36 -> 37
Other:
- note removed: "Power the Pico when inserted in Loopy for monitoring serial etc use the 0R as a jumper to enable this option uses one of the +5V from cart edge, not connected to VCC"
- note removed: "Use one of the +5V pins, which are connected on the console side, to power Pico when inserted. When USB connected, this goes to nowhere."
Changed lines of the file:
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@@
   (no_connect (at 419.1 157.48))
   (no_connect (at 241.3 134.62))
+  (no_connect (at 358.14 40.64))
   (no_connect (at 218.44 58.42))
   (no_connect (at 218.44 48.26))
@@
     (stroke (width 0) (type default))
   )
-  (wire (pts (xy 325.12 40.64) (xy 332.74 40.64))
-    (stroke (width 0) (type default))
-  )
   (wire (pts (xy 111.76 127) (xy 120.65 127))
     (stroke (width 0) (type default))
@@
     (stroke (width 0) (type default))
   )
-  (wire (pts (xy 340.36 40.64) (xy 358.14 40.64))
-    (stroke (width 0) (type default))
-  )
   (wire (pts (xy 124.46 132.08) (xy 124.46 137.16))
     (stroke (width 0) (type default))
@@
   )
   (wire (pts (xy 208.28 119.38) (xy 218.44 119.38))
-    (stroke (width 0) (type default))
-  )
-  (wire (pts (xy 325.12 36.83) (xy 325.12 40.64))
     (stroke (width 0) (type default))
   )
@@
   (text "Power SRAM from battery when disconnected\nPower SRAM from VCC when connected to pico (3.3V) or loopy (5V)\nPrevent VCC from charging battery"
     (at 110.49 27.94 0)
-    (effects (font (size 1.27 1.27)) (justify right bottom))
-  )
-  (text "Power the Pico when inserted in Loopy\nfor monitoring serial etc\nuse the 0R as a jumper to enable this option\nuses one of the +5V from cart edge, not connected to VCC"
-    (at 339.09 29.21 0)
-    (effects (font (size 1.27 1.27)) (justify right bottom))
-  )
-  (text "Use one of the +5V pins,\nwhich are connected on the console side,\nto power Pico when inserted.\nWhen USB connected, this goes to nowhere."
-    (at 196.85 40.64 0)
     (effects (font (size 1.27 1.27)) (justify right bottom))
   )
@@
         (path "/5081f4fb-0c92-4cfc-8c52-39777c6d96ed"
           (reference "#PWR015") (unit 1)
-        )
-      )
-    )
-  )
-  (symbol (lib_id "Device:R") (at 336.55 40.64 90) (unit 1)
-    (in_bom yes) (on_board yes) (dnp no)
-    (property "Reference" "R13" (at 336.55 34.29 90)
-      (effects (font (size 1.27 1.27)))
-    )
-    (property "Value" "0R" (at 336.55 36.83 90)
-      (effects (font (size 1.27 1.27)))
-    )
-    (property "Footprint" "Resistor_SMD:R_0805_2012Metric_Pad1.20x1.40mm_HandSolder" (at 336.55 42.418 90)
-      (effects (font (size 1.27 1.27)) hide)
-    )
-    (property "Datasheet" "~" (at 336.55 40.64 0)
-      (effects (font (size 1.27 1.27)) hide)
-    )
-    (pin "1")
-    (pin "2")
-    (instances
-      (project "flash-32mbit"
-        (path "/5081f4fb-0c92-4cfc-8c52-39777c6d96ed"
-          (reference "R13") (unit 1)
         )
       )
@@
     )
   )
+  (symbol (lib_id "power:VCC") (at 200.66 36.83 0) (mirror y) (unit 1)
+    (in_bom yes) (on_board yes) (dnp no) (fields_autoplaced)
+    (property "Reference" "#PWR040" (at 200.66 40.64 0)
+      (effects (font (size 1.27 1.27)) hide)
+    )
+    (property "Value" "VCC" (at 200.66 33.3281 0)
+      (effects (font (size 1.27 1.27)))
+    )
+    (property "Footprint" "" (at 200.66 36.83 0)
+      (effects (font (size 1.27 1.27)) hide)
+    )
+    (property "Datasheet" "" (at 200.66 36.83 0)
+      (effects (font (size 1.27 1.27)) hide)
+    )
+    (pin "1")
+    (instances
+      (project "flash-32mbit"
+        (path "/5081f4fb-0c92-4cfc-8c52-39777c6d96ed"
+          (reference "#PWR040") (unit 1)
+        )
+      )
+    )
+  )
   (symbol (lib_id "power:GND") (at 259.08 80.01 0) (unit 1)
     (in_bom yes) (on_board yes) (dnp no) (fields_autoplaced)
@@
         )
       )
-    )
-  )
-  (symbol (lib_id "power:+5V") (at 200.66 36.83 0) (unit 1)
-    (in_bom yes) (on_board yes) (dnp no) (fields_autoplaced)
-    (property "Reference" "#PWR09" (at 200.66 40.64 0)
-      (effects (font (size 1.27 1.27)) hide)
-    )
-    (property "Value" "+5V" (at 200.66 31.75 0)
-      (effects (font (size 1.27 1.27)))
-    )
-    (property "Footprint" "" (at 200.66 36.83 0)
-      (effects (font (size 1.27 1.27)) hide)
-    )
-    (property "Datasheet" "" (at 200.66 36.83 0)
-      (effects (font (size 1.27 1.27)) hide)
-    )
-    (pin "1")
-    (instances
-      (project "flash-32mbit"
-        (path "/5081f4fb-0c92-4cfc-8c52-39777c6d96ed"
-          (reference "#PWR09") (unit 1)
-        )
-      )
-    )
-  )
-  (symbol (lib_id "power:+5V") (at 325.12 36.83 0) (unit 1)
-    (in_bom yes) (on_board yes) (dnp no)
-    (property "Reference" "#PWR037" (at 325.12 40.64 0)
-      (effects (font (size 1.27 1.27)) hide)
-    )
-    (property "Value" "+5V" (at 325.12 33.02 0)
-      (effects (font (size 1.27 1.27)))
-    )
-    (property "Footprint" "" (at 325.12 36.83 0)
-      (effects (font (size 1.27 1.27)) hide)
-    )
-    (property "Datasheet" "" (at 325.12 36.83 0)
-      (effects (font (size 1.27 1.27)) hide)
-    )
-    (pin "1")
-    (instances
-      (project "flash-32mbit"
-        (path "/5081f4fb-0c92-4cfc-8c52-39777c6d96ed"
-          (reference "#PWR037") (unit 1)
-        )
-      )
