File: pcb/flash-32mbit/flash-32mbit.kicad_sch (KiCad schematic)
At the start: 34 parts, among them U1 IS62C256AL-45ULI, U2 SN74LVC1G04, U3 RP2040-Tiny, U4 LH28F320SKTD-L70, U5 MCP23S17-E/SO, U6 MCP23S17-E/SO, U7 MCP23S17-E/SO

Commit message: Fixes SRAM low power mode on schematic, needs routing
Connections:
- net VCC: no longer R4.2
- net at C1.2, D1.3, U1.28 (VDD): now also R4.2
Other:
- note added: "/INSERTED allows Pico to run a different program when connected to USB or Loopy for example, run a USB host and forward serial when the cart is plugged in but run the flashing firmware when ejected"
- note added: "CE pulled high when disconnected for low power/data retention state This should not depend on cart power!"
- note added: "Provide 3V power to board when plugged into USB Protect board from being powered when plugged into console"
- note removed: "CE pulled high when disconnected for power down"
- note removed: "Inserted allows Pico to run a different program when connected to USB or Loopy for example, run a USB host and forward serial when connected to Loopy but run the flashing firmware when connected to USB"
- note removed: "Provide 3V power to board when plugged into USB Protect board from being powered when plugged into console or 5V entering 3.3V net when R13 populated"
- moved on the sheet: C1, D1, R6

Commit message: rev6 RC
Parts:
- removed R14, R16: 1K, Resistor_SMD:R_0805_2012Metric_Pad1.20x1.40mm_HandSolder, symbol Device:R
- removed R15, R17: 2K2, Resistor_SMD:R_0805_2012Metric_Pad1.20x1.40mm_HandSolder, symbol Device:R
Connections:
- net UART1_RX: no longer names the net of U3.9 (GP9)
- net UART1_TX: no longer names the net of U3.8 (GP8)
- no-connect marks 37 -> 39
Changed lines of the file:
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@@
   (junction (at 53.34 139.7) (diameter 0) (color 0 0 0 0)
   )
-  (junction (at 429.26 60.96) (diameter 0) (color 0 0 0 0)
-  )
   (junction (at 340.36 45.72) (diameter 0) (color 0 0 0 0)
   )
@@
   (junction (at 387.35 92.71) (diameter 0) (color 0 0 0 0)
   )
-  (junction (at 425.45 83.82) (diameter 0) (color 0 0 0 0)
-  )
   (junction (at 123.19 43.18) (diameter 0) (color 0 0 0 0)
   )
@@
   (junction (at 344.17 162.56) (diameter 0) (color 0 0 0 0)
   )
-  (junction (at 425.45 72.39) (diameter 0) (color 0 0 0 0)
-  )
   (junction (at 142.24 99.06) (diameter 0) (color 0 0 0 0)
   )
@@
   (junction (at 147.32 43.18) (diameter 0) (color 0 0 0 0)
   )
+  (no_connect (at 378.46 68.58))
   (no_connect (at 358.14 48.26))
   (no_connect (at 449.58 162.56))
@@
   (no_connect (at 358.14 53.34))
   (no_connect (at 241.3 101.6))
+  (no_connect (at 388.62 60.96))
   (no_connect (at 218.44 43.18))
   (no_connect (at 375.92 68.58))
@@
     (stroke (width 0) (type default))
   )
-  (wire (pts (xy 429.26 60.96) (xy 440.69 60.96))
-    (stroke (width 0) (type default))
-  )
   (wire (pts (xy 147.32 34.29) (xy 147.32 43.18))
     (stroke (width 0) (type default))
@@
     (stroke (width 0) (type default))
   )
-  (wire (pts (xy 425.45 83.82) (xy 429.26 83.82))
-    (stroke (width 0) (type default))
-  )
   (wire (pts (xy 241.3 114.3) (xy 251.46 114.3))
     (stroke (width 0) (type default))
@@
     (stroke (width 0) (type default))
   )
-  (wire (pts (xy 425.45 80.01) (xy 425.45 83.82))
-    (stroke (width 0) (type default))
-  )
   (wire (pts (xy 124.46 132.08) (xy 124.46 137.16))
     (stroke (width 0) (type default))
@@
     (stroke (width 0) (type default))
   )
-  (wire (pts (xy 425.45 83.82) (xy 425.45 87.63))
-    (stroke (width 0) (type default))
-  )
   (wire (pts (xy 346.71 69.85) (xy 358.14 69.85))
     (stroke (width 0) (type default))
@@
     (stroke (width 0) (type default))
   )
-  (wire (pts (xy 420.37 60.96) (xy 429.26 60.96))
-    (stroke (width 0) (type default))
-  )
   (wire (pts (xy 370.84 81.28) (xy 375.92 81.28))
     (stroke (width 0) (type default))
@@
     (stroke (width 0) (type default))
   )
-  (wire (pts (xy 425.45 72.39) (xy 440.69 72.39))
-    (stroke (width 0) (type default))
-  )
   (wire (pts (xy 208.28 104.14) (xy 218.44 104.14))
     (stroke (width 0) (type default))
@@
     (stroke (width 0) (type default))
   )
-  (wire (pts (xy 429.26 68.58) (xy 429.26 83.82))
-    (stroke (width 0) (type default))
-  )
   (wire (pts (xy 111.76 142.24) (xy 120.65 142.24))
     (stroke (width 0) (type default))
@@
     (stroke (width 0) (type default))
   )
-  (wire (pts (xy 378.46 72.39) (xy 378.46 68.58))
-    (stroke (width 0) (type default))
-  )
   (wire (pts (xy 111.76 114.3) (xy 120.65 114.3))
     (stroke (width 0) (type default))
@@
     (stroke (width 0) (type default))
   )
-  (wire (pts (xy 420.37 72.39) (xy 425.45 72.39))
-    (stroke (width 0) (type default))
-  )
   (wire (pts (xy 241.3 93.98) (xy 251.46 93.98))
     (stroke (width 0) (type default))
@@
     (stroke (width 0) (type default))
   )
-  (wire (pts (xy 388.62 60.96) (xy 412.75 60.96))
-    (stroke (width 0) (type default))
-  )
   (wire (pts (xy 72.39 142.24) (xy 86.36 142.24))
     (stroke (width 0) (type default))
@@
     (stroke (width 0) (type default))
   )
-  (wire (pts (xy 378.46 72.39) (xy 412.75 72.39))
-    (stroke (width 0) (type default))
-  )
   (wire (pts (xy 208.28 142.24) (xy 218.44 142.24))
     (stroke (width 0) (type default))
@@
     (effects (font (size 1.27 1.27)) (justify left bottom))
   )
-  (label "RX_D1" (at 440.69 60.96 180) (fields_autoplaced)
-    (effects (font (size 1.27 1.27)) (justify right bottom))
-  )
   (label "GND" (at 449.58 172.72 0) (fields_autoplaced)
     (effects (font (size 1.27 1.27)) (justify left bottom))
@@
     (effects (font (size 1.27 1.27)) (justify right bottom))
   )
-  (label "TX_D1" (at 440.69 72.39 180) (fields_autoplaced)
-    (effects (font (size 1.27 1.27)) (justify right bottom))
-  )
   (label "VCC" (at 297.18 160.02 180) (fields_autoplaced)
     (effects (font (size 1.27 1.27)) (justify right bottom))
@@
     (effects (font (size 1.27 1.27)) (justify left bottom))
   )
-  (label "UART1_RX" (at 378.46 72.39 0) (fields_autoplaced)
-    (effects (font (size 1.27 1.27)) (justify left bottom))
-  )
   (label "D12" (at 120.65 132.08 180) (fields_autoplaced)
     (effects (font (size 1.27 1.27)) (justify right bottom))
@@
     (effects (font (size 1.27 1.27)) (justify left bottom))
   )
-  (label "UART1_TX" (at 388.62 60.96 0) (fields_autoplaced)
-    (effects (font (size 1.27 1.27)) (justify left bottom))
-  )
   (label "A2" (at 251.46 71.12 180) (fields_autoplaced)
     (effects (font (size 1.27 1.27)) (justify right bottom))
@@
     )
   )
-  (symbol (lib_id "Device:R") (at 416.56 72.39 90) (unit 1)
-    (in_bom yes) (on_board yes) (dnp no) (fields_autoplaced)
-    (property "Reference" "R14" (at 416.56 66.04 90)
-      (effects (font (size 1.27 1.27)))
-    )
-    (property "Value" "1K" (at 416.56 68.58 90)
-      (effects (font (size 1.27 1.27)))
-    )
-    (property "Footprint" "Resistor_SMD:R_0805_2012Metric_Pad1.20x1.40mm_HandSolder" (at 416.56 74.168 90)
-      (effects (font (size 1.27 1.27)) hide)
-    )
-    (property "Datasheet" "~" (at 416.56 72.39 0)
-      (effects (font (size 1.27 1.27)) hide)
-    )
-    (pin "1")
-    (pin "2")
-    (instances
-      (project "flash-32mbit"
-        (path "/5081f4fb-0c92-4cfc-8c52-39777c6d96ed"
-          (reference "R14") (unit 1)
-        )
-      )
-    )
-  )
   (symbol (lib_id "power:VCC") (at 106.68 200.66 0) (unit 1)
     (in_bom yes) (on_board yes) (dnp no)
@@
     )
   )
-  (symbol (lib_id "Device:R") (at 416.56 60.96 90) (unit 1)
-    (in_bom yes) (on_board yes) (dnp no) (fields_autoplaced)
-    (property "Reference" "R16" (at 416.56 54.61 90)
-      (effects (font (size 1.27 1.27)))
-    )
-    (property "Value" "1K" (at 416.56 57.15 90)
-      (effects (font (size 1.27 1.27)))
-    )
-    (property "Footprint" "Resistor_SMD:R_0805_2012Metric_Pad1.20x1.40mm_HandSolder" (at 416.56 62.738 90)
-      (effects (font (size 1.27 1.27)) hide)
-    )
-    (property "Datasheet" "~" (at 416.56 60.96 0)
-      (effects (font (size 1.27 1.27)) hide)
-    )
-    (pin "1")
-    (pin "2")
-    (instances
-      (project "flash-32mbit"
-        (path "/5081f4fb-0c92-4cfc-8c52-39777c6d96ed"
-          (reference "R16") (unit 1)
-        )
-      )
-    )
-  )
   (symbol (lib_id "power:VCC") (at 72.39 121.92 0) (unit 1)
     (in_bom yes) (on_board yes) (dnp no)
@@
     )
   )
-  (symbol (lib_id "power:GND") (at 425.45 87.63 0) (unit 1)
-    (in_bom yes) (on_board yes) (dnp no) (fields_autoplaced)
-    (property "Reference" "#PWR013" (at 425.45 93.98 0)
-      (effects (font (size 1.27 1.27)) hide)
-    )
-    (property "Value" "GND" (at 425.45 92.71 0)
-      (effects (font (size 1.27 1.27)))
-    )
-    (property "Footprint" "" (at 425.45 87.63 0)
-      (effects (font (size 1.27 1.27)) hide)
-    )
-    (property "Datasheet" "" (at 425.45 87.63 0)
-      (effects (font (size 1.27 1.27)) hide)
-    )
-    (pin "1")
-    (instances
-      (project "flash-32mbit"
-        (path "/5081f4fb-0c92-4cfc-8c52-39777c6d96ed"
-          (reference "#PWR013") (unit 1)
-        )
-      )
-    )
-  )
   (symbol (lib_id "Device:R_Small") (at 265.43 149.86 270) (unit 1)
     (in_bom yes) (on_board yes) (dnp no) (fields_autoplaced)
@@
         )
       )
-    )
-  )
-  (symbol (lib_id "Device:R") (at 425.45 76.2 0) (unit 1)
-    (in_bom yes) (on_board yes) (dnp no)
-    (property "Reference" "R15" (at 419.1 74.93 0)
-      (effects (font (size 1.27 1.27)) (justify left))
-    )
-    (property "Value" "2K2" (at 419.1 77.47 0)
-      (effects (font (size 1.27 1.27)) (justify left))
-    )
-    (property "Footprint" "Resistor_SMD:R_0805_2012Metric_Pad1.20x1.40mm_HandSolder" (at 423.672 76.2 90)
-      (effects (font (size 1.27 1.27)) hide)
-    )
-    (property "Datasheet" "~" (at 425.45 76.2 0)
-      (effects (font (size 1.27 1.27)) hide)
-    )
-    (pin "1")
-    (pin "2")
-    (instances
-      (project "flash-32mbit"
-        (path "/5081f4fb-0c92-4cfc-8c52-39777c6d96ed"
-          (reference "R15") (unit 1)
-        )
-      )
-    )
-  )
-  (symbol (lib_id "Device:R") (at 429.26 64.77 0) (unit 1)
-    (in_bom yes) (on_board yes) (dnp no)
-    (property "Reference" "R17" (at 422.91 63.5 0)
-      (effects (font (size 1.27 1.27)) (justify left))
-    )
-    (property "Value" "2K2" (at 422.91 66.04 0)
-      (effects (font (size 1.27 1.27)) (justify left))
-    )
-    (property "Footprint" "Resistor_SMD:R_0805_2012Metric_Pad1.20x1.40mm_HandSolder" (at 427.482 64.77 90)
-      (effects (font (size 1.27 1.27)) hide)
-    )
-    (property "Datasheet" "~" (at 429.26 64.77 0)
-      (effects (font (size 1.27 1.27)) hide)
-    )
-    (pin "1")
-    (pin "2")
-    (instances
-      (project "flash-32mbit"
-        (path "/5081f4fb-0c92-4cfc-8c52-39777c6d96ed"
-          (reference "R17") (unit 1)
-        )
-      )

Commit message: Rev7 hardware changes: new SRAM part
Parts:
- removed R4: 100K, Resistor_SMD:R_0805_2012Metric_Pad1.20x1.40mm_HandSolder, symbol Device:R_Small
- removed U1: IS62C256AL-45ULI, LOOPY_SRAM:SOP_28L_330MIL_ISI-L, symbol LOOPY_SRAM:IS62C256AL-45ULI
- added R13, R4: 100K, Resistor_SMD:R_0805_2012Metric_Pad1.20x1.40mm_HandSolder, symbol Device:R
- added U2: AS6C1008-55SIN, LOOPY_SRAM:SOIC127P1410X300-32N, symbol LOOPY_SRAM:AS6C1008-55SIN
- R6: value 1K -> 1K2
- renumbered U4 to U1, U2 to U3, U3 to U4
Connections:
- net +BATT: now also BT1.1 (+); no longer BT1.2 (+)
- net A0: now also U2.12 (A0)
- net A1: now also U2.11 (A1)
- net A10: now also U2.23 (A10)
- net A11: now also U2.25 (A11)
- net A12: now also U2.4 (A12)
- net A13: now also U2.28 (A13)
- net A14: now also U2.3 (A14)
- net A15: now also U2.31 (A15)
- net A16: now also U2.2 (A16)
- net A2: now also U2.10 (A2)
- net A3: now also U2.9 (A3)
- net A4: now also U2.8 (A4)
- net A5: now also U2.7 (A5)
- net A6: now also U2.6 (A6)
- net A7: now also U2.5 (A7)
- net A8: now also U2.27 (A8)
- net A9: now also U2.26 (A9)
- net D0: now also U2.13 (DQ0)
- net D1: now also U2.14 (DQ1)
- net D2: now also U2.15 (DQ2)
- net D3: now also U2.17 (DQ3)
- net D4: now also U2.18 (DQ4)
- net D5: now also U2.19 (DQ5)
- net D6: now also U2.20 (DQ6)
- net D7: now also U2.21 (DQ7)
- net GND: now also BT1.2 (-), R4.1, U2.16 (VSS); no longer BT1.1 (-)
- net OE: now also U2.24 (OE#)
- net RAMCE: now also R13.2, U2.22 (CE#)
- net RAMWE: now also U2.29 (WE#)
- net RESET: now also R4.2, U2.30 (CE2)
- net VCC: now also R13.1
- net VCC_OR_BATT: now reaches C1.2, D1.3
- net VCC_OR_BATT: now also U2.32 (VCC)
- net CLK: no longer names the net of J1.60 (CLK)
- net ROMSTS: no longer names the net of U1.53 (STS)
- net RX_D1: no longer names the net of J1.18 (PB10)
- net TX_D1: no longer names the net of J1.19 (PB11)
- no-connect marks 39 -> 44
Other:
- note added: "CE# is ACTIVE LOW (standby when HIGH) CE2 is ACTIVE HIGH (standby when LOW)"
- note added: "Power SRAM from battery (<3V) when disconnected Power SRAM from VCC when connected to pico (3.3V) or loopy (5V) Prevent VCC from charging battery"
- note added: "Unused SH1 ports"
- note removed: "/INSERTED allows Pico to run a different program when connected to USB or Loopy for example, run a USB host and forward serial when the cart is plugged in but run the flashing firmware when ejected"
- note removed: "CE pulled high when disconnected for low power/data retention state This should not depend on cart power!"
- note removed: "Feature detect pins?"
- note removed: "Loopy UART D0 = available for brew D1 = MIDI"
- note removed: "Power SRAM from battery when disconnected Power SRAM from VCC when connected to pico (3.3V) or loopy (5V) Prevent VCC from charging battery"
- company: (none) -> @partlyhuman
- title: LOOPY Flash Devcart -> FloopyDrive
- moved on the sheet: BT1, C1, C5, C6, C7, D1, D2, J1, R1, R10, R11, R12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

Commit message: Remove redundant pullups?
Parts:
- removed R13: 100K, Resistor_SMD:R_0805_2012Metric_Pad1.20x1.40mm_HandSolder, symbol Device:R
- C1: symbol Device:C -> Device:C_Small
Connections:
- net GND: no longer R4.1
- net VCC: now also R4.1
- net VCC_OR_BATT renamed RAMVDD
Other:
- moved on the sheet: C1

Commit message: Tidying, using RESET to power down flash, marking potentially redundant pullups
Parts:
- removed R1, R2: 1K, Resistor_SMD:R_0805_2012Metric_Pad1.20x1.40mm_HandSolder, symbol Device:R
- added R1, R2: 1K, Resistor_SMD:R_0805_2012Metric_Pad1.20x1.40mm_HandSolder, symbol Device:R_Small
- R10, R11, R12, R4, R9: symbol Device:R -> Device:R_Small
- R3, R5: now not fitted
Connections:
- net F16: now also R2.2
- net F61: now also R1.1
- net GND: now also C3.2
- net RESET: now also U1.16 (~{RP})
- net VCC: now also R1.2, R2.1; no longer U1.16 (~{RP})
- no-connect marks 44 -> 43
Other:
- note added: "* Redundant, depopulate?"
- note removed: "Provide 3V power to board when plugged into USB Protect board from being powered when plugged into console"
- note removed: "Unused SH1 ports"
- note removed: "When Pico disconnected WE pulled high to write protect"
- note removed: "When ROMCE disconnected (no cart), pull CE high for standby"
- moved on the sheet: D2, R10, R4, R8, R9
