File: pcb/flash-32mbit/flash-32mbit.kicad_sch (KiCad schematic)
At the start: 30 parts, among them U1 LH28F320SKTD-L70, U2 AS6C1008-55SIN, U3 SN74LVC1G04, U4 RP2040-Tiny, U5 MCP23S17-E/SO, U6 MCP23S17-E/SO, U7 MCP23S17-E/SO

Commit message: Now that asserting RESET low keeps some things safe, let pico drive RESET high only when ready
Parts:
- removed R4: 100K, Resistor_SMD:R_0805_2012Metric_Pad1.20x1.40mm_HandSolder, symbol Device:R_Small
- added R13: 100K, Resistor_SMD:R_0805_2012Metric_Pad1.20x1.40mm_HandSolder, symbol Device:R_Small
- R3: now fitted
Connections:
- net RAMWE: now also R13.2
- net RESET: now also U7.6 (GPB5)
- net VCC: now also R13.1
- no-connect marks 43 -> 42
Other:
- moved on the sheet: C1
Changed lines of the file:
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@@
   (junction (at 129.54 139.7) (diameter 0) (color 0 0 0 0)
   )
+  (junction (at 124.46 39.37) (diameter 0) (color 0 0 0 0)
+  )
   (junction (at 346.71 215.9) (diameter 0) (color 0 0 0 0)
   )
@@
   (junction (at 167.64 72.39) (diameter 0) (color 0 0 0 0)
   )
-  (junction (at 127 39.37) (diameter 0) (color 0 0 0 0)
-  )
   (junction (at 340.36 148.59) (diameter 0) (color 0 0 0 0)
   )
@@
   (no_connect (at 391.16 193.04))
   (no_connect (at 330.2 106.68))
-  (no_connect (at 360.68 205.74))
   (no_connect (at 299.72 124.46))
   (no_connect (at 299.72 121.92))
@@
     (stroke (width 0) (type default))
   )
-  (wire (pts (xy 185.42 128.27) (xy 173.99 128.27))
+  (wire (pts (xy 175.26 100.33) (xy 185.42 100.33))
     (stroke (width 0) (type default))
   )
-  (wire (pts (xy 175.26 100.33) (xy 185.42 100.33))
+  (wire (pts (xy 175.26 128.27) (xy 185.42 128.27))
     (stroke (width 0) (type default))
   )
@@
     (stroke (width 0) (type default))
   )
-  (wire (pts (xy 110.49 39.37) (xy 127 39.37))
-    (stroke (width 0) (type default))
-  )
   (wire (pts (xy 111.76 127) (xy 120.65 127))
     (stroke (width 0) (type default))
@@
     (stroke (width 0) (type default))
   )
-  (wire (pts (xy 127 39.37) (xy 130.81 39.37))
-    (stroke (width 0) (type default))
-  )
   (wire (pts (xy 288.29 127) (xy 299.72 127))
     (stroke (width 0) (type default))
@@
     (stroke (width 0) (type default))
   )
-  (wire (pts (xy 119.38 46.99) (xy 110.49 46.99))
+  (wire (pts (xy 110.49 46.99) (xy 134.62 46.99))
+    (stroke (width 0) (type default))
+  )
+  (wire (pts (xy 110.49 39.37) (xy 124.46 39.37))
     (stroke (width 0) (type default))
   )
@@
     (stroke (width 0) (type default))
   )
-  (wire (pts (xy 168.91 128.27) (xy 167.64 128.27))
-    (stroke (width 0) (type default))
-  )
   (wire (pts (xy 226.06 121.92) (xy 226.06 123.19))
     (stroke (width 0) (type default))
@@
     (stroke (width 0) (type default))
   )
+  (wire (pts (xy 124.46 39.37) (xy 130.81 39.37))
+    (stroke (width 0) (type default))
+  )
   (wire (pts (xy 111.76 149.86) (xy 120.65 149.86))
     (stroke (width 0) (type default))
@@
     (effects (font (size 1.27 1.27)) (justify right bottom))
   )
-  (text "* Redundant, depopulate?" (at 132.08 111.76 0)
-    (effects (font (size 1.27 1.27)) (justify left bottom))
-  )
   (text "SPI IO Expanders, sharing a bus" (at 299.72 181.61 0)
     (effects (font (size 1.27 1.27)) (justify left bottom))
@@
     (effects (font (size 1.27 1.27)) (justify right bottom))
   )
+  (label "RESET" (at 360.68 205.74 180) (fields_autoplaced)
+    (effects (font (size 1.27 1.27)) (justify right bottom))
+  )
   (label "D0" (at 175.26 125.73 0) (fields_autoplaced)
     (effects (font (size 1.27 1.27)) (justify left bottom))
@@
   )
   (symbol (lib_id "Device:R_Small") (at 128.27 106.68 270) (mirror x) (unit 1)
-    (in_bom yes) (on_board yes) (dnp yes)
+    (in_bom yes) (on_board yes) (dnp no)
     (property "Reference" "R3" (at 128.27 109.22 90)
       (effects (font (size 1.27 1.27)))
@@
     )
   )
-  (symbol (lib_id "power:VCC") (at 167.64 128.27 0) (unit 1)
-    (in_bom yes) (on_board yes) (dnp no) (fields_autoplaced)
-    (property "Reference" "#PWR05" (at 167.64 132.08 0)
-      (effects (font (size 1.27 1.27)) hide)
-    )
-    (property "Value" "VCC" (at 167.64 124.7681 0)
-      (effects (font (size 1.27 1.27)))
-    )
-    (property "Footprint" "" (at 167.64 128.27 0)
-      (effects (font (size 1.27 1.27)) hide)
-    )
-    (property "Datasheet" "" (at 167.64 128.27 0)
-      (effects (font (size 1.27 1.27)) hide)
-    )
-    (pin "1")
-    (instances
-      (project "flash-32mbit"
-        (path "/5081f4fb-0c92-4cfc-8c52-39777c6d96ed"
-          (reference "#PWR05") (unit 1)
-        )
-      )
-    )
-  )
   (symbol (lib_id "power:GND") (at 72.39 156.21 0) (unit 1)
     (in_bom yes) (on_board yes) (dnp no) (fields_autoplaced)
@@
     )
   )
+  (symbol (lib_id "Device:R_Small") (at 134.62 44.45 0) (unit 1)
+    (in_bom yes) (on_board yes) (dnp no) (fields_autoplaced)
+    (property "Reference" "R13" (at 137.16 43.18 0)
+      (effects (font (size 1.27 1.27)) (justify left))
+    )
+    (property "Value" "100K" (at 137.16 45.72 0)
+      (effects (font (size 1.27 1.27)) (justify left))
+    )
+    (property "Footprint" "Resistor_SMD:R_0805_2012Metric_Pad1.20x1.40mm_HandSolder" (at 134.62 44.45 0)
+      (effects (font (size 1.27 1.27)) hide)
+    )
+    (property "Datasheet" "~" (at 134.62 44.45 0)
+      (effects (font (size 1.27 1.27)) hide)
+    )
+    (pin "1")
+    (pin "2")
+    (instances
+      (project "flash-32mbit"
+        (path "/5081f4fb-0c92-4cfc-8c52-39777c6d96ed"
+          (reference "R13") (unit 1)
+        )
+      )
+    )
+  )
   (symbol (lib_id "power:GND") (at 167.64 152.4 0) (unit 1)
     (in_bom yes) (on_board yes) (dnp no) (fields_autoplaced)
@@
     )
   )
-  (symbol (lib_id "Device:C_Small") (at 288.29 213.36 90) (unit 1)
-    (in_bom yes) (on_board yes) (dnp no) (fields_autoplaced)
-    (property "Reference" "C6" (at 288.2963 208.28 90)
-      (effects (font (size 1.27 1.27)))
+  (symbol (lib_id "power:VCC") (at 134.62 41.91 0) (unit 1)
+    (in_bom yes) (on_board yes) (dnp no)
+    (property "Reference" "#PWR09" (at 134.62 45.72 0)
+      (effects (font (size 1.27 1.27)) hide)
     )
-    (property "Value" "0.1u" (at 288.2963 210.82 90)
+    (property "Value" "VCC" (at 134.62 38.1 0)
       (effects (font (size 1.27 1.27)))
     )
-    (property "Footprint" "Capacitor_SMD:C_0805_2012Metric_Pad1.18x1.45mm_HandSolder" (at 288.29 213.36 0)
+    (property "Footprint" "" (at 134.62 41.91 0)
       (effects (font (size 1.27 1.27)) hide)
     )
-    (property "Datasheet" "~" (at 288.29 213.36 0)
+    (property "Datasheet" "" (at 134.62 41.91 0)
       (effects (font (size 1.27 1.27)) hide)
     )
     (pin "1")
-    (pin "2")
     (instances
       (project "flash-32mbit"
         (path "/5081f4fb-0c92-4cfc-8c52-39777c6d96ed"
-          (reference "C6") (unit 1)
+          (reference "#PWR09") (unit 1)
         )
       )
     )
   )
-  (symbol (lib_id "Device:R_Small") (at 171.45 128.27 90) (unit 1)
-    (in_bom yes) (on_board yes) (dnp no)
-    (property "Reference" "R4" (at 171.45 132.08 90)
+  (symbol (lib_id "Device:C_Small") (at 288.29 213.36 90) (unit 1)
+    (in_bom yes) (on_board yes) (dnp no) (fields_autoplaced)
+    (property "Reference" "C6" (at 288.2963 208.28 90)
       (effects (font (size 1.27 1.27)))
     )
-    (property "Value" "100K" (at 171.45 134.62 90)
+    (property "Value" "0.1u" (at 288.2963 210.82 90)
       (effects (font (size 1.27 1.27)))
     )
-    (property "Footprint" "Resistor_SMD:R_0805_2012Metric_Pad1.20x1.40mm_HandSolder" (at 171.45 130.048 90)
+    (property "Footprint" "Capacitor_SMD:C_0805_2012Metric_Pad1.18x1.45mm_HandSolder" (at 288.29 213.36 0)
       (effects (font (size 1.27 1.27)) hide)
     )
-    (property "Datasheet" "~" (at 171.45 128.27 0)
+    (property "Datasheet" "~" (at 288.29 213.36 0)
       (effects (font (size 1.27 1.27)) hide)
     )
@@
       (project "flash-32mbit"
         (path "/5081f4fb-0c92-4cfc-8c52-39777c6d96ed"
-          (reference "R4") (unit 1)
+          (reference "C6") (unit 1)
         )
       )
@@
     )
   )
-  (symbol (lib_id "Device:C_Small") (at 127 41.91 180) (unit 1)
+  (symbol (lib_id "Device:C_Small") (at 124.46 36.83 0) (unit 1)
     (in_bom yes) (on_board yes) (dnp no)
-    (property "Reference" "C1" (at 132.08 44.45 0)
+    (property "Reference" "C1" (at 119.38 34.29 0)
       (effects (font (size 1.27 1.27)) (justify left))
     )
-    (property "Value" "1u" (at 132.08 41.91 0)
+    (property "Value" "1u" (at 119.38 36.83 0)
       (effects (font (size 1.27 1.27)) (justify left))
     )
-    (property "Footprint" "Capacitor_SMD:C_0805_2012Metric_Pad1.18x1.45mm_HandSolder" (at 126.0348 38.1 0)
+    (property "Footprint" "Capacitor_SMD:C_0805_2012Metric_Pad1.18x1.45mm_HandSolder" (at 125.4252 40.64 0)
       (effects (font (size 1.27 1.27)) hide)
     )
-    (property "Datasheet" "~" (at 127 41.91 0)
+    (property "Datasheet" "~" (at 124.46 36.83 0)
       (effects (font (size 1.27 1.27)) hide)
     )
@@
     )
   )
-  (symbol (lib_id "power:GND") (at 127 44.45 0) (mirror y) (unit 1)
+  (symbol (lib_id "power:GND") (at 124.46 34.29 90) (mirror x) (unit 1)
     (in_bom yes) (on_board yes) (dnp no)
-    (property "Reference" "#PWR016" (at 127 50.8 0)
+    (property "Reference" "#PWR016" (at 130.81 34.29 0)
       (effects (font (size 1.27 1.27)) hide)
     )
-    (property "Value" "GND" (at 127 49.53 0)
+    (property "Value" "GND" (at 128.27 34.29 0)
       (effects (font (size 1.27 1.27)))
     )
-    (property "Footprint" "" (at 127 44.45 0)
+    (property "Footprint" "" (at 124.46 34.29 0)
       (effects (font (size 1.27 1.27)) hide)
     )
-    (property "Datasheet" "" (at 127 44.45 0)
+    (property "Datasheet" "" (at 124.46 34.29 0)
       (effects (font (size 1.27 1.27)) hide)
     )

Commit message: /RESET pulled low, power up and down conditions should be covered by this and extra control pullups should be redundant
Parts:
- added R4: 100K, Resistor_SMD:R_0805_2012Metric_Pad1.20x1.40mm_HandSolder, symbol Device:R_Small
- R13, R3: now not fitted
Connections:
- net GND: now also R4.2
- net RESET: now also R4.1
Changed lines of the file:
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@@
   (title_block
     (title "FloopyDrive")
-    (date "2023-09-27")
+    (date "2023-09-28")
     (rev "7")
     (company "@partlyhuman")
@@
     (stroke (width 0) (type default))
   )
-  (wire (pts (xy 175.26 128.27) (xy 185.42 128.27))
-    (stroke (width 0) (type default))
-  )
   (wire (pts (xy 74.93 46.99) (xy 85.09 46.99))
     (stroke (width 0) (type default))
@@
     (stroke (width 0) (type default))
   )
+  (wire (pts (xy 167.64 129.54) (xy 167.64 128.27))
+    (stroke (width 0) (type default))
+  )
   (wire (pts (xy 208.28 49.53) (xy 218.44 49.53))
     (stroke (width 0) (type default))
@@
     (stroke (width 0) (type default))
   )
+  (wire (pts (xy 172.72 128.27) (xy 185.42 128.27))
+    (stroke (width 0) (type default))
+  )
   (wire (pts (xy 39.37 139.7) (xy 53.34 139.7))
     (stroke (width 0) (type default))
@@
   )
   (symbol (lib_id "Device:R_Small") (at 128.27 106.68 270) (mirror x) (unit 1)
-    (in_bom yes) (on_board yes) (dnp no)
+    (in_bom yes) (on_board yes) (dnp yes)
     (property "Reference" "R3" (at 128.27 109.22 90)
       (effects (font (size 1.27 1.27)))
@@
     )
   )
+  (symbol (lib_id "power:GND") (at 167.64 129.54 0) (unit 1)
+    (in_bom yes) (on_board yes) (dnp no) (fields_autoplaced)
+    (property "Reference" "#PWR05" (at 167.64 135.89 0)
+      (effects (font (size 1.27 1.27)) hide)
+    )
+    (property "Value" "GND" (at 167.64 134.62 0)
+      (effects (font (size 1.27 1.27)))
+    )
+    (property "Footprint" "" (at 167.64 129.54 0)
+      (effects (font (size 1.27 1.27)) hide)
+    )
+    (property "Datasheet" "" (at 167.64 129.54 0)
+      (effects (font (size 1.27 1.27)) hide)
+    )
+    (pin "1")
+    (instances
+      (project "flash-32mbit"
+        (path "/5081f4fb-0c92-4cfc-8c52-39777c6d96ed"
+          (reference "#PWR05") (unit 1)
+        )
+      )
+    )
+  )
   (symbol (lib_id "Device:R_Small") (at 53.34 143.51 0) (mirror x) (unit 1)
     (in_bom yes) (on_board yes) (dnp no) (fields_autoplaced)
@@
   )
   (symbol (lib_id "Device:R_Small") (at 134.62 44.45 0) (unit 1)
-    (in_bom yes) (on_board yes) (dnp no) (fields_autoplaced)
+    (in_bom yes) (on_board yes) (dnp yes) (fields_autoplaced)
     (property "Reference" "R13" (at 137.16 43.18 0)
       (effects (font (size 1.27 1.27)) (justify left))
@@
         )
       )
+    )
+  )
+  (symbol (lib_id "Device:R_Small") (at 170.18 128.27 270) (unit 1)
+    (in_bom yes) (on_board yes) (dnp no) (fields_autoplaced)
+    (property "Reference" "R4" (at 170.18 123.19 90)
+      (effects (font (size 1.27 1.27)))
+    )
+    (property "Value" "100K" (at 170.18 125.73 90)
+      (effects (font (size 1.27 1.27)))
+    )
+    (property "Footprint" "Resistor_SMD:R_0805_2012Metric_Pad1.20x1.40mm_HandSolder" (at 170.18 128.27 0)
+      (effects (font (size 1.27 1.27)) hide)
+    )
+    (property "Datasheet" "~" (at 170.18 128.27 0)
+      (effects (font (size 1.27 1.27)) hide)
+    )
+    (pin "1")
+    (pin "2")
+    (instances
+      (project "flash-32mbit"
+        (path "/5081f4fb-0c92-4cfc-8c52-39777c6d96ed"
+          (reference "R4") (unit 1)
+        )
+      )

Commit message: Fixes voltage divider resistor order
Parts:
- R10, R12: value 2K2 -> 1K
- R11, R9: value 1K -> 2K2
Changed lines of the file:
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@@
       (effects (font (size 1.27 1.27)) (justify left))
     )
-    (property "Value" "2K2" (at 345.44 144.78 0)
+    (property "Value" "1K" (at 345.44 144.78 0)
       (effects (font (size 1.27 1.27)) (justify left))
     )
@@
       (effects (font (size 1.27 1.27)))
     )
-    (property "Value" "1K" (at 332.74 137.16 90)
+    (property "Value" "2K2" (at 332.74 137.16 90)
       (effects (font (size 1.27 1.27)))
     )
@@
       (effects (font (size 1.27 1.27)))
     )
-    (property "Value" "1K" (at 332.74 146.05 90)
+    (property "Value" "2K2" (at 332.74 146.05 90)
       (effects (font (size 1.27 1.27)))
     )
@@
   (symbol (lib_id "Device:R_Small") (at 340.36 152.4 0) (unit 1)
     (in_bom yes) (on_board yes) (dnp no) (fields_autoplaced)
-    (property "Reference" "R10" (at 337.82 151.13 0)
-      (effects (font (size 1.27 1.27)) (justify right))
-    )
-    (property "Value" "2K2" (at 337.82 153.67 0)
-      (effects (font (size 1.27 1.27)) (justify right))
+    (property "Reference" "R10" (at 342.9 151.13 0)
+      (effects (font (size 1.27 1.27)) (justify left))
+    )
+    (property "Value" "1K" (at 342.9 153.67 0)
+      (effects (font (size 1.27 1.27)) (justify left))
     )
     (property "Footprint" "Resistor_SMD:R_0805_2012Metric_Pad1.20x1.40mm_HandSolder" (at 338.582 152.4 90)
