File: pcb/flash-32mbit/flash-32mbit.kicad_sch (KiCad schematic)
At the start: 31 parts, among them U1 LH28F320SKTD-L70, U2 AS6C1008-55SIN, U3 SN74LVC1G04, U4 RP2040-Tiny, U5 MCP23S17-E/SO, U6 MCP23S17-E/SO, U7 MCP23S17-E/SO

Commit message: Revert "Fixes voltage divider resistor order"
This reverts commit 804d36860d2d035c957d0a79ec73a7ea4df5a67d.
Parts:
- R10, R12: value 1K -> 2K2
- R11, R9: value 2K2 -> 1K
Changed lines of the file:
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@@
       (effects (font (size 1.27 1.27)) (justify left))
     )
-    (property "Value" "1K" (at 345.44 144.78 0)
+    (property "Value" "2K2" (at 345.44 144.78 0)
       (effects (font (size 1.27 1.27)) (justify left))
     )
@@
       (effects (font (size 1.27 1.27)))
     )
-    (property "Value" "2K2" (at 332.74 137.16 90)
+    (property "Value" "1K" (at 332.74 137.16 90)
       (effects (font (size 1.27 1.27)))
     )
@@
       (effects (font (size 1.27 1.27)))
     )
-    (property "Value" "2K2" (at 332.74 146.05 90)
+    (property "Value" "1K" (at 332.74 146.05 90)
       (effects (font (size 1.27 1.27)))
     )
@@
   (symbol (lib_id "Device:R_Small") (at 340.36 152.4 0) (unit 1)
     (in_bom yes) (on_board yes) (dnp no) (fields_autoplaced)
-    (property "Reference" "R10" (at 342.9 151.13 0)
-      (effects (font (size 1.27 1.27)) (justify left))
-    )
-    (property "Value" "1K" (at 342.9 153.67 0)
-      (effects (font (size 1.27 1.27)) (justify left))
+    (property "Reference" "R10" (at 337.82 151.13 0)
+      (effects (font (size 1.27 1.27)) (justify right))
+    )
+    (property "Value" "2K2" (at 337.82 153.67 0)
+      (effects (font (size 1.27 1.27)) (justify right))
     )
     (property "Footprint" "Resistor_SMD:R_0805_2012Metric_Pad1.20x1.40mm_HandSolder" (at 338.582 152.4 90)

Commit message: Corrects serial RX and fixes issue with unpowered serial TX
Parts:
- added Q1: BSS138, Package_TO_SOT_SMD:SOT-23, symbol Transistor_FET:BSS138
- added R13: 1K, Resistor_SMD:R_0805_2012Metric_Pad1.20x1.40mm_HandSolder, symbol Device:R_Small
- R11: value 1K -> 10K
- renumbered R13 to R14
Connections:
- net GND: now also R11.1; no longer R12.2
- net RX_D0: now also R13.2; no longer R11.2, R12.1
- net TX_D0: no longer R10.1
- net UART0_RX: now also R10.1
- net UART0_TX: now also R11.2, Q1.2 (S); no longer R11.1
- net VCC: now also R12.1
- net 3V3 renamed +3V3
- net +3V3: now also Q1.1 (G)
- new net: Q1.3 (D), R12.2, R13.1
Other:
- note added: "Loopy TX / Pico RX Divide down Loopy 5V to Pico 3.5V"
- note added: "Pico TX / Loopy RX Level shift 3.3V to 5V Prevent unpowered Pico from sinking to 0, seen as invalid data by UART"
- note added: "SPI IO Expanders, sharing a single SPI bus"
- note added: "Serial debugging (optional, do not populate if not needed)"
- note removed: "SPI IO Expanders, sharing a bus"
- moved on the sheet: D2, R10, R11, R12, R9, U4

Commit message: Rev8 changes mostly to serial
Parts:
- R11: value 10K -> 100K
- renumbered Q1 to D3
Other:
- note added: "Programming power only when pico on No programming power when pico off + decoupling"
- note removed: "* Redundant, depopulate?"
- moved on the sheet: C4, R7

Commit message: Micro minor tweaks
Other:
- moved on the sheet: R2
Changed lines of the file:
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@@
   (junction (at 46.99 139.7) (diameter 0) (color 0 0 0 0)
   )
+  (junction (at 163.83 74.93) (diameter 0) (color 0 0 0 0)
+  )
   (junction (at 29.21 27.94) (diameter 0) (color 0 0 0 0)
   )
@@
   )
   (junction (at 325.12 142.24) (diameter 0) (color 0 0 0 0)
-  )
-  (junction (at 167.64 72.39) (diameter 0) (color 0 0 0 0)
   )
   (junction (at 349.25 142.24) (diameter 0) (color 0 0 0 0)
@@
     (stroke (width 0) (type default))
   )
-  (wire (pts (xy 167.64 77.47) (xy 167.64 72.39))
+  (wire (pts (xy 163.83 68.58) (xy 163.83 74.93))
     (stroke (width 0) (type default))
   )
@@
     (stroke (width 0) (type default))
   )
+  (wire (pts (xy 185.42 72.39) (xy 175.26 72.39))
+    (stroke (width 0) (type default))
+  )
   (wire (pts (xy 60.96 137.16) (xy 86.36 137.16))
     (stroke (width 0) (type default))
@@
     (stroke (width 0) (type default))
   )
+  (wire (pts (xy 175.26 72.39) (xy 175.26 74.93))
+    (stroke (width 0) (type default))
+  )
   (wire (pts (xy 185.42 110.49) (xy 167.64 110.49))
     (stroke (width 0) (type default))
@@
     (stroke (width 0) (type default))
   )
-  (wire (pts (xy 167.64 68.58) (xy 167.64 72.39))
-    (stroke (width 0) (type default))
-  )
   (wire (pts (xy 110.49 41.91) (xy 119.38 41.91))
     (stroke (width 0) (type default))
@@
     (stroke (width 0) (type default))
   )
+  (wire (pts (xy 175.26 74.93) (xy 163.83 74.93))
+    (stroke (width 0) (type default))
+  )
   (wire (pts (xy 285.75 215.9) (xy 285.75 218.44))
     (stroke (width 0) (type default))
@@
     (stroke (width 0) (type default))
   )
-  (wire (pts (xy 167.64 77.47) (xy 168.91 77.47))
+  (wire (pts (xy 163.83 77.47) (xy 165.1 77.47))
     (stroke (width 0) (type default))
   )
@@
     (stroke (width 0) (type default))
   )
-  (wire (pts (xy 167.64 72.39) (xy 185.42 72.39))
-    (stroke (width 0) (type default))
-  )
   (wire (pts (xy 226.06 148.59) (xy 224.79 148.59))
     (stroke (width 0) (type default))
@@
     (stroke (width 0) (type default))
   )
-  (wire (pts (xy 173.99 77.47) (xy 185.42 77.47))
+  (wire (pts (xy 170.18 77.47) (xy 185.42 77.47))
     (stroke (width 0) (type default))
   )
@@
   )
   (wire (pts (xy 77.47 160.02) (xy 86.36 160.02))
+    (stroke (width 0) (type default))
+  )
+  (wire (pts (xy 163.83 74.93) (xy 163.83 77.47))
     (stroke (width 0) (type default))
   )
@@
     )
   )
-  (symbol (lib_id "power:VCC") (at 167.64 68.58 0) (unit 1)
+  (symbol (lib_id "power:VCC") (at 163.83 68.58 0) (unit 1)
     (in_bom yes) (on_board yes) (dnp no)
-    (property "Reference" "#PWR025" (at 167.64 72.39 0)
-      (effects (font (size 1.27 1.27)) hide)
-    )
-    (property "Value" "VCC" (at 167.64 64.77 0)
-      (effects (font (size 1.27 1.27)))
-    )
-    (property "Footprint" "" (at 167.64 68.58 0)
-      (effects (font (size 1.27 1.27)) hide)
-    )
-    (property "Datasheet" "" (at 167.64 68.58 0)
+    (property "Reference" "#PWR025" (at 163.83 72.39 0)
+      (effects (font (size 1.27 1.27)) hide)
+    )
+    (property "Value" "VCC" (at 163.83 64.77 0)
+      (effects (font (size 1.27 1.27)))
+    )
+    (property "Footprint" "" (at 163.83 68.58 0)
+      (effects (font (size 1.27 1.27)) hide)
+    )
+    (property "Datasheet" "" (at 163.83 68.58 0)
       (effects (font (size 1.27 1.27)) hide)
     )
@@
     )
   )
-  (symbol (lib_id "Device:R_Small") (at 171.45 77.47 90) (unit 1)
+  (symbol (lib_id "Device:R_Small") (at 167.64 77.47 90) (unit 1)
     (in_bom yes) (on_board yes) (dnp no) (fields_autoplaced)
-    (property "Reference" "R2" (at 171.45 80.01 90)
-      (effects (font (size 1.27 1.27)))
-    )
-    (property "Value" "1K" (at 171.45 82.55 90)
-      (effects (font (size 1.27 1.27)))
-    )
-    (property "Footprint" "Resistor_SMD:R_0805_2012Metric_Pad1.20x1.40mm_HandSolder" (at 171.45 79.248 90)
-      (effects (font (size 1.27 1.27)) hide)
-    )
-    (property "Datasheet" "~" (at 171.45 77.47 0)
+    (property "Reference" "R2" (at 167.64 80.01 90)
+      (effects (font (size 1.27 1.27)))
+    )
+    (property "Value" "1K" (at 167.64 82.55 90)
+      (effects (font (size 1.27 1.27)))
+    )
+    (property "Footprint" "Resistor_SMD:R_0805_2012Metric_Pad1.20x1.40mm_HandSolder" (at 167.64 79.248 90)
+      (effects (font (size 1.27 1.27)) hide)
+    )
+    (property "Datasheet" "~" (at 167.64 77.47 0)
       (effects (font (size 1.27 1.27)) hide)
     )
@@
   )
   (symbol (lib_id "power:GND") (at 226.06 78.74 0) (unit 1)
-    (in_bom yes) (on_board yes) (dnp no) (fields_autoplaced)
+    (in_bom yes) (on_board yes) (dnp no)
     (property "Reference" "#PWR026" (at 226.06 85.09 0)
       (effects (font (size 1.27 1.27)) hide)
     )
-    (property "Value" "GND" (at 226.06 83.82 0)
+    (property "Value" "GND" (at 226.06 82.55 0)
       (effects (font (size 1.27 1.27)))
     )
@@
       (effects (font (size 1.27 1.27)) hide)
     )
-    (property "Value" "GND" (at 172.72 74.93 0)
-      (effects (font (size 1.27 1.27)))
-    )
+    (property "Value" "GND" (at 172.72 73.66 0)
+      (effects (font (size 1.27 1.27)))
+    )

Commit message: Reorganize power nets
Parts:
- added D4, D5: BAT54C, Package_TO_SOT_SMD:SOT-23, symbol Diode:BAT54C
- R1: value 1K -> 1K2
- R2: footprint Resistor_SMD:R_0805_2012Metric_Pad1.20x1.40mm_HandSolder -> (none)
- R6: value 1K2 -> 1K; footprint Resistor_SMD:R_0805_2012Metric_Pad1.20x1.40mm_HandSolder -> (none)
Connections:
- net +BATT: now also R1.2; no longer R6.2
- net F16: now also R2.1; no longer R2.2
- net F61: now also R6.1; no longer R1.1
- net VCC: now also D4.3, D5.3; no longer J1.1 (+5V), J1.14 (+5V), J1.29 (+5V), J1.57 (+5V), J1.89 (+5V), R1.2, R14.1, R2.1
- net at D1.1: now also R1.1; no longer R6.1
- net RAMVDD renamed VMEM
- net VMEM: now also R14.1
- new net +5V: D4.1, D4.2, D5.1, D5.2, J1.1 (+5V), J1.14 (+5V), J1.29 (+5V), J1.57 (+5V), J1.89 (+5V), R2.2, R6.2
Other:
- moved on the sheet: BT1, C1

Commit message: Firewall VCC fill from pins
Parts:
- R2, R6: footprint (none) -> Resistor_SMD:R_0805_2012Metric_Pad1.20x1.40mm_HandSolder
Changed lines of the file:
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@@
       (effects (font (size 1.27 1.27)))
     )
-    (property "Footprint" "" (at 184.15 189.23 0)
+    (property "Footprint" "Resistor_SMD:R_0805_2012Metric_Pad1.20x1.40mm_HandSolder" (at 184.15 189.23 0)
       (effects (font (size 1.27 1.27)) hide)
     )
@@
   )
   (symbol (lib_id "Device:R_Small") (at 134.62 44.45 0) (unit 1)
-    (in_bom yes) (on_board yes) (dnp yes) (fields_autoplaced)
+    (in_bom yes) (on_board no) (dnp yes) (fields_autoplaced)
     (property "Reference" "R14" (at 137.16 43.18 0)
       (effects (font (size 1.27 1.27)) (justify left))
@@
       (effects (font (size 1.27 1.27)) hide)
     )
+    (property "Notes" "" (at 134.62 44.45 0)
+      (effects (font (size 1.27 1.27)))
+    )
     (pin "1")
     (pin "2")
@@
       (effects (font (size 1.27 1.27)))
     )
-    (property "Footprint" "" (at 207.01 189.23 0)
-      (effects (font (size 1.27 1.27)) hide)
-    )
+    (property "Footprint" "Resistor_SMD:R_0805_2012Metric_Pad1.20x1.40mm_HandSolder" (at 207.01 189.23 0)
+      (effects (font (size 1.27 1.27)) hide)
+    )

Commit message: Cleaning up REV8 design
Other:
- note added: "CONTROLLER"
- note added: "CONTROLLER I/O"
- note added: "POWER"
- note added: "Pullups, may indicate features to Loopy"
- note added: "SERIAL"
- note removed: "PROGRAM"
Changed lines of the file:
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@@
     (effects (font (size 1.27 1.27)) (justify right bottom))
+  )
+  (text "POWER" (at 63.5 228.6 0)
+    (effects (font (size 5.08 5.08)) (justify left bottom))
   )
   (text "RAM" (at 64.77 34.29 0)
@@
     (effects (font (size 1.27 1.27)) (justify right bottom))
   )
+  (text "Pullups, may indicate features to Loopy" (at 175.26 177.8 0)
+    (effects (font (size 1.27 1.27)) (justify left bottom))
+  )
   (text "Serial debugging\n(optional, do not populate if not needed)"
     (at 299.72 100.33 0)
@@
     (effects (font (size 1.27 1.27)) (justify left bottom))
   )
+  (text "SERIAL" (at 299.72 115.57 0)
+    (effects (font (size 5.08 5.08)) (justify left bottom))
+  )
   (text "SPI IO Expanders, sharing a single SPI bus" (at 299.72 181.61 0)
     (effects (font (size 1.27 1.27)) (justify left bottom))
@@
     (effects (font (size 1.27 1.27)) (justify left bottom))
   )
-  (text "PROGRAM" (at 299.72 34.29 0)
+  (text "CONTROLLER" (at 299.72 34.29 0)
+    (effects (font (size 5.08 5.08)) (justify left bottom))
+  )
+  (text "CONTROLLER I/O" (at 300.99 175.26 0)
     (effects (font (size 5.08 5.08)) (justify left bottom))
   )
@@
   )
   (symbol (lib_id "Device:R_Small") (at 134.62 44.45 0) (unit 1)
-    (in_bom yes) (on_board no) (dnp yes) (fields_autoplaced)
+    (in_bom yes) (on_board yes) (dnp yes) (fields_autoplaced)
     (property "Reference" "R14" (at 137.16 43.18 0)
       (effects (font (size 1.27 1.27)) (justify left))

Commit message: Consolidating blocker diodes and using higher current PMEG2005CT
Parts:
- removed D2, D4, D5: BAT54C, Package_TO_SOT_SMD:SOT-23, symbol Diode:BAT54C
- removed R7: 100K, Resistor_SMD:R_0805_2012Metric_Pad1.20x1.40mm_HandSolder, symbol Device:R_Small
- added D2: PMEG2005CT_215, Package_TO_SOT_SMD:SOT-23-3, symbol LOOPY_Diode:PMEG2005CT_215
- R3: now fitted
Connections:
- net +3V3: now also D2.2
- net +5V: now also D2.1
- net VCC: now also D2.3
Other:
- moved on the sheet: BT1, D1, R1, R5
